File: ultrasonic_localization/ultrasonic_localization.sch (KiCad schematic (older format))
At the start: 2 parts

Commit message: updated and created some schematic components
Parts:
- added U?: LSF0204PWR, Housings_SSOP:TSSOP-14_4.4x5mm_Pitch0.65mm, symbol LSF0204PWR
- added U? (x2): TCT40-16R/T, TCT40-16R_T:TCT40-16R_T, symbol TCT40-16R/T
- added Y?: ABM11AIG-20.000MHZ-4Z-T3, Crystals:Crystal_SMD_2016-4pin_2.0x1.6mm, symbol Crystal_GND24
Connections:
- net +3V3: now also U?.1 (A3V3)
- new net +5V: U?.11 (B5V)
Changed lines of the file:
@@
 LIBS:contrib
 LIBS:valves
+LIBS:custom
 LIBS:ultrasonic_localization-cache
 EELAYER 25 0
@@
 	1    0    0    -1
 $EndComp
+$Comp
+L +3V3 #PWR?
+U 1 1 59F78431
+P 6900 2475
+F 0 "#PWR?" H 6900 2325 50  0001 C CNN
+F 1 "+3V3" H 6900 2615 50  0000 C CNN
+F 2 "" H 6900 2475 50  0001 C CNN
+F 3 "" H 6900 2475 50  0001 C CNN
+	1    6900 2475
+	1    0    0    -1
+$EndComp
+$Comp
+L +5V #PWR?
+U 1 1 59F7844B
+P 8050 2675
+F 0 "#PWR?" H 8050 2525 50  0001 C CNN
+F 1 "+5V" H 8050 2815 50  0000 C CNN
+F 2 "" H 8050 2675 50  0001 C CNN
+F 3 "" H 8050 2675 50  0001 C CNN
+	1    8050 2675
+	1    0    0    -1
+$EndComp
+$Comp
+L LSF0204PWR U?
+U 1 1 59F78590
+P 7475 2975
+F 0 "U?" H 7475 2975 60  0000 C CNN
+F 1 "LSF0204PWR" H 7475 2300 60  0000 C CNN
+F 2 "Housings_SSOP:TSSOP-14_4.4x5mm_Pitch0.65mm" H 7475 2975 60  0001 C CNN
+F 3 "" H 7475 2975 60  0001 C CNN
+	1    7475 2975
+	1    0    0    -1
+$EndComp
+$Comp
+L Crystal_GND24 Y?
+U 1 1 59F78768
+P 2275 3950
+F 0 "Y?" H 2400 4150 50  0000 L CNN
+F 1 "ABM11AIG-20.000MHZ-4Z-T3" H 1725 3650 50  0000 L CNN
+F 2 "Crystals:Crystal_SMD_2016-4pin_2.0x1.6mm" H 2275 3950 50  0001 C CNN
+F 3 "" H 2275 3950 50  0001 C CNN
+	1    2275 3950
+	1    0    0    -1
+$EndComp
+$Comp
+L TCT40-16R/T U?
+U 1 1 59F78BB5
+P 7625 4425
+F 0 "U?" H 7625 4425 60  0000 C CNN
+F 1 "TCT40-16R/T" H 7625 4700 60  0000 C CNN
+F 2 "TCT40-16R_T:TCT40-16R_T" H 7625 4425 60  0001 C CNN
+F 3 "" H 7625 4425 60  0001 C CNN
+	1    7625 4425
+	1    0    0    -1
+$EndComp
+$Comp
+L TCT40-16R/T U?
+U 1 1 59F78C46
+P 7625 4950
+F 0 "U?" H 7625 4950 60  0000 C CNN
+F 1 "TCT40-16R/T" H 7625 5225 60  0000 C CNN
+F 2 "TCT40-16R_T:TCT40-16R_T" H 7625 4950 60  0001 C CNN
+F 3 "" H 7625 4950 60  0001 C CNN
+	1    7625 4950
+	1    0    0    -1
+$EndComp

Commit message: updated oscillator connections
Parts:
- added C? (x2): 10pF, symbol C
Connections:
- net GND: now also Y?.2, Y?.4, C?.2, C?.2
- net at U?.16 (XTAL2): now also Y?.3, C?.1
- net at U?.17 (XTAL1): now also Y?.1, C?.1
Other:
- moved on the sheet: Y?
Changed lines of the file:
@@
 L Crystal_GND24 Y?
 U 1 1 59F78768
-P 2275 3950
-F 0 "Y?" H 2400 4150 50  0000 L CNN
-F 1 "ABM11AIG-20.000MHZ-4Z-T3" H 1725 3650 50  0000 L CNN
-F 2 "Crystals:Crystal_SMD_2016-4pin_2.0x1.6mm" H 2275 3950 50  0001 C CNN
-F 3 "" H 2275 3950 50  0001 C CNN
-	1    2275 3950
-	1    0    0    -1
+P 3150 2325
+F 0 "Y?" V 3000 2375 50  0000 L CNN
+F 1 "ABM11AIG-20.000MHZ-4Z-T3" V 3550 1700 50  0000 L CNN
+F 2 "Crystals:Crystal_SMD_2016-4pin_2.0x1.6mm" H 3150 2325 50  0001 C CNN
+F 3 "" H 3150 2325 50  0001 C CNN
+	1    3150 2325
+	0    1    1    0
 $EndComp
 $Comp
@@
 	1    0    0    -1
 $EndComp
+$Comp
+L GND #PWR?
+U 1 1 59F78D8A
+P 3425 2325
+F 0 "#PWR?" H 3425 2075 50  0001 C CNN
+F 1 "GND" H 3425 2375 50  0000 C CNN
+F 2 "" H 3425 2325 50  0001 C CNN
+F 3 "" H 3425 2325 50  0001 C CNN
+	1    3425 2325
+	1    0    0    -1
+$EndComp
+Wire Wire Line
+	3350 2325 3425 2325
+$Comp
+L GND #PWR?
+U 1 1 59F78F19
+P 2550 2325
+F 0 "#PWR?" H 2550 2075 50  0001 C CNN
+F 1 "GND" H 2550 2175 50  0000 C CNN
+F 2 "" H 2550 2325 50  0001 C CNN
+F 3 "" H 2550 2325 50  0001 C CNN
+	1    2550 2325
+	1    0    0    -1
+$EndComp
+$Comp
+L C C?
+U 1 1 59F78F38
+P 2825 2475
+F 0 "C?" V 2875 2325 50  0000 L CNN
+F 1 "10pF" V 2975 2400 50  0000 L CNN
+F 2 "" H 2863 2325 50  0001 C CNN
+F 3 "" H 2825 2475 50  0001 C CNN
+	1    2825 2475
+	0    1    1    0
+$EndComp
+$Comp
+L C C?
+U 1 1 59F7904A
+P 2825 2175
+F 0 "C?" V 2775 2025 50  0000 L CNN
+F 1 "10pF" V 2675 2100 50  0000 L CNN
+F 2 "" H 2863 2025 50  0001 C CNN
+F 3 "" H 2825 2175 50  0001 C CNN
+	1    2825 2175
+	0    1    1    0
+$EndComp
+Wire Wire Line
+	2975 2475 3575 2475
+Wire Wire Line
+	3575 2475 3575 2400
+Wire Wire Line
+	2975 2175 3575 2175
+Wire Wire Line
+	3575 2175 3575 2200
+Connection ~ 3150 2175
+Connection ~ 3150 2475
+Wire Wire Line
+	2950 2325 2550 2325
+Wire Wire Line
+	2675 2175 2675 2475
+Connection ~ 2675 2325
 $EndSCHEMATC

Commit message: Made a power switching module work
Parts:
- added BT?: Battery_Cell, symbol Battery_Cell
- added C? (x2): 10uF, symbol C
- added C?: 1uF, symbol C
- added D? (x2): LED, symbol LED
- added R?: 10K, symbol R
- added R?: 3.57K, symbol R
- added R?: 2.94K, symbol R
- added R?: 4.32K, symbol R
- added R?: 56.2K, symbol R
- added R? (x2): 1.5K, symbol R
- added U?: BQ2423, MODULE, symbol BQ2423
Connections:
- net +5V: now also C?.1, U?.13 (IN)
- net GND: now also BT?.2 (-), C?.1, C?.2, C?.2, R?.1, R?.2, R?.2, R?.2, R?.2, U?.4 (CE), U?.6 (EN1), U?.8 (VSS)
- new net: R?.2, U?.1 (TS)
- new net: C?.2, R?.1, R?.1, U?.10 (OUT), U?.11 (OUT), U?.5 (EN2)
- new net: R?.1, U?.12 (ILIM)
- new net: R?.1, U?.14 (TMR)
- new net: R?.1, U?.15 (ITERM)
- new net: R?.1, U?.16 (ISET)
- new net: BT?.1 (+), C?.1, U?.2 (BAT), U?.3 (BAT)
- new net: D?.1 (K), U?.7 (PGOOD)
- new net: D?.1 (K), U?.9 (CHG)
- new net: D?.2 (A), R?.2 (x2)

Commit message: adding more cxns
Parts:
- added C? (x2): 1uF, symbol C
- added C?: 10uF, symbol C
- added Cp? (x5): 0.1uF, symbol C
- added R?: 10K, symbol R
- added R? (x2): 22, symbol R
- added SW?: SW_Push, symbol SW_Push
Connections:
- net +3V3: no longer U?.14 (VCC), U?.2 (UVCC), U?.24 (AVCC), U?.34 (VCC), U?.44 (AVCC)
- net +5V: now also U?.14 (VCC), U?.2 (UVCC), U?.24 (AVCC), U?.34 (VCC), U?.44 (AVCC), C?.1, Cp?.1, Cp?.1, Cp?.1, Cp?.1, Cp?.1, R?.2
- net GND: now also J?.5 (GND), J?.6 (Shield), U?.33 ((~HWB~)PE2), C?.1, C?.1, C?.2, Cp?.2, Cp?.2, Cp?.2, Cp?.2, Cp?.2, SW?.1
- net MOSI: now reaches U?.10 ((PDI/MOSI/PCINT2)PB2)
- net MISO: now reaches U?.11 ((PDO/MISO/PCINT3)PB3)
- net at U?.13 (~RESET~): now also R?.1, SW?.2
- net at U?.3 (D-): now also R?.1
- net at U?.4 (D+): now also R?.2
- net at U?.42 (AREF): now also C?.2
- net at U?.6 (UCAP): now also C?.2
- net USB5V: now reaches U?.7 (VBUS)
- net USB5V: now also J?.1 (VBUS)
- net SS: now reaches U?.8 ((SS/PCINT0)PB0)
- net SCK: now reaches U?.9 ((SCLK/PCINT1)PB1)
- net at J?.2 (D-): now also R?.2
- net at J?.3 (D+): now also R?.1
Other:
- note added: "**20MHz exceeds specification,\nneeds ADPS2:0 Division\nAlso, is the crystal necessary?"
- note added: "Bypass Capacitors"
- note added: "Needs 3v7-5V Step Converter for LiPo\nas well as 3V3 regulator"
- moved on the sheet: J?, U?
