File: ultrasonic_localization/ultrasonic_localization.sch (KiCad schematic (older format))
At the start: 19 parts

Commit message: finished ultrasound and some other stuff
Parts:
- added Q?: BUK9Y29-40E, symbol BUK9Y29-40E
- added SW?: SW_SPDT, symbol SW_SPDT
Connections:
- net +26V: now also Q?.1 (S), Q?.2 (S), Q?.3 (S)
- net +5V: now also SW?.3 (C)
- net GND: now also SW?.1 (A)
- net ID: now reaches U?.1 ((INT6/AIN0)PE6)
- net ID: now also SW?.2 (B)
- net SIG2: now reaches U?.22 ((XCK1/~CTS~)PD5)
- net SIG1: now reaches U?.25 ((ICP2/ADC8)PD4)
- net SIG3: now reaches U?.26 ((T1/~OC4D~/ADC9)PD6)
- net SIG4: now reaches U?.27 ((T0/OC4D/ADC10)PD7)
- net OSC: now reaches U?.29 ((ADC12/OC1A/~OC4B~/PCINT12)PB5)
- net OSC: now also Q?.4 (G)
- new net TXa: Q?.5 (D)
- no-connect marks 42 -> 36
Other:
- note added: "40kHz PWM"
- note added: "CHECK DIGITAL SIG"
- note added: "Check CE does what we think it does"
- note added: "IMU somebody"
- moved on the sheet: U?
Changed lines of the file:
@@
 Power & Bypass Capacitors
-$Comp
-L ATMEGA32U4RC-AU U?
-U 1 1 59F4A6C5
-P 3100 3425
-F 0 "U?" H 3100 3450 50  0000 C CNN
-F 1 "ATMEGA32U4RC-AU" H 3800 1925 50  0000 C CNN
-F 2 "TQFP44" H 3100 3425 50  0001 C CIN
-F 3 "" H 4200 4525 50  0001 C CNN
-	1    3100 3425
-	1    0    0    -1
-$EndComp
 $Comp
 L Crystal_GND23 Y?
@@
 L MD0105 U?
 U 1 1 59FAAFC6
-P 10200 1725
-F 0 "U?" H 10200 1625 50  0000 C CNN
-F 1 "MD0105" H 10200 1825 50  0000 C CNN
-F 2 "MODULE" H 10200 1725 50  0001 C CNN
-F 3 "DOCUMENTATION" H 10200 1725 50  0001 C CNN
-	1    10200 1725
+P 10200 2000
+F 0 "U?" H 10200 1900 50  0000 C CNN
+F 1 "MD0105" H 10200 2100 50  0000 C CNN
+F 2 "MODULE" H 10200 2000 50  0001 C CNN
+F 3 "DOCUMENTATION" H 10200 2000 50  0001 C CNN
+	1    10200 2000
 	1    0    0    -1
 $EndComp
@@
 Text Label 8025 1900 2    60   ~ 0
 THRESH
-Text Label 9450 1425 2    60   ~ 0
+Text Label 9450 1700 2    60   ~ 0
 SW1a
-Text Label 9450 1625 2    60   ~ 0
+Text Label 9450 1900 2    60   ~ 0
 SW2a
-Text Label 9450 1825 2    60   ~ 0
+Text Label 9450 2100 2    60   ~ 0
 SW3a
-Text Label 9450 2025 2    60   ~ 0
+Text Label 9450 2300 2    60   ~ 0
 SW4a
-NoConn ~ 9450 1325
-NoConn ~ 9450 1525
-NoConn ~ 9450 1725
-NoConn ~ 9450 1925
-NoConn ~ 9450 2125
-NoConn ~ 10950 2125
-NoConn ~ 10950 1925
-NoConn ~ 10950 1725
-NoConn ~ 10950 1525
-NoConn ~ 10950 1325
-Text Label 10950 1425 0    60   ~ 0
+NoConn ~ 9450 1600
+NoConn ~ 9450 1800
+NoConn ~ 9450 2000
+NoConn ~ 9450 2200
+NoConn ~ 9450 2400
+NoConn ~ 10950 2400
+NoConn ~ 10950 2200
+NoConn ~ 10950 2000
+NoConn ~ 10950 1800
+NoConn ~ 10950 1600
+Text Label 10950 1700 0    60   ~ 0
 SW1b
-Text Label 10950 1625 0    60   ~ 0
+Text Label 10950 1900 0    60   ~ 0
 SW2b
-Text Label 10950 1825 0    60   ~ 0
+Text Label 10950 2100 0    60   ~ 0
 SW3b
-Text Label 10950 2025 0    60   ~ 0
+Text Label 10950 2300 0    60   ~ 0
 SW4b
 Text Label 6800 950  2    60   ~ 0
@@
 Ultrasonic Transceivers
 NoConn ~ 4200 2275
-NoConn ~ 4200 2375
 NoConn ~ 4200 2475
 NoConn ~ 4200 2575
 NoConn ~ 4200 2775
 NoConn ~ 4200 2875
-NoConn ~ 4200 3075
 NoConn ~ 4200 3175
 NoConn ~ 4200 3275
 NoConn ~ 4200 3375
-NoConn ~ 4200 3475
-NoConn ~ 4200 3575
-NoConn ~ 4200 3675
-NoConn ~ 4200 3775
-NoConn ~ 4200 4075
-NoConn ~ 4200 4275
-NoConn ~ 4200 4375
-NoConn ~ 4200 4475
-NoConn ~ 4200 4575
 NoConn ~ 4200 4675
 NoConn ~ 4200 4775
@@
 Text Notes 1375 6150 0    60   ~ 0
 ID of module\n
+$Comp
+L SW_SPDT SW?
+U 1 1 59FCFB66
+P 1675 6450
+F 0 "SW?" H 1675 6620 50  0000 C CNN
+F 1 "SW_SPDT" H 1675 6250 50  0000 C CNN
+F 2 "" H 1675 6450 50  0001 C CNN
+F 3 "" H 1675 6450 50  0001 C CNN
+	1    1675 6450
+	-1   0    0    1
+$EndComp
+$Comp
+L GND #PWR?
+U 1 1 59FD074D
+P 1475 6550
+F 0 "#PWR?" H 1475 6300 50  0001 C CNN
+F 1 "GND" H 1475 6400 50  0000 C CNN
+F 2 "" H 1475 6550 50  0001 C CNN
+F 3 "" H 1475 6550 50  0001 C CNN
+	1    1475 6550
+	1    0    0    -1
+$EndComp
+$Comp
+L +5V #PWR?
+U 1 1 59FD0DEE
+P 1475 6350
+F 0 "#PWR?" H 1475 6200 50  0001 C CNN
+F 1 "+5V" H 1475 6490 50  0000 C CNN
+F 2 "" H 1475 6350 50  0001 C CNN
+F 3 "" H 1475 6350 50  0001 C CNN
+	1    1475 6350
+	1    0    0    -1
+$EndComp
+Text Label 1875 6450 0    60   ~ 0
+ID
+$Comp
+L BUK9Y29-40E Q?
+U 1 1 59FD4416
+P 10300 800
+F 0 "Q?" H 10500 850 50  0000 L CNN
+F 1 "BUK9Y29-40E" H 10500 750 50  0000 L CNN
+F 2 "" H 10500 900 50  0001 C CNN
+F 3 "" H 10300 800 50  0001 C CNN
+	1    10300 800
+	1    0    0    -1
+$EndComp
+Text Label 10400 625  0    60   ~ 0
+TXa
+Text Label 10100 800  2    60   ~ 0
+OSC
+Text Label 10375 1000 3    60   ~ 0
++26V
+Wire Wire Line
+	10350 1000 10400 1000
+Connection ~ 10375 1000
+Text Label 6800 1200 2    60   ~ 0
+TXa
+Text Label 8025 1200 2    60   ~ 0
+TXa
+Text Label 8025 2275 2    60   ~ 0
+TXa
+Text Label 6800 2275 2    60   ~ 0
+TXa
+$Comp
+L GND #PWR?
+U 1 1 59FD82C0
+P 6700 1325
+F 0 "#PWR?" H 6700 1075 50  0001 C CNN
+F 1 "GND" H 6700 1175 50  0000 C CNN
+F 2 "" H 6700 1325 50  0001 C CNN
+F 3 "" H 6700 1325 50  0001 C CNN
+	1    6700 1325
+	1    0    0    -1
+$EndComp
+Wire Wire Line
+	6700 1325 6800 1325
+$Comp
+L GND #PWR?
+U 1 1 59FD880A
+P 7925 1325
+F 0 "#PWR?" H 7925 1075 50  0001 C CNN
+F 1 "GND" H 7925 1175 50  0000 C CNN
+F 2 "" H 7925 1325 50  0001 C CNN
+F 3 "" H 7925 1325 50  0001 C CNN
+	1    7925 1325
+	1    0    0    -1
+$EndComp
+Wire Wire Line
+	7925 1325 8025 1325
+$Comp
+L GND #PWR?
+U 1 1 59FD8AC0
+P 6675 2400
+F 0 "#PWR?" H 6675 2150 50  0001 C CNN
+F 1 "GND" H 6675 2250 50  0000 C CNN
+F 2 "" H 6675 2400 50  0001 C CNN
+F 3 "" H 6675 2400 50  0001 C CNN
+	1    6675 2400
+	1    0    0    -1
+$EndComp
+Wire Wire Line
+	6675 2400 6800 2400
+$Comp
+L GND #PWR?
+U 1 1 59FD8E67
+P 7925 2400
+F 0 "#PWR?" H 7925 2150 50  0001 C CNN
+F 1 "GND" H 7925 2250 50  0000 C CNN
+F 2 "" H 7925 2400 50  0001 C CNN
+F 3 "" H 7925 2400 50  0001 C CNN
+	1    7925 2400
+	1    0    0    -1
+$EndComp
+Wire Wire Line
+	7925 2400 8025 2400
+Text Label 7425 1075 0    60   ~ 0
+SIG1
+Text Label 8650 1075 0    60   ~ 0
+SIG2
+Text Label 7425 2150 0    60   ~ 0
+SIG3
+Text Label 8650 2150 0    60   ~ 0
+SIG4
+$Comp
+L ATMEGA32U4RC-AU U?
+U 1 1 59F4A6C5
+P 3100 3425
+F 0 "U?" H 3100 3450 50  0000 C CNN
+F 1 "ATMEGA32U4RC-AU" H 3800 1925 50  0000 C CNN
+F 2 "TQFP44" H 3100 3425 50  0001 C CIN
+F 3 "" H 4200 4525 50  0001 C CNN
+	1    3100 3425
+	1    0    0    -1
+$EndComp
+Text Label 4200 3475 0    60   ~ 0
+SIG1
+Text Label 4200 3575 0    60   ~ 0
+SIG2
+Text Label 4200 3675 0    60   ~ 0
+SIG3
+Text Label 4200 3775 0    60   ~ 0
+SIG4
+Text Label 4200 2375 0    60   ~ 0
+OSC
+Text Notes 4425 2350 0    60   ~ 0
+40kHz PWM
+Text Notes 4450 3625 0    60   ~ 0
+CHECK DIGITAL SIG
+NoConn ~ 4200 4275
+NoConn ~ 4200 4375
+NoConn ~ 4200 4475
+NoConn ~ 4200 4575
+NoConn ~ 4200 3075
+Text Label 4200 4075 0    60   ~ 0
+ID
+Text Label 8000 3400 2    60   ~ 0
+SS
+Text Label 8000 3600 2    60   ~ 0
+SCK
+Text Label 8000 3800 2    60   ~ 0
+MOSI
+Text Label 8000 3975 2    60   ~ 0
+MISO
+$Comp
+L +5V #PWR?
+U 1 1 59FE2F7E
+P 7900 4150
+F 0 "#PWR?" H 7900 4000 50  0001 C CNN
+F 1 "+5V" H 7900 4290 50  0000 C CNN
+F 2 "" H 7900 4150 50  0001 C CNN
+F 3 "" H 7900 4150 50  0001 C CNN
+	1    7900 4150
+	1    0    0    -1
+$EndComp
+Wire Wire Line
+	8000 4150 7900 4150
+Text Notes 7775 4175 2    60   ~ 0
+Check CE does what we think it does
+Wire Notes Line
+	11200 4600 6975 4600
+Wire Notes Line
+	6975 4600 6975 6500
+Wire Notes Line
+	6975 6500 11200 6500
+Wire Notes Line
+	11200 6500 11200 4600
+Text Notes 8950 4775 0    60   ~ 0
+IMU somebody
 $EndSCHEMATC

Commit message: added osc src
Parts:
- added C?: 10nF, symbol C
- added D?: LED, symbol LED
- added R?: 9.53K, symbol R
- added R? (x3): 10K, symbol R
- added R?: 604, symbol R
- added SW?: SW_SPDT, symbol SW_SPDT
- added U?: 4047, symbol 4047
Connections:
- net +5V: now also U?.14 (VDD), U?.4 (~ASTABLE), U?.5 (ASTABLE), U?.6 (-TRIGGER)
- net GND: now also D?.1 (K), R?.2, R?.2, U?.12 (RETRIGGER), U?.7 (VSS), U?.8 (+TRIGGER); no longer SW?.1 (A)
- net ID: now also R?.1
- net TX_EN: now reaches U?.30 ((ADC13/OC1B/OC4B/PCINT13)PB6)
- net TX_EN: now also U?.9 (EXT_RESET)
- net OSC: no longer names the net of Q?.4 (G)
- net OSC: now also SW?.2 (B); no longer U?.29 ((ADC12/OC1A/~OC4B~/PCINT12)PB5)
- new net: C?.1, U?.1 (C)
- new net: R?.2, R?.2, U?.2 (R)
- new net: C?.2, R?.1, R?.1, U?.3 (RC_COMMON)
- new net: D?.2 (A), R?.2
- new net OSC_IC: R?.1, SW?.1 (A), U?.13 (OSC_OUT)
- new net OSC_MCU: SW?.3 (C), U?.29 ((ADC12/OC1A/~OC4B~/PCINT12)PB5)
- no-connect marks 36 -> 37
Other:
- note added: "40kHz SQW"
- note added: "Module ID"
- note added: "TODO : CHECK DIGITAL SIG\n& Pin Assignments"
- note added: "TODO : Check CE does what we think it does"
- note added: "TODO : NEEDED?"
- note removed: "40kHz PWM"
- note removed: "CHECK DIGITAL SIG"
- note removed: "Check CE does what we think it does"
- note removed: "ID of module\n"
- note removed: "NEEDED?"
- moved on the sheet: Q?, SW?, U?

Commit message: Added IMU
Parts:
- removed U?: LSF0204PWR, Housings_SSOP:TSSOP-14_4.4x5mm_Pitch0.65mm, symbol LSF0204PWR
- added C?: 100nF, symbol C
- added R? (x7): 10K, symbol R
- added U?: IMU, symbol IMU
- added U?: Level_Shifter_4Channel, symbol Level_Shifter_4Channel
Connections:
- net +5V: now also R?.2, R?.2, R?.2, R?.2, U?.11 (Vref_B), U?.12 (EN)
- net GND: now also C?.2, U?.2 (SDx), U?.3 (SCx), U?.6 (GND), U?.6 (GND), U?.7 (GND)
- net SCL: now reaches U?.18 ((OC0B/SCL/INT0)PD0)
- net SCL: now also R?.1, U?.10 (B1)
- net SDA: now reaches U?.19 ((SDA/INT1)PD1)
- net SDA: now also R?.1, U?.9 (B2)
- net D2: now reaches U?.20 ((RXD/INT2)PD2)
- net D2: now also R?.1, U?.8 (B3)
- net D3: now reaches U?.21 ((TXD/INT3)PD3)
- net D3: now also R?.1, U?.7 (B4)
- new net: R?.1, U?.12 (CS)
- new net +1V8: C?.1, R?.2, R?.2, R?.2, U?.1 (Vref_A), U?.5 (VDDIO), U?.8 (VDD)
- new net INT1: U?.4 (INT1), U?.5 (A4)
- new net INT2: U?.4 (A3), U?.9 (INT2)
- new net L_HI: U?.1 (SDO/SA0)
- new net SCL_1V8: R?.1, U?.13 (SCL), U?.3 (A2)
- new net SDA_1V8: R?.1, U?.14 (SDA), U?.2 (A1)
- no-connect marks 37 -> 25

Commit message: Added ICSP header
Parts:
- removed C?: 100nF, symbol C
- removed R? (x7): 10K, symbol R
- removed U?: IMU, symbol IMU
- removed U?: Level_Shifter_4Channel, symbol Level_Shifter_4Channel
- added C?: 10uF, symbol C
- added J?: CONN_02X03, symbol CONN_02X03
Connections:
- net +26V: now also C?.1
- net +5V: now also J?.2 (P2)
- net GND: now also SW?.1 (A), C?.2, J?.6 (P6)
- net MISO: now also J?.1 (P1)
- net MOSI: now also J?.4 (P4)
- net SCK: now also J?.3 (P3)
- net RESET: now reaches R?.1, SW?.2, U?.13 (~RESET~)
- net RESET: now also J?.5 (P5)
- net RF_CE: now reaches U?.41 ((ADC0)PF0)
- no-connect marks 25 -> 22
Other:
- note added: "ICSP HEADER"
- note added: "IMU Module"
- note added: "RF Module"
- note removed: "IMU somebody"
- note removed: "LEVEL SHIFTER, IF NEEDED\n( FOR IMU )"
- note removed: "TODO : Check CE does what we think it does"
- moved on the sheet: R?, SW?
