File: ultrasonic_localization/ultrasonic_localization.sch (KiCad schematic (older format))
At the start: 29 parts, among them J1 USB_OTG, Q1 BUK9Y29-40E, SW1 SW_Push, SW2 SW_SPDT, SW3 SW_SPDT, U1 ATMEGA32U4RC-AU, U3 MD0105, U5 4047, Y1 16MHz

Commit message: pushing stuff
Parts:
- added J?: Conn_02x03_Odd_Even, symbol Conn_02x03_Odd_Even
Connections:
- wire segments 78 -> 79
Other:
- note added: "ICSP HEADER"
- note removed: "TODO : ICSP HEADER"
- moved on the sheet: C2, C3, C4, C5, R1, R2, R3, R5, SW1, SW2, U1, Y1

Commit message: meh
Other:
- note removed: "TODO : Check CE does what we think it does"
Changed lines of the file:
@@
 Text Label 6550 5675 2    60   ~ 0
 MISO
-Text Notes 8375 6225 2    60   ~ 0
-TODO : Check CE does what we think it does
 $Comp
 L 4047 U5

Commit message: IMU pulldown
Connections:
- wire segments 79 -> 49
Other:
- note removed: "TODO : CHECK ANALOG/DIGITAL THRESH"
Changed lines of the file:
@@
 Connection ~ 9225 2650
 Wire Wire Line
-	8975 2650 9125 2650
-Wire Wire Line
-	9125 2650 9225 2650
+	8975 2650 9225 2650
 Wire Wire Line
 	9225 2950 8875 2950
@@
 Connection ~ 8800 3550
 Wire Wire Line
-	9225 2550 9225 2650
-Wire Wire Line
-	9225 2650 9225 2750
+	9225 2550 9225 2750
 Wire Wire Line
 	9050 3250 9225 3250
 Wire Wire Line
-	8600 3150 8800 3150
-Wire Wire Line
-	8800 3150 9225 3150
+	8600 3150 9225 3150
 Wire Wire Line
 	8800 3250 8800 3150
@@
 	9225 3250 9225 3350
 Wire Wire Line
-	8600 3550 8800 3550
-Wire Wire Line
-	8800 3550 9050 3550
-Wire Wire Line
-	9050 3550 9225 3550
+	8600 3550 9225 3550
 Connection ~ 9225 2250
 Wire Wire Line
 	9925 1850 9225 1850
 Wire Wire Line
-	9225 1850 9225 2150
-Wire Wire Line
-	9225 2150 9225 2250
-Wire Wire Line
-	9225 2250 9225 2450
+	9225 1850 9225 2450
 Wire Wire Line
 	9975 1275 10075 1275
@@
 Connection ~ 1075 4300
 Wire Wire Line
-	700  3875 700  4175
-Wire Wire Line
-	700  4175 700  4300
+	700  3875 700  4300
 Connection ~ 1275 4175
 Connection ~ 1275 3875
@@
 	1475 4300 1475 4025
 Wire Wire Line
-	700  4300 1075 4300
-Wire Wire Line
-	1075 4300 1275 4300
-Wire Wire Line
-	1275 4300 1475 4300
+	700  4300 1475 4300
 Wire Wire Line
 	1075 4025 1075 4300
 Wire Wire Line
-	1000 4175 1275 4175
-Wire Wire Line
-	1275 4175 1950 4175
+	1000 4175 1950 4175
 Wire Wire Line
 	1950 4175 1950 4125
 Wire Wire Line
-	1000 3875 1275 3875
-Wire Wire Line
-	1275 3875 1950 3875
+	1000 3875 1950 3875
 Wire Wire Line
 	1950 3875 1950 3925
@@
 Connection ~ 3250 3275
 Wire Wire Line
-	2650 3275 2900 3275
-Wire Wire Line
-	2900 3275 3000 3275
-Wire Wire Line
-	3000 3275 3125 3275
-Wire Wire Line
-	3125 3275 3250 3275
-Wire Wire Line
-	3250 3275 3350 3275
+	2650 3275 3350 3275
 Connection ~ 1000 725
 Connection ~ 1000 1025
@@
 Connection ~ 1225 1025
 Wire Wire Line
-	750  1025 1000 1025
-Wire Wire Line
-	1000 1025 1225 1025
-Wire Wire Line
-	1225 1025 1450 1025
-Wire Wire Line
-	1450 1025 1675 1025
-Wire Wire Line
-	1675 1025 1900 1025
-Wire Wire Line
-	1900 1025 2125 1025
+	750  1025 2125 1025
 Connection ~ 1675 725
 Connection ~ 1450 725
 Connection ~ 1225 725
 Wire Wire Line
-	750  725  1000 725
-Wire Wire Line
-	1000 725  1225 725
-Wire Wire Line
-	1225 725  1450 725
-Wire Wire Line
-	1450 725  1675 725
-Wire Wire Line
-	1675 725  1900 725
+	750  725  1900 725
 Wire Wire Line
 	4200 5625 4450 5625
@@
 Connection ~ 2825 6675
 Wire Wire Line
-	2700 6675 2825 6675
-Wire Wire Line
-	2825 6675 2950 6675
-Wire Wire Line
-	2950 6675 3050 6675
-Wire Wire Line
-	3050 6675 3150 6675
-Wire Wire Line
-	3150 6675 3250 6675
+	2700 6675 3250 6675
 Text Label 6625 7000 0    60   ~ 0
 ID
 Wire Wire Line
-	1950 3275 1950 3525
-Wire Wire Line
-	1950 3525 1950 3725
+	1950 3275 1950 3725
 Text Label 4200 4225 0    60   ~ 0
 THRESH
-Text Notes 2300 7200 0    60   ~ 0
-TODO : CHECK ANALOG/DIGITAL THRESH
 $Comp
 L Conn_02x03_Odd_Even J?

Commit message: Assigned many footprints to things
Parts:
- Q1: footprint (none) -> TO_SOT_Packages_SMD:SOT-669_LFPAK
- U1: footprint TQFP44 -> Housings_QFP:TQFP-44-1EP_10x10mm_Pitch0.8mm
- U3: footprint MODULE -> Custom:DFN-18-1EP_5x5mm_Pitch0.5mm
- U5: footprint (none) -> Housings_SOIC:SOIC-14_3.9x8.7mm_Pitch1.27mm
Changed lines of the file:
@@
 F 0 "U3" H 7275 3075 50  0000 C CNN
 F 1 "MD0105" H 7275 3275 50  0000 C CNN
-F 2 "MODULE" H 7275 3175 50  0001 C CNN
+F 2 "Custom:DFN-18-1EP_5x5mm_Pitch0.5mm" H 7275 3175 50  0001 C CNN
 F 3 "DOCUMENTATION" H 7275 3175 50  0001 C CNN
 	1    7275 3175
@@
 F 0 "Q1" H 7775 1850 50  0000 L CNN
 F 1 "BUK9Y29-40E" H 7400 1500 50  0000 L CNN
-F 2 "" H 7775 1900 50  0001 C CNN
+F 2 "TO_SOT_Packages_SMD:SOT-669_LFPAK" H 7775 1900 50  0001 C CNN
 F 3 "" H 7575 1800 50  0001 C CNN
 	1    7575 1800
@@
 F 0 "U1" H 3100 5100 50  0000 C CNN
 F 1 "ATMEGA32U4RC-AU" H 3800 3575 50  0000 C CNN
-F 2 "TQFP44" H 3100 5075 50  0001 C CIN
+F 2 "Housings_QFP:TQFP-44-1EP_10x10mm_Pitch0.8mm" H 3100 5075 50  0001 C CIN
 F 3 "" H 4200 6175 50  0001 C CNN
 	1    3100 5075
@@
 F 0 "U5" H 9425 3750 50  0000 C CNN
 F 1 "4047" H 10375 1950 50  0000 C CNN
-F 2 "" H 9325 3650 50  0001 C CNN
+F 2 "Housings_SOIC:SOIC-14_3.9x8.7mm_Pitch1.27mm" H 9325 3650 50  0001 C CNN
 F 3 "" H 9425 3750 50  0001 C CNN
 	1    9925 2850

Commit message: almost resolved DRC
Parts:
- removed J1: USB_OTG, symbol USB_OTG
- added J1: USB_OTG_fix, symbol USB_OTG_fix
- gave numbers to parts that had none: 1
Connections:
- net labels added: IRQ
- no-connect marks 21 -> 20
Other:
- note removed: "TODO : NEEDED?"
Changed lines of the file:
@@
 $EndComp
 $Sheet
-S 6550 4825 1800 1150
+S 6550 4825 550  1025
 U 59FC41DC
 F0 "RF Module" 60
 F1 "rfModule.sch" 60
-F2 "CSN" I L 6550 5100 60
-F3 "SCK" I L 6550 5300 60
-F4 "MOSI" I L 6550 5500 60
-F5 "MISO" I L 6550 5675 60
-F6 "CE" I L 6550 5850 60
+F2 "CSN" I L 6550 4975 60
+F3 "SCK" I L 6550 5125 60
+F4 "MOSI" I L 6550 5275 60
+F5 "MISO" I L 6550 5400 60
+F6 "CE" I L 6550 5550 60
+F7 "IRQ" I L 6550 5700 60
 $EndSheet
 $Comp
@@
 Text Notes 3725 1325 0    60   ~ 0
 (encloses BAT)
-$Comp
-L USB_OTG J1
-U 1 1 59FC9F9F
-P 1200 4925
-F 0 "J1" H 1000 5375 50  0000 L CNN
-F 1 "USB_OTG" H 1000 5275 50  0000 L CNN
-F 2 "" H 1350 4875 50  0001 C CNN
-F 3 "" H 1350 4875 50  0001 C CNN
-	1    1200 4925
-	1    0    0    -1
-$EndComp
-Text Notes 1325 4575 0    60   ~ 0
-TODO : NEEDED?
 Text Label 4200 600  0    60   ~ 0
 +26V
@@
 Text Notes 4450 5275 0    60   ~ 0
 TODO : CHECK DIGITAL SIG\n& Pin Assignments
-NoConn ~ 4200 6025
 NoConn ~ 4200 6125
 NoConn ~ 4200 6225
 Text Label 4200 5725 0    60   ~ 0
 ID
-Text Label 6550 5100 2    60   ~ 0
+Text Label 6550 4975 2    60   ~ 0
 SS
-Text Label 6550 5300 2    60   ~ 0
+Text Label 6550 5125 2    60   ~ 0
 SCK
-Text Label 6550 5500 2    60   ~ 0
+Text Label 6550 5275 2    60   ~ 0
 MOSI
-Text Label 6550 5675 2    60   ~ 0
+Text Label 6550 5400 2    60   ~ 0
 MISO
 $Comp
@@
 $EndComp
 $Comp
-L GND #PWR019
+L GND #PWR018
 U 1 1 5A0021A9
 P 9925 3850
-F 0 "#PWR019" H 9925 3600 50  0001 C CNN
+F 0 "#PWR018" H 9925 3600 50  0001 C CNN
 F 1 "GND" H 9925 3700 50  0000 C CNN
 F 2 "" H 9925 3850 50  0001 C CNN
@@
 $EndComp
 $Comp
-L +5V #PWR020
+L +5V #PWR019
 U 1 1 5A0026FD
 P 9925 1850
-F 0 "#PWR020" H 9925 1700 50  0001 C CNN
+F 0 "#PWR019" H 9925 1700 50  0001 C CNN
 F 1 "+5V" H 9925 1990 50  0000 C CNN
 F 2 "" H 9925 1850 50  0001 C CNN
@@
 $EndComp
 $Comp
-L GND #PWR021
+L GND #PWR020
 U 1 1 5A005A93
 P 9125 2750
-F 0 "#PWR021" H 9125 2500 50  0001 C CNN
+F 0 "#PWR020" H 9125 2500 50  0001 C CNN
 F 1 "GND" H 9125 2600 50  0000 C CNN
 F 2 "" H 9125 2750 50  0001 C CNN
@@
 $EndComp
 $Comp
-L GND #PWR022
+L GND #PWR021
 U 1 1 5A013A28
 P 10750 2750
-F 0 "#PWR022" H 10750 2500 50  0001 C CNN
+F 0 "#PWR021" H 10750 2500 50  0001 C CNN
 F 1 "GND" H 10750 2600 50  0000 C CNN
 F 2 "" H 10750 2750 50  0001 C CNN
@@
 	-1   0    0    1
 $EndComp
-Text Label 8875 2950 2    60   ~ 0
+Text Label 8825 2950 2    60   ~ 0
 TX_EN
 $Comp
@@
 $EndComp
 $Comp
-L GND #PWR023
+L GND #PWR022
 U 1 1 5A04AAA6
 P 6625 7300
-F 0 "#PWR023" H 6625 7050 50  0001 C CNN
+F 0 "#PWR022" H 6625 7050 50  0001 C CNN
 F 1 "GND" H 6625 7150 50  0000 C CNN
 F 2 "" H 6625 7300 50  0001 C CNN
@@
 ICSP HEADER
 $Comp
-L +1V8 #PWR027
+L +1V8 #PWR023
 U 1 1 5A07E30F
 P 4500 1150
-F 0 "#PWR027" H 4500 1000 50  0001 C CNN
+F 0 "#PWR023" H 4500 1000 50  0001 C CNN
 F 1 "+1V8" H 4500 1290 50  0000 C CNN
 F 2 "" H 4500 1150 50  0001 C CNN
@@
 Text Label 4200 5025 0    60   ~ 0
 D3
-Text Label 6550 5850 2    60   ~ 0
+Text Label 6550 5550 2    60   ~ 0
 RF_CE
 Wire Wire Line
@@
 	8975 2650 9225 2650
 Wire Wire Line
-	9225 2950 8875 2950
+	8825 2950 9225 2950
 Connection ~ 9225 2150
 Connection ~ 8800 3150
@@
 Wire Notes Line
 	4775 500  4775 1400
-Connection ~ 2900 3275
-Connection ~ 3000 3275
-Connection ~ 3125 3275
-Connection ~ 3250 3275
-Wire Wire Line
-	2650 3275 3350 3275
 Connection ~ 1000 725
 Connection ~ 1000 1025
@@
 THRESH
 $Comp
-L Conn_02x03_Odd_Even J?
+L Conn_02x03_Odd_Even J2
 U 1 1 5A01AC29
 P 5400 1150
-F 0 "J?" H 5450 1350 50  0000 C CNN
+F 0 "J2" H 5450 1350 50  0000 C CNN
 F 1 "Conn_02x03_Odd_Even" H 5450 800 50  0000 C CNN
 F 2 "" H 5400 1150 50  0001 C CNN
@@
 Connection ~ 1950 3525
 $Comp
-L +5V #PWR?
+L +5V #PWR024
 U 1 1 5A01C4EA
 P 5700 1050
-F 0 "#PWR?" H 5700 900 50  0001 C CNN
+F 0 "#PWR024" H 5700 900 50  0001 C CNN
 F 1 "+5V" H 5700 1190 50  0000 C CNN
 F 2 "" H 5700 1050 50  0001 C CNN
@@
 MOSI
 $Comp
-L GND #PWR?
+L GND #PWR025
 U 1 1 5A01C829
 P 5700 1250
-F 0 "#PWR?" H 5700 1000 50  0001 C CNN
+F 0 "#PWR025" H 5700 1000 50  0001 C CNN
 F 1 "GND" H 5700 1100 50  0000 C CNN
 F 2 "" H 5700 1250 50  0001 C CNN
@@
 Wire Notes Line
 	5925 1600 5925 550
+Connection ~ 8975 2950
+$Comp
+L USB_OTG_fix J1
+U 1 1 5A04DC98
+P 1200 4925
+F 0 "J1" H 1000 5375 50  0000 L CNN
+F 1 "USB_OTG_fix" H 1000 5275 50  0000 L CNN
+F 2 "" H 1350 4875 50  0001 C CNN
+F 3 "" H 1350 4875 50  0001 C CNN
+	1    1200 4925
+	1    0    0    -1
+$EndComp
+Text Label 6550 5700 2    60   ~ 0
+IRQ
+Text Label 4200 6025 0    60   ~ 0
+IRQ
+Wire Wire Line
+	2650 3275 3350 3275
+Connection ~ 3250 3275
+Connection ~ 3125 3275
+Connection ~ 3000 3275
+Connection ~ 2900 3275
 $EndSCHEMATC

Commit message: Assigned footprints to menial components
Parts:
- C1: footprint (none) -> Capacitors_SMD:C_0805
- C2, C3, C4, C5, C7, Cp1, Cp2, Cp3, Cp4, Cp5: footprint (none) -> Capacitors_SMD:C_0603
- D1: footprint (none) -> LEDs:LED_0805
- J2: footprint (none) -> Socket_Strips:Socket_Strip_Straight_2x03_Pitch2.54mm
- R1, R10, R15, R2, R3, R5, R8, R9: footprint (none) -> Resistors_SMD:R_0603
- SW1: footprint (none) -> Buttons_Switches_SMD:SW_SPST_B3S-1000
- Y1: footprint (none) -> Crystals:Crystal_SMD_3225-4pin_3.2x2.5mm
Changed lines of the file:
@@
 F 0 "C4" V 1850 4975 50  0000 L CNN
 F 1 "1uF" V 1675 5050 50  0000 L CNN
-F 2 "" H 1838 4975 50  0001 C CNN
+F 2 "Capacitors_SMD:C_0603" H 1838 4975 50  0001 C CNN
 F 3 "" H 1800 5125 50  0001 C CNN
 	1    1800 5125
@@
 F 0 "C5" V 1850 5775 50  0000 L CNN
 F 1 "1uF" V 1950 5850 50  0000 L CNN
-F 2 "" H 1838 5775 50  0001 C CNN
+F 2 "Capacitors_SMD:C_0603" H 1838 5775 50  0001 C CNN
 F 3 "" H 1800 5925 50  0001 C CNN
 	1    1800 5925
@@
 F 0 "R3" V 1700 3325 50  0000 C CNN
 F 1 "10K" V 1800 3275 50  0000 C CNN
-F 2 "" V 1730 3275 50  0001 C CNN
+F 2 "Resistors_SMD:R_0603" V 1730 3275 50  0001 C CNN
 F 3 "" H 1800 3275 50  0001 C CNN
 	1    1800 3275
@@
 F 0 "R2" V 1800 4925 50  0000 C CNN
 F 1 "22" V 1725 4975 50  0000 C CNN
-F 2 "" V 1655 4975 50  0001 C CNN
+F 2 "Resistors_SMD:R_0603" V 1655 4975 50  0001 C CNN
 F 3 "" H 1725 4975 50  0001 C CNN
 	1    1725 4975
@@
 F 0 "R1" V 1800 4925 50  0000 C CNN
 F 1 "22" V 1725 4875 50  0000 C CNN
-F 2 "" V 1655 4875 50  0001 C CNN
+F 2 "Resistors_SMD:R_0603" V 1655 4875 50  0001 C CNN
 F 3 "" H 1725 4875 50  0001 C CNN
 	1    1725 4875
@@
 F 0 "SW1" H 1525 3625 50  0000 L CNN
 F 1 "SW_Push" H 1750 3465 50  0000 C CNN
-F 2 "" H 1750 3725 50  0001 C CNN
+F 2 "Buttons_Switches_SMD:SW_SPST_B3S-1000" H 1750 3725 50  0001 C CNN
 F 3 "" H 1750 3725 50  0001 C CNN
 	1    1750 3525
@@
 F 0 "Cp1" H 1025 975 50  0000 L CNN
 F 1 "0.1uF" H 925 650 50  0000 L CNN
-F 2 "" H 1038 725 50  0001 C CNN
+F 2 "Capacitors_SMD:C_0603" H 1038 725 50  0001 C CNN
 F 3 "" H 1000 875 50  0001 C CNN
 	1    1000 875
@@
 F 0 "Cp2" H 1250 975 50  0000 L CNN
 F 1 "0.1uF" H 1150 650 50  0000 L CNN
-F 2 "" H 1263 725 50  0001 C CNN
+F 2 "Capacitors_SMD:C_0603" H 1263 725 50  0001 C CNN
 F 3 "" H 1225 875 50  0001 C CNN
 	1    1225 875
@@
 F 0 "Cp3" H 1475 975 50  0000 L CNN
 F 1 "0.1uF" H 1375 650 50  0000 L CNN
-F 2 "" H 1488 725 50  0001 C CNN
+F 2 "Capacitors_SMD:C_0603" H 1488 725 50  0001 C CNN
 F 3 "" H 1450 875 50  0001 C CNN
 	1    1450 875
@@
 F 0 "Cp4" H 1700 975 50  0000 L CNN
 F 1 "0.1uF" H 1600 650 50  0000 L CNN
-F 2 "" H 1713 725 50  0001 C CNN
+F 2 "Capacitors_SMD:C_0603" H 1713 725 50  0001 C CNN
 F 3 "" H 1675 875 50  0001 C CNN
 	1    1675 875
@@
 F 0 "Cp5" H 1925 975 50  0000 L CNN
 F 1 "0.1uF" H 1825 650 50  0000 L CNN
-F 2 "" H 1938 725 50  0001 C CNN
+F 2 "Capacitors_SMD:C_0603" H 1938 725 50  0001 C CNN
 F 3 "" H 1900 875 50  0001 C CNN
 	1    1900 875
@@
 F 0 "C1" H 775 975 50  0000 L CNN
 F 1 "10uF" H 675 650 50  0000 L CNN
-F 2 "" H 788 725 50  0001 C CNN
+F 2 "Capacitors_SMD:C_0805" H 788 725 50  0001 C CNN
 F 3 "" H 750 875 50  0001 C CNN
 	1    750  875
@@
 F 0 "Y1" V 1275 4000 50  0000 L CNN
 F 1 "16MHz" V 1075 3900 50  0000 L CNN
-F 2 "" H 1275 4025 50  0001 C CNN
+F 2 "Crystals:Crystal_SMD_3225-4pin_3.2x2.5mm" H 1275 4025 50  0001 C CNN
 F 3 "" H 1275 4025 50  0001 C CNN
 	1    1275 4025
@@
 F 0 "C2" H 875 3975 50  0000 L CNN
 F 1 "12pF" H 875 3775 50  0000 L CNN
-F 2 "" H 888 3725 50  0001 C CNN
+F 2 "Capacitors_SMD:C_0603" H 888 3725 50  0001 C CNN
 F 3 "" H 850 3875 50  0001 C CNN
 	1    850  3875
@@
 F 0 "C3" H 875 4275 50  0000 L CNN
 F 1 "12pF" H 875 4075 50  0000 L CNN
-F 2 "" H 888 4025 50  0001 C CNN
+F 2 "Capacitors_SMD:C_0603" H 888 4025 50  0001 C CNN
 F 3 "" H 850 4175 50  0001 C CNN
 	1    850  4175
@@
 F 0 "R9" V 8900 3400 50  0000 C CNN
 F 1 "9.53K" V 8800 3400 50  0000 C CNN
-F 2 "" V 8730 3400 50  0001 C CNN
+F 2 "Resistors_SMD:R_0603" V 8730 3400 50  0001 C CNN
 F 3 "" H 8800 3400 50  0001 C CNN
 	1    8800 3400
@@
 F 0 "C7" V 9175 3350 50  0000 L CNN
 F 1 "10nF" V 8925 3325 50  0000 L CNN
-F 2 "" H 9088 3250 50  0001 C CNN
+F 2 "Capacitors_SMD:C_0603" H 9088 3250 50  0001 C CNN
 F 3 "" H 9050 3400 50  0001 C CNN
 	1    9050 3400
@@
 F 0 "D1" H 10750 2425 50  0000 C CNN
 F 1 "LED" H 10750 2500 50  0000 C CNN
-F 2 "" H 10750 2600 50  0001 C CNN
+F 2 "LEDs:LED_0805" H 10750 2600 50  0001 C CNN
 F 3 "" H 10750 2600 50  0001 C CNN
 	1    10750 2600
@@
 F 0 "R15" V 10850 2300 50  0000 C CNN
 F 1 "10K" V 10750 2300 50  0000 C CNN
-F 2 "" V 10680 2300 50  0001 C CNN
+F 2 "Resistors_SMD:R_0603" V 10680 2300 50  0001 C CNN
 F 3 "" H 10750 2300 50  0001 C CNN
 	1    10750 2300
@@
 F 0 "R8" V 8700 3400 50  0000 C CNN
 F 1 "604" V 8600 3400 50  0000 C CNN
-F 2 "" V 8530 3400 50  0001 C CNN
+F 2 "Resistors_SMD:R_0603" V 8530 3400 50  0001 C CNN
 F 3 "" H 8600 3400 50  0001 C CNN
 	1    8600 3400
@@
 F 0 "R10" V 9075 2800 50  0000 C CNN
 F 1 "10K" V 8975 2800 50  0000 C CNN
-F 2 "" V 8905 2800 50  0001 C CNN
+F 2 "Resistors_SMD:R_0603" V 8905 2800 50  0001 C CNN
 F 3 "" H 8975 2800 50  0001 C CNN
 	1    8975 2800
@@
 F 0 "R5" V 6725 7150 50  0000 C CNN
 F 1 "10K" V 6625 7150 50  0000 C CNN
-F 2 "" V 6555 7150 50  0001 C CNN
+F 2 "Resistors_SMD:R_0603" V 6555 7150 50  0001 C CNN
 F 3 "" H 6625 7150 50  0001 C CNN
 	1    6625 7150
@@
 F 0 "J2" H 5450 1350 50  0000 C CNN
 F 1 "Conn_02x03_Odd_Even" H 5450 800 50  0000 C CNN
-F 2 "" H 5400 1150 50  0001 C CNN
+F 2 "Socket_Strips:Socket_Strip_Straight_2x03_Pitch2.54mm" H 5400 1150 50  0001 C CNN
 F 3 "" H 5400 1150 50  0001 C CNN
 	1    5400 1150

Commit message: all associated
Parts:
- J1: footprint (none) -> Custom:USB_microB_2040002-1_alt
- SW2, SW3: value SW_SPDT -> SW_DPDT; footprint (none) -> Custom:JS202011SCQN
Changed lines of the file:
@@
 $EndDescr
 $Comp
-L GND #PWR01
+L GND #PWR8
 U 1 1 59F4A74C
 P 2825 6675
-F 0 "#PWR01" H 2825 6425 50  0001 C CNN
+F 0 "#PWR8" H 2825 6425 50  0001 C CNN
 F 1 "GND" H 2825 6525 50  0000 C CNN
 F 2 "" H 2825 6675 50  0001 C CNN
@@
 $EndComp
 $Comp
-L GND #PWR02
+L GND #PWR6
 U 1 1 59FA48AB
 P 1650 5925
-F 0 "#PWR02" H 1650 5675 50  0001 C CNN
+F 0 "#PWR6" H 1650 5675 50  0001 C CNN
 F 1 "GND" H 1650 5775 50  0000 C CNN
 F 2 "" H 1650 5925 50  0001 C CNN
@@
 $EndComp
 $Comp
-L GND #PWR03
+L GND #PWR2
 U 1 1 59FA5C44
 P 1200 5325
-F 0 "#PWR03" H 1200 5075 50  0001 C CNN
+F 0 "#PWR2" H 1200 5075 50  0001 C CNN
 F 1 "GND" H 1200 5175 50  0000 C CNN
 F 2 "" H 1200 5325 50  0001 C CNN
@@
 $EndComp
 $Comp
-L GND #PWR04
+L GND #PWR4
 U 1 1 59FA6358
 P 1550 3525
-F 0 "#PWR04" H 1550 3275 50  0001 C CNN
+F 0 "#PWR4" H 1550 3275 50  0001 C CNN
 F 1 "GND" H 1550 3375 50  0000 C CNN
 F 2 "" H 1550 3525 50  0001 C CNN
@@
 SS
 $Comp
-L GND #PWR05
+L GND #PWR12
 U 1 1 59FA820D
 P 4450 5625
-F 0 "#PWR05" H 4450 5375 50  0001 C CNN
+F 0 "#PWR12" H 4450 5375 50  0001 C CNN
 F 1 "GND" H 4450 5475 50  0000 C CNN
 F 2 "" H 4450 5625 50  0001 C CNN
@@
 $EndComp
 $Comp
-L GND #PWR06
+L GND #PWR7
 U 1 1 59FA9EFC
 P 2125 1025
-F 0 "#PWR06" H 2125 775 50  0001 C CNN
+F 0 "#PWR7" H 2125 775 50  0001 C CNN
 F 1 "GND" H 2125 875 50  0000 C CNN
 F 2 "" H 2125 1025 50  0001 C CNN
@@
 $EndComp
 $Comp
-L +5V #PWR07
+L +5V #PWR5
 U 1 1 59FABF21
 P 1650 3275
-F 0 "#PWR07" H 1650 3125 50  0001 C CNN
+F 0 "#PWR5" H 1650 3125 50  0001 C CNN
 F 1 "+5V" H 1650 3415 50  0000 C CNN
 F 2 "" H 1650 3275 50  0001 C CNN
@@
 $EndComp
 $Comp
-L +5V #PWR08
+L +5V #PWR1
 U 1 1 59FABFF9
 P 750 725
-F 0 "#PWR08" H 750 575 50  0001 C CNN
+F 0 "#PWR1" H 750 575 50  0001 C CNN
 F 1 "+5V" H 750 865 50  0000 C CNN
 F 2 "" H 750 725 50  0001 C CNN
@@
 $EndComp
 $Comp
-L +5V #PWR09
+L +5V #PWR9
 U 1 1 59FAD814
 P 3125 3275
-F 0 "#PWR09" H 3125 3125 50  0001 C CNN
+F 0 "#PWR9" H 3125 3125 50  0001 C CNN
 F 1 "+5V" H 3125 3415 50  0000 C CNN
 F 2 "" H 3125 3275 50  0001 C CNN
@@
 $EndComp
 $Comp
-L GND #PWR010
+L GND #PWR3
 U 1 1 59FBA8CC
 P 1275 4300
-F 0 "#PWR010" H 1275 4050 50  0001 C CNN
+F 0 "#PWR3" H 1275 4050 50  0001 C CNN
 F 1 "GND" H 1275 4150 50  0000 C CNN
 F 2 "" H 1275 4300 50  0001 C CNN
@@
 USB5V
 $Comp
-L +5V #PWR011
+L +5V #PWR10
 U 1 1 59FB83A3
 P 4275 850
-F 0 "#PWR011" H 4275 700 50  0001 C CNN
+F 0 "#PWR10" H 4275 700 50  0001 C CNN
 F 1 "+5V" H 4275 990 50  0000 C CNN
 F 2 "" H 4275 850 50  0001 C CNN
@@
 $EndComp
 $Comp
-L +3V3 #PWR012
+L +3V3 #PWR11
 U 1 1 59FB8639
 P 4350 1000
-F 0 "#PWR012" H 4350 850 50  0001 C CNN
+F 0 "#PWR11" H 4350 850 50  0001 C CNN
 F 1 "+3V3" H 4350 1140 50  0000 C CNN
 F 2 "" H 4350 1000 50  0001 C CNN
@@
 P 6425 7000
 F 0 "SW2" H 6425 7170 50  0000 C CNN
-F 1 "SW_SPDT" H 6300 6825 50  0000 C CNN
-F 2 "" H 6425 7000 50  0001 C CNN
+F 1 "SW_DPDT" H 6300 6825 50  0000 C CNN
+F 2 "Custom:JS202011SCQN" H 6425 7000 50  0001 C CNN
 F 3 "" H 6425 7000 50  0001 C CNN
 	1    6425 7000
@@
 $EndComp
 $Comp
-L +5V #PWR013
+L +5V #PWR16
 U 1 1 59FD0DEE
 P 6225 6900
-F 0 "#PWR013" H 6225 6750 50  0001 C CNN
+F 0 "#PWR16" H 6225 6750 50  0001 C CNN
 F 1 "+5V" H 6225 7040 50  0000 C CNN
 F 2 "" H 6225 6900 50  0001 C CNN
@@
 TXa
 $Comp
-L GND #PWR014
+L GND #PWR17
 U 1 1 59FD82C0
 P 6425 1275
-F 0 "#PWR014" H 6425 1025 50  0001 C CNN
+F 0 "#PWR17" H 6425 1025 50  0001 C CNN
 F 1 "GND" H 6425 1125 50  0000 C CNN
 F 2 "" H 6425 1275 50  0001 C CNN
@@
 $EndComp
 $Comp
-L GND #PWR015
+L GND #PWR19
 U 1 1 59FD880A
 P 7600 1275
-F 0 "#PWR015" H 7600 1025 50  0001 C CNN
+F 0 "#PWR19" H 7600 1025 50  0001 C CNN
 F 1 "GND" H 7600 1125 50  0000 C CNN
 F 2 "" H 7600 1275 50  0001 C CNN
@@
 $EndComp
 $Comp
-L GND #PWR016
+L GND #PWR20
 U 1 1 59FD8AC0
 P 8800 1275
-F 0 "#PWR016" H 8800 1025 50  0001 C CNN
+F 0 "#PWR20" H 8800 1025 50  0001 C CNN
 F 1 "GND" H 8800 1125 50  0000 C CNN
 F 2 "" H 8800 1275 50  0001 C CNN
@@
 $EndComp
 $Comp
-L GND #PWR017
+L GND #PWR24
 U 1 1 59FD8E67
 P 9975 1275
-F 0 "#PWR017" H 9975 1025 50  0001 C CNN
+F 0 "#PWR24" H 9975 1025 50  0001 C CNN
 F 1 "GND" H 9975 1125 50  0000 C CNN
 F 2 "" H 9975 1275 50  0001 C CNN
@@
 $EndComp
 $Comp
-L GND #PWR018
+L GND #PWR23
 U 1 1 5A0021A9
 P 9925 3850
-F 0 "#PWR018" H 9925 3600 50  0001 C CNN
+F 0 "#PWR23" H 9925 3600 50  0001 C CNN
 F 1 "GND" H 9925 3700 50  0000 C CNN
 F 2 "" H 9925 3850 50  0001 C CNN
@@
 $EndComp
 $Comp
-L +5V #PWR019
+L +5V #PWR22
 U 1 1 5A0026FD
 P 9925 1850
-F 0 "#PWR019" H 9925 1700 50  0001 C CNN
+F 0 "#PWR22" H 9925 1700 50  0001 C CNN
 F 1 "+5V" H 9925 1990 50  0000 C CNN
 F 2 "" H 9925 1850 50  0001 C CNN
@@
 $EndComp
 $Comp
-L GND #PWR020
+L GND #PWR21
 U 1 1 5A005A93
 P 9125 2750
-F 0 "#PWR020" H 9125 2500 50  0001 C CNN
+F 0 "#PWR21" H 9125 2500 50  0001 C CNN
 F 1 "GND" H 9125 2600 50  0000 C CNN
 F 2 "" H 9125 2750 50  0001 C CNN
@@
 $EndComp
 $Comp
-L GND #PWR021
+L GND #PWR25
 U 1 1 5A013A28
 P 10750 2750
-F 0 "#PWR021" H 10750 2500 50  0001 C CNN
+F 0 "#PWR25" H 10750 2500 50  0001 C CNN
 F 1 "GND" H 10750 2600 50  0000 C CNN
 F 2 "" H 10750 2750 50  0001 C CNN
@@
 P 7175 1800
 F 0 "SW3" H 7175 1970 50  0000 C CNN
-F 1 "SW_SPDT" H 7175 2100 50  0000 C CNN
-F 2 "" H 7175 1800 50  0001 C CNN
+F 1 "SW_DPDT" H 7175 2100 50  0000 C CNN
+F 2 "Custom:JS202011SCQN" H 7175 1800 50  0001 C CNN
 F 3 "" H 7175 1800 50  0001 C CNN
 	1    7175 1800
@@
 $EndComp
 $Comp
-L GND #PWR022
+L GND #PWR18
 U 1 1 5A04AAA6
 P 6625 7300
-F 0 "#PWR022" H 6625 7050 50  0001 C CNN
+F 0 "#PWR18" H 6625 7050 50  0001 C CNN
 F 1 "GND" H 6625 7150 50  0000 C CNN
 F 2 "" H 6625 7300 50  0001 C CNN
@@
 ICSP HEADER
 $Comp
-L +1V8 #PWR023
+L +1V8 #PWR13
 U 1 1 5A07E30F
 P 4500 1150
-F 0 "#PWR023" H 4500 1000 50  0001 C CNN
+F 0 "#PWR13" H 4500 1000 50  0001 C CNN
 F 1 "+1V8" H 4500 1290 50  0000 C CNN
 F 2 "" H 4500 1150 50  0001 C CNN
@@
 Connection ~ 1950 3525
 $Comp
-L +5V #PWR024
+L +5V #PWR14
 U 1 1 5A01C4EA
 P 5700 1050
-F 0 "#PWR024" H 5700 900 50  0001 C CNN
+F 0 "#PWR14" H 5700 900 50  0001 C CNN
 F 1 "+5V" H 5700 1190 50  0000 C CNN
 F 2 "" H 5700 1050 50  0001 C CNN
@@
 MOSI
 $Comp
-L GND #PWR025
+L GND #PWR15
 U 1 1 5A01C829
 P 5700 1250
-F 0 "#PWR025" H 5700 1000 50  0001 C CNN
+F 0 "#PWR15" H 5700 1000 50  0001 C CNN
 F 1 "GND" H 5700 1100 50  0000 C CNN
 F 2 "" H 5700 1250 50  0001 C CNN
@@
 F 0 "J1" H 1000 5375 50  0000 L CNN
 F 1 "USB_OTG_fix" H 1000 5275 50  0000 L CNN
-F 2 "" H 1350 4875 50  0001 C CNN
+F 2 "Custom:USB_microB_2040002-1_alt" H 1350 4875 50  0001 C CNN
 F 3 "" H 1350 4875 50  0001 C CNN
 	1    1200 4925
