File: ultrasonic_localization/rfModule.sch (KiCad schematic (older format))
At the start: 16 parts

Commit message: refactoring some stuff
Changed lines of the file:
@@
 LIBS:power
 LIBS:device
+LIBS:switches
+LIBS:relays
+LIBS:motors
 LIBS:transistors
 LIBS:conn
@@
 LIBS:valves
 LIBS:custom
+LIBS:ultrasonic_localization-cache
 EELAYER 25 0
 EELAYER END
@@
 	4400 2150 4400 2250
 Connection ~ 4300 2150
-Text Label 3200 3150 2    60   ~ 0
-CE
-Text Label 3200 3250 2    60   ~ 0
-CSN
-Text Label 3200 3350 2    60   ~ 0
-SCK
-Text Label 3200 3450 2    60   ~ 0
-MOSI
-Text Label 3200 3550 2    60   ~ 0
-MISO
 $Comp
 L C C?
@@
 Wire Wire Line
 	4700 5300 4700 5400
+Text HLabel 3200 3250 0    60   Input ~ 0
+CSN
+Text HLabel 3200 3350 0    60   Input ~ 0
+SCK
+Text HLabel 3200 3450 0    60   Input ~ 0
+MOSI
+Text HLabel 3200 3550 0    60   Input ~ 0
+MISO
+Text HLabel 3200 3150 0    60   Input ~ 0
+CE
 $EndSCHEMATC

Commit message: Added a antenna
Parts:
- added U?: ANT016008LCS2442MA2, symbol ANT016008LCS2442MA2
Connections:
- net 50ohmRF: no longer names the net of C?.1, C?.1
- net 50ohmRF: now also U?.4 (IN)
- new net RF: U?.1 (OUT)
- no-connect marks 0 -> 4
Changed lines of the file:
@@
 LIBS:power
 LIBS:device
-LIBS:switches
-LIBS:relays
-LIBS:motors
 LIBS:transistors
 LIBS:conn
@@
 LIBS:valves
 LIBS:custom
-LIBS:ultrasonic_localization-cache
+LIBS:rfModule-cache
 EELAYER 25 0
 EELAYER END
 $Descr A4 11693 8268
 encoding utf-8
-Sheet 2 7
+Sheet 1 1
 Title ""
 Date ""
@@
 	6450 3350 6800 3350
 Wire Wire Line
-	7100 3350 7650 3350
+	7100 3350 8000 3350
 Wire Wire Line
 	7400 3350 7400 3450
@@
 Wire Wire Line
 	7400 3750 7400 3900
-Text Label 7650 3350 0    60   ~ 0
-50ohmRF
 Connection ~ 7400 3350
 $Comp
@@
 Text HLabel 3200 3150 0    60   Input ~ 0
 CE
+$Comp
+L ANT016008LCS2442MA2 U?
+U 1 1 59FC6AEB
+P 8450 3450
+F 0 "U?" H 8450 3650 60  0000 C CNN
+F 1 "ANT016008LCS2442MA2" H 8450 3750 60  0000 C CNN
+F 2 "" H 8450 3450 60  0001 C CNN
+F 3 "" H 8450 3450 60  0001 C CNN
+	1    8450 3450
+	1    0    0    -1
+$EndComp
+Text Label 8900 3350 0    60   ~ 0
+RF
+NoConn ~ 8300 3800
+NoConn ~ 8400 3800
+NoConn ~ 8500 3800
+NoConn ~ 8600 3800
 $EndSCHEMATC
