File: ultrasonic_localization/rfModule.sch (KiCad schematic (older format))
At the start: 17 parts

Commit message: finished ultrasound and some other stuff
Other:
- note added: "PULLUP RESISTORS"
Changed lines of the file:
@@
 NoConn ~ 8500 3800
 NoConn ~ 8600 3800
+Text Notes 2550 3700 0    60   ~ 0
+PULLUP RESISTORS
 $EndSCHEMATC

Commit message: added osc src
Other:
- note added: "TODO : PULLUP RESISTORS"
- note removed: "PULLUP RESISTORS"
Changed lines of the file:
@@
 NoConn ~ 8500 3800
 NoConn ~ 8600 3800
-Text Notes 2550 3700 0    60   ~ 0
-PULLUP RESISTORS
+Text Notes 2250 3700 0    60   ~ 0
+TODO : PULLUP RESISTORS
 $EndSCHEMATC

Commit message: sim + analysis for 40kHz filter
Parts:
- gave numbers to parts that had none: 17
Changed lines of the file:
@@
 $EndDescr
 $Comp
-L nRF24L01+ U?
+L nRF24L01+ U6
 U 1 1 59FAA669
 P 4200 3350
-F 0 "U?" H 4200 3250 50  0000 C CNN
+F 0 "U6" H 4200 3250 50  0000 C CNN
 F 1 "nRF24L01+" H 4200 3450 50  0000 C CNN
 F 2 "MODULE" H 4200 3350 50  0001 C CNN
@@
 $EndComp
 $Comp
-L Crystal_GND24 Y?
+L Crystal_GND24 Y2
 U 1 1 59FAA717
 P 4350 4500
-F 0 "Y?" H 4475 4700 50  0000 L CNN
+F 0 "Y2" H 4475 4700 50  0000 L CNN
 F 1 "16MHz" H 4475 4625 50  0000 L CNN
 F 2 "" H 4350 4500 50  0001 C CNN
@@
 $EndComp
 $Comp
-L C C?
+L C C11
 U 1 1 59FAA746
 P 4000 5150
-F 0 "C?" H 4025 5250 50  0000 L CNN
+F 0 "C11" H 4025 5250 50  0000 L CNN
 F 1 "C" H 4025 5050 50  0000 L CNN
 F 2 "" H 4038 5000 50  0001 C CNN
@@
 $EndComp
 $Comp
-L C C?
+L C C12
 U 1 1 59FAA76F
 P 4700 5150
-F 0 "C?" H 4725 5250 50  0000 L CNN
+F 0 "C12" H 4725 5250 50  0000 L CNN
 F 1 "C" H 4725 5050 50  0000 L CNN
 F 2 "" H 4738 5000 50  0001 C CNN
@@
 $EndComp
 $Comp
-L GND #PWR?
+L GND #PWR033
 U 1 1 59FAA7D6
 P 4350 4700
-F 0 "#PWR?" H 4350 4450 50  0001 C CNN
+F 0 "#PWR033" H 4350 4450 50  0001 C CNN
 F 1 "GND" H 4350 4550 50  0000 C CNN
 F 2 "" H 4350 4700 50  0001 C CNN
@@
 $EndComp
 $Comp
-L R R?
+L R R16
 U 1 1 59FAA826
 P 4350 5000
-F 0 "R?" V 4430 5000 50  0000 C CNN
+F 0 "R16" V 4430 5000 50  0000 C CNN
 F 1 "1M" V 4350 5000 50  0000 C CNN
 F 2 "" V 4280 5000 50  0001 C CNN
@@
 $EndComp
 $Comp
-L GND #PWR?
+L GND #PWR034
 U 1 1 59FAA95E
 P 4100 4300
-F 0 "#PWR?" H 4100 4050 50  0001 C CNN
+F 0 "#PWR034" H 4100 4050 50  0001 C CNN
 F 1 "GND" H 4100 4150 50  0000 C CNN
 F 2 "" H 4100 4300 50  0001 C CNN
@@
 IRQ
 $Comp
-L C C?
+L C C8
 U 1 1 59FAAA86
 P 2750 2750
-F 0 "C?" H 2775 2850 50  0000 L CNN
+F 0 "C8" H 2775 2850 50  0000 L CNN
 F 1 "10nF" H 2775 2650 50  0000 L CNN
 F 2 "" H 2788 2600 50  0001 C CNN
@@
 $EndComp
 $Comp
-L C C?
+L C C9
 U 1 1 59FAAAB3
 P 3100 2750
-F 0 "C?" H 3125 2850 50  0000 L CNN
+F 0 "C9" H 3125 2850 50  0000 L CNN
 F 1 "1nF" H 3125 2650 50  0000 L CNN
 F 2 "" H 3138 2600 50  0001 C CNN
@@
 VDD
 $Comp
-L GND #PWR?
+L GND #PWR035
 U 1 1 59FC0938
 P 2950 2950
-F 0 "#PWR?" H 2950 2700 50  0001 C CNN
+F 0 "#PWR035" H 2950 2700 50  0001 C CNN
 F 1 "GND" H 2950 2800 50  0000 C CNN
 F 2 "" H 2950 2950 50  0001 C CNN
@@
 $EndComp
 $Comp
-L GND #PWR?
+L GND #PWR036
 U 1 1 59FAAD07
 P 5400 4200
-F 0 "#PWR?" H 5400 3950 50  0001 C CNN
+F 0 "#PWR036" H 5400 3950 50  0001 C CNN
 F 1 "GND" H 5400 4050 50  0000 C CNN
 F 2 "" H 5400 4200 50  0001 C CNN
@@
 $EndComp
 $Comp
-L C C?
+L C C10
 U 1 1 59FAAF03
 P 3750 2250
-F 0 "C?" H 3775 2350 50  0000 L CNN
+F 0 "C10" H 3775 2350 50  0000 L CNN
 F 1 "33nF" H 3775 2150 50  0000 L CNN
 F 2 "" H 3788 2100 50  0001 C CNN
@@
 $EndComp
 $Comp
-L GND #PWR?
+L GND #PWR037
 U 1 1 59FAB064
 P 3750 2400
-F 0 "#PWR?" H 3750 2150 50  0001 C CNN
+F 0 "#PWR037" H 3750 2150 50  0001 C CNN
 F 1 "GND" H 3750 2250 50  0000 C CNN
 F 2 "" H 3750 2400 50  0001 C CNN
@@
 $EndComp
 $Comp
-L GND #PWR?
+L GND #PWR038
 U 1 1 59FAB1D4
 P 4200 2150
-F 0 "#PWR?" H 4200 1900 50  0001 C CNN
+F 0 "#PWR038" H 4200 1900 50  0001 C CNN
 F 1 "GND" H 4200 2000 50  0000 C CNN
 F 2 "" H 4200 2150 50  0001 C CNN
@@
 $EndComp
 $Comp
-L R R?
+L R R17
 U 1 1 59FAB24D
 P 4400 2400
-F 0 "R?" V 4480 2400 50  0000 C CNN
+F 0 "R17" V 4480 2400 50  0000 C CNN
 F 1 "22K" V 4400 2400 50  0000 C CNN
 F 2 "" V 4330 2400 50  0001 C CNN
@@
 Connection ~ 4300 2150
 $Comp
-L C C?
+L C C13
 U 1 1 59FAB50E
 P 6050 4200
-F 0 "C?" H 6075 4300 50  0000 L CNN
+F 0 "C13" H 6075 4300 50  0000 L CNN
 F 1 "2.2nF" H 6075 4100 50  0000 L CNN
 F 2 "" H 6088 4050 50  0001 C CNN
@@
 $EndComp
 $Comp
-L C C?
+L C C14
 U 1 1 59FAB5D9
 P 6400 4200
-F 0 "C?" H 6425 4300 50  0000 L CNN
+F 0 "C14" H 6425 4300 50  0000 L CNN
 F 1 "4.7pF" H 6425 4100 50  0000 L CNN
 F 2 "" H 6438 4050 50  0001 C CNN
@@
 $EndComp
 $Comp
-L C C?
+L C C15
 U 1 1 59FAB614
 P 6950 3350
-F 0 "C?" H 6975 3450 50  0000 L CNN
+F 0 "C15" H 6975 3450 50  0000 L CNN
 F 1 "1.5pF" H 6975 3250 50  0000 L CNN
 F 2 "" H 6988 3200 50  0001 C CNN
@@
 $EndComp
 $Comp
-L C C?
+L C C16
 U 1 1 59FAB67A
 P 7400 3600
-F 0 "C?" H 7425 3700 50  0000 L CNN
+F 0 "C16" H 7425 3700 50  0000 L CNN
 F 1 "1pF" H 7425 3500 50  0000 L CNN
 F 2 "" H 7438 3450 50  0001 C CNN
@@
 $EndComp
 $Comp
-L L L?
+L L L1
 U 1 1 59FAB803
 P 5800 3500
-F 0 "L?" V 5750 3500 50  0000 C CNN
+F 0 "L1" V 5750 3500 50  0000 C CNN
 F 1 "8.2nH" V 5875 3500 50  0000 C CNN
 F 2 "" H 5800 3500 50  0001 C CNN
@@
 $EndComp
 $Comp
-L L L?
+L L L2
 U 1 1 59FAB858
 P 6300 3350
-F 0 "L?" V 6250 3350 50  0000 C CNN
+F 0 "L2" V 6250 3350 50  0000 C CNN
 F 1 "3.9nH" V 6375 3350 50  0000 C CNN
 F 2 "" H 6300 3350 50  0001 C CNN
@@
 $EndComp
 $Comp
-L L L?
+L L L3
 U 1 1 59FAB893
 P 6300 3650
-F 0 "L?" V 6250 3650 50  0000 C CNN
+F 0 "L3" V 6250 3650 50  0000 C CNN
 F 1 "2.7nH" V 6375 3650 50  0000 C CNN
 F 2 "" H 6300 3650 50  0001 C CNN
@@
 	7400 3350 7400 3450
 $Comp
-L GND #PWR?
+L GND #PWR039
 U 1 1 59FAC373
 P 7400 3900
-F 0 "#PWR?" H 7400 3650 50  0001 C CNN
+F 0 "#PWR039" H 7400 3650 50  0001 C CNN
 F 1 "GND" H 7400 3750 50  0000 C CNN
 F 2 "" H 7400 3900 50  0001 C CNN
@@
 $EndComp
 $Comp
-L GND #PWR?
+L GND #PWR040
 U 1 1 59FAC3A7
 P 6050 4500
-F 0 "#PWR?" H 6050 4250 50  0001 C CNN
+F 0 "#PWR040" H 6050 4250 50  0001 C CNN
 F 1 "GND" H 6050 4350 50  0000 C CNN
 F 2 "" H 6050 4500 50  0001 C CNN
@@
 $EndComp
 $Comp
-L GND #PWR?
+L GND #PWR041
 U 1 1 59FAC3E9
 P 6400 4500
-F 0 "#PWR?" H 6400 4250 50  0001 C CNN
+F 0 "#PWR041" H 6400 4250 50  0001 C CNN
 F 1 "GND" H 6400 4350 50  0000 C CNN
 F 2 "" H 6400 4500 50  0001 C CNN
@@
 Connection ~ 7400 3350
 $Comp
-L GND #PWR?
+L GND #PWR042
 U 1 1 59FAC80D
 P 4000 5400
-F 0 "#PWR?" H 4000 5150 50  0001 C CNN
+F 0 "#PWR042" H 4000 5150 50  0001 C CNN
 F 1 "GND" H 4000 5250 50  0000 C CNN
 F 2 "" H 4000 5400 50  0001 C CNN
@@
 $EndComp
 $Comp
-L GND #PWR?
+L GND #PWR043
 U 1 1 59FAC948
 P 4700 5400
-F 0 "#PWR?" H 4700 5150 50  0001 C CNN
+F 0 "#PWR043" H 4700 5150 50  0001 C CNN
 F 1 "GND" H 4700 5250 50  0000 C CNN
 F 2 "" H 4700 5400 50  0001 C CNN
@@
 CE
 $Comp
-L ANT016008LCS2442MA2 U?
+L ANT016008LCS2442MA2 U7
 U 1 1 59FC6AEB
 P 8450 3450
-F 0 "U?" H 8450 3650 60  0000 C CNN
+F 0 "U7" H 8450 3650 60  0000 C CNN
 F 1 "ANT016008LCS2442MA2" H 8450 3750 60  0000 C CNN
 F 2 "" H 8450 3450 60  0001 C CNN
