File: ultrasonic_localization/rfModule.sch (KiCad schematic (older format))
At the start: 17 parts, among them U6 nRF24L01+, U7 ANT016008LCS2442MA2, Y2 16MHz

Commit message: Assigned many footprints to things
Parts:
- U6: footprint MODULE -> Housings_DFN_QFN:QFN-20-1EP_4x4mm_Pitch0.5mm
Changed lines of the file:
@@
 F 0 "U6" H 4200 3250 50  0000 C CNN
 F 1 "nRF24L01+" H 4200 3450 50  0000 C CNN
-F 2 "MODULE" H 4200 3350 50  0001 C CNN
+F 2 "Housings_DFN_QFN:QFN-20-1EP_4x4mm_Pitch0.5mm" H 4200 3350 50  0001 C CNN
 F 3 "DOCUMENTATION" H 4200 3350 50  0001 C CNN
 	1    4200 3350

Commit message: almost resolved DRC
Connections:
- net +3V3: no longer U6.6 (~IRQ)
- new net IRQ: U6.6 (~IRQ)
- no-connect marks 4 -> 5
Other:
- moved on the sheet: C8, C9
Changed lines of the file:
@@
 $EndComp
 $Comp
-L GND #PWR033
+L GND #PWR026
 U 1 1 59FAA7D6
 P 4350 4700
-F 0 "#PWR033" H 4350 4450 50  0001 C CNN
+F 0 "#PWR026" H 4350 4450 50  0001 C CNN
 F 1 "GND" H 4350 4550 50  0000 C CNN
 F 2 "" H 4350 4700 50  0001 C CNN
@@
 $EndComp
 $Comp
-L GND #PWR034
+L GND #PWR027
 U 1 1 59FAA95E
 P 4100 4300
-F 0 "#PWR034" H 4100 4050 50  0001 C CNN
+F 0 "#PWR027" H 4100 4050 50  0001 C CNN
 F 1 "GND" H 4100 4150 50  0000 C CNN
 F 2 "" H 4100 4300 50  0001 C CNN
@@
 	1    0    0    -1
 $EndComp
-Text Label 3750 4050 2    60   ~ 0
-IRQ
 $Comp
 L C C8
 U 1 1 59FAAA86
-P 2750 2750
-F 0 "C8" H 2775 2850 50  0000 L CNN
-F 1 "10nF" H 2775 2650 50  0000 L CNN
-F 2 "" H 2788 2600 50  0001 C CNN
-F 3 "" H 2750 2750 50  0001 C CNN
-	1    2750 2750
+P 2750 2700
+F 0 "C8" H 2775 2800 50  0000 L CNN
+F 1 "10nF" H 2775 2600 50  0000 L CNN
+F 2 "" H 2788 2550 50  0001 C CNN
+F 3 "" H 2750 2700 50  0001 C CNN
+	1    2750 2700
 	1    0    0    -1
 $EndComp
@@
 L C C9
 U 1 1 59FAAAB3
-P 3100 2750
-F 0 "C9" H 3125 2850 50  0000 L CNN
-F 1 "1nF" H 3125 2650 50  0000 L CNN
-F 2 "" H 3138 2600 50  0001 C CNN
-F 3 "" H 3100 2750 50  0001 C CNN
-	1    3100 2750
-	1    0    0    -1
-$EndComp
-$Comp
-L GND #PWR035
+P 3100 2700
+F 0 "C9" H 3125 2800 50  0000 L CNN
+F 1 "1nF" H 3125 2600 50  0000 L CNN
+F 2 "" H 3138 2550 50  0001 C CNN
+F 3 "" H 3100 2700 50  0001 C CNN
+	1    3100 2700
+	1    0    0    -1
+$EndComp
+$Comp
+L GND #PWR028
 U 1 1 59FC0938
 P 2950 2950
-F 0 "#PWR035" H 2950 2700 50  0001 C CNN
+F 0 "#PWR028" H 2950 2700 50  0001 C CNN
 F 1 "GND" H 2950 2800 50  0000 C CNN
 F 2 "" H 2950 2950 50  0001 C CNN
@@
 $EndComp
 $Comp
-L GND #PWR036
+L GND #PWR029
 U 1 1 59FAAD07
 P 5400 4200
-F 0 "#PWR036" H 5400 3950 50  0001 C CNN
+F 0 "#PWR029" H 5400 3950 50  0001 C CNN
 F 1 "GND" H 5400 4050 50  0000 C CNN
 F 2 "" H 5400 4200 50  0001 C CNN
@@
 $EndComp
 $Comp
-L GND #PWR037
+L GND #PWR030
 U 1 1 59FAB064
 P 3750 2400
-F 0 "#PWR037" H 3750 2150 50  0001 C CNN
+F 0 "#PWR030" H 3750 2150 50  0001 C CNN
 F 1 "GND" H 3750 2250 50  0000 C CNN
 F 2 "" H 3750 2400 50  0001 C CNN
@@
 $EndComp
 $Comp
-L GND #PWR038
+L GND #PWR031
 U 1 1 59FAB1D4
 P 4200 2150
-F 0 "#PWR038" H 4200 1900 50  0001 C CNN
+F 0 "#PWR031" H 4200 1900 50  0001 C CNN
 F 1 "GND" H 4200 2000 50  0000 C CNN
 F 2 "" H 4200 2150 50  0001 C CNN
@@
 	4350 4300 4100 4300
 Wire Wire Line
-	3750 4050 4000 4050
-Wire Wire Line
-	2750 2900 2750 2950
+	2750 2850 2750 2950
 Wire Wire Line
 	2750 2950 3100 2950
 Wire Wire Line
-	3100 2950 3100 2900
+	3100 2950 3100 2850
 Connection ~ 2950 2950
 Wire Wire Line
-	4200 2600 4200 2650
-Wire Wire Line
-	2500 2600 5200 2600
-Wire Wire Line
-	4100 4050 3300 4050
-Wire Wire Line
-	3300 4050 3300 2600
-Connection ~ 3300 2600
-Connection ~ 3100 2600
-Connection ~ 2750 2600
-Wire Wire Line
-	5200 2600 5200 3150
-Connection ~ 4200 2600
+	3300 2550 3300 4150
+Connection ~ 3300 2550
+Connection ~ 3100 2550
 Wire Wire Line
 	4200 4050 5400 4050
@@
 	5400 3250 5400 4200
 Connection ~ 5400 4050
-Wire Wire Line
-	4100 2650 4100 2100
 Wire Wire Line
 	4100 2100 3750 2100
@@
 	7400 3350 7400 3450
 $Comp
-L GND #PWR039
+L GND #PWR032
 U 1 1 59FAC373
 P 7400 3900
-F 0 "#PWR039" H 7400 3650 50  0001 C CNN
+F 0 "#PWR032" H 7400 3650 50  0001 C CNN
 F 1 "GND" H 7400 3750 50  0000 C CNN
 F 2 "" H 7400 3900 50  0001 C CNN
@@
 $EndComp
 $Comp
-L GND #PWR040
+L GND #PWR033
 U 1 1 59FAC3A7
 P 6050 4500
-F 0 "#PWR040" H 6050 4250 50  0001 C CNN
+F 0 "#PWR033" H 6050 4250 50  0001 C CNN
 F 1 "GND" H 6050 4350 50  0000 C CNN
 F 2 "" H 6050 4500 50  0001 C CNN
@@
 $EndComp
 $Comp
-L GND #PWR041
+L GND #PWR034
 U 1 1 59FAC3E9
 P 6400 4500
-F 0 "#PWR041" H 6400 4250 50  0001 C CNN
+F 0 "#PWR034" H 6400 4250 50  0001 C CNN
 F 1 "GND" H 6400 4350 50  0000 C CNN
 F 2 "" H 6400 4500 50  0001 C CNN
@@
 Connection ~ 7400 3350
 $Comp
-L GND #PWR042
+L GND #PWR035
 U 1 1 59FAC80D
 P 4000 5400
-F 0 "#PWR042" H 4000 5150 50  0001 C CNN
+F 0 "#PWR035" H 4000 5150 50  0001 C CNN
 F 1 "GND" H 4000 5250 50  0000 C CNN
 F 2 "" H 4000 5400 50  0001 C CNN
@@
 $EndComp
 $Comp
-L GND #PWR043
+L GND #PWR036
 U 1 1 59FAC948
 P 4700 5400
-F 0 "#PWR043" H 4700 5150 50  0001 C CNN
+F 0 "#PWR036" H 4700 5150 50  0001 C CNN
 F 1 "GND" H 4700 5250 50  0000 C CNN
 F 2 "" H 4700 5400 50  0001 C CNN
@@
 RF
 NoConn ~ 8300 3800
-NoConn ~ 8400 3800
 NoConn ~ 8500 3800
 NoConn ~ 8600 3800
-$Comp
-L +3V3 #PWR?
-U 1 1 5A14A190
-P 2500 2600
-F 0 "#PWR?" H 2500 2450 50  0001 C CNN
-F 1 "+3V3" H 2500 2740 50  0000 C CNN
-F 2 "" H 2500 2600 50  0001 C CNN
-F 3 "" H 2500 2600 50  0001 C CNN
-	1    2500 2600
-	1    0    0    -1
-$EndComp
+NoConn ~ 8900 3350
+NoConn ~ 8400 3800
+Text HLabel 3200 4050 0    60   Input ~ 0
+IRQ
+Wire Wire Line
+	3300 4150 4100 4150
+Wire Wire Line
+	3200 4050 4000 4050
+Wire Wire Line
+	4100 4150 4100 4050
+Wire Wire Line
+	4100 2650 4100 2100
+$Comp
+L +3V3 #PWR037
+U 1 1 5A050D21
+P 2750 2550
+F 0 "#PWR037" H 2750 2400 50  0001 C CNN
+F 1 "+3V3" H 2750 2690 50  0000 C CNN
+F 2 "" H 2750 2550 50  0001 C CNN
+F 3 "" H 2750 2550 50  0001 C CNN
+	1    2750 2550
+	1    0    0    -1
+$EndComp
+$Comp
+L +3V3 #PWR038
+U 1 1 5A051A80
+P 4200 2650
+F 0 "#PWR038" H 4200 2500 50  0001 C CNN
+F 1 "+3V3" H 4200 2790 50  0000 C CNN
+F 2 "" H 4200 2650 50  0001 C CNN
+F 3 "" H 4200 2650 50  0001 C CNN
+	1    4200 2650
+	1    0    0    -1
+$EndComp
+$Comp
+L +3V3 #PWR039
+U 1 1 5A051B2E
+P 5200 3150
+F 0 "#PWR039" H 5200 3000 50  0001 C CNN
+F 1 "+3V3" H 5200 3290 50  0000 C CNN
+F 2 "" H 5200 3150 50  0001 C CNN
+F 3 "" H 5200 3150 50  0001 C CNN
+	1    5200 3150
+	1    0    0    -1
+$EndComp
+Wire Wire Line
+	2750 2550 3300 2550
+Connection ~ 5200 3150
 $EndSCHEMATC

Commit message: Assigned footprints to menial components
Parts:
- C10, C13, C14, C15, C16, C8, C9: footprint (none) -> Capacitors_SMD:C_0603
- C11, C12: value C -> 12pF; footprint (none) -> Capacitors_SMD:C_0603
- L1, L2, L3: footprint (none) -> Inductors_SMD:L_0603
- R16, R17: footprint (none) -> Resistors_SMD:R_0603
- U7: footprint (none) -> Custom:ANT016008LCS2442MA2
- Y2: footprint (none) -> Crystals:Crystal_SMD_3225-4pin_3.2x2.5mm
Changed lines of the file:
@@
 F 0 "Y2" H 4475 4700 50  0000 L CNN
 F 1 "16MHz" H 4475 4625 50  0000 L CNN
-F 2 "" H 4350 4500 50  0001 C CNN
+F 2 "Crystals:Crystal_SMD_3225-4pin_3.2x2.5mm" H 4350 4500 50  0001 C CNN
 F 3 "" H 4350 4500 50  0001 C CNN
 	1    4350 4500
@@
 P 4000 5150
 F 0 "C11" H 4025 5250 50  0000 L CNN
-F 1 "C" H 4025 5050 50  0000 L CNN
-F 2 "" H 4038 5000 50  0001 C CNN
+F 1 "12pF" H 4025 5050 50  0000 L CNN
+F 2 "Capacitors_SMD:C_0603" H 4038 5000 50  0001 C CNN
 F 3 "" H 4000 5150 50  0001 C CNN
 	1    4000 5150
@@
 P 4700 5150
 F 0 "C12" H 4725 5250 50  0000 L CNN
-F 1 "C" H 4725 5050 50  0000 L CNN
-F 2 "" H 4738 5000 50  0001 C CNN
+F 1 "12pF" H 4725 5050 50  0000 L CNN
+F 2 "Capacitors_SMD:C_0603" H 4738 5000 50  0001 C CNN
 F 3 "" H 4700 5150 50  0001 C CNN
 	1    4700 5150
@@
 F 0 "R16" V 4430 5000 50  0000 C CNN
 F 1 "1M" V 4350 5000 50  0000 C CNN
-F 2 "" V 4280 5000 50  0001 C CNN
+F 2 "Resistors_SMD:R_0603" V 4280 5000 50  0001 C CNN
 F 3 "" H 4350 5000 50  0001 C CNN
 	1    4350 5000
@@
 F 0 "C8" H 2775 2800 50  0000 L CNN
 F 1 "10nF" H 2775 2600 50  0000 L CNN
-F 2 "" H 2788 2550 50  0001 C CNN
+F 2 "Capacitors_SMD:C_0603" H 2788 2550 50  0001 C CNN
 F 3 "" H 2750 2700 50  0001 C CNN
 	1    2750 2700
@@
 F 0 "C9" H 3125 2800 50  0000 L CNN
 F 1 "1nF" H 3125 2600 50  0000 L CNN
-F 2 "" H 3138 2550 50  0001 C CNN
+F 2 "Capacitors_SMD:C_0603" H 3138 2550 50  0001 C CNN
 F 3 "" H 3100 2700 50  0001 C CNN
 	1    3100 2700
@@
 F 0 "C10" H 3775 2350 50  0000 L CNN
 F 1 "33nF" H 3775 2150 50  0000 L CNN
-F 2 "" H 3788 2100 50  0001 C CNN
+F 2 "Capacitors_SMD:C_0603" H 3788 2100 50  0001 C CNN
 F 3 "" H 3750 2250 50  0001 C CNN
 	1    3750 2250
@@
 F 0 "R17" V 4480 2400 50  0000 C CNN
 F 1 "22K" V 4400 2400 50  0000 C CNN
-F 2 "" V 4330 2400 50  0001 C CNN
+F 2 "Resistors_SMD:R_0603" V 4330 2400 50  0001 C CNN
 F 3 "" H 4400 2400 50  0001 C CNN
 	1    4400 2400
@@
 F 0 "C13" H 6075 4300 50  0000 L CNN
 F 1 "2.2nF" H 6075 4100 50  0000 L CNN
-F 2 "" H 6088 4050 50  0001 C CNN
+F 2 "Capacitors_SMD:C_0603" H 6088 4050 50  0001 C CNN
 F 3 "" H 6050 4200 50  0001 C CNN
 	1    6050 4200
@@
 F 0 "C14" H 6425 4300 50  0000 L CNN
 F 1 "4.7pF" H 6425 4100 50  0000 L CNN
-F 2 "" H 6438 4050 50  0001 C CNN
+F 2 "Capacitors_SMD:C_0603" H 6438 4050 50  0001 C CNN
 F 3 "" H 6400 4200 50  0001 C CNN
 	1    6400 4200
@@
 F 0 "C15" H 6975 3450 50  0000 L CNN
 F 1 "1.5pF" H 6975 3250 50  0000 L CNN
-F 2 "" H 6988 3200 50  0001 C CNN
+F 2 "Capacitors_SMD:C_0603" H 6988 3200 50  0001 C CNN
 F 3 "" H 6950 3350 50  0001 C CNN
 	1    6950 3350
@@
 F 0 "C16" H 7425 3700 50  0000 L CNN
 F 1 "1pF" H 7425 3500 50  0000 L CNN
-F 2 "" H 7438 3450 50  0001 C CNN
+F 2 "Capacitors_SMD:C_0603" H 7438 3450 50  0001 C CNN
 F 3 "" H 7400 3600 50  0001 C CNN
 	1    7400 3600
@@
 F 0 "L1" V 5750 3500 50  0000 C CNN
 F 1 "8.2nH" V 5875 3500 50  0000 C CNN
-F 2 "" H 5800 3500 50  0001 C CNN
+F 2 "Inductors_SMD:L_0603" H 5800 3500 50  0001 C CNN
 F 3 "" H 5800 3500 50  0001 C CNN
 	1    5800 3500
@@
 F 0 "L2" V 6250 3350 50  0000 C CNN
 F 1 "3.9nH" V 6375 3350 50  0000 C CNN
-F 2 "" H 6300 3350 50  0001 C CNN
+F 2 "Inductors_SMD:L_0603" H 6300 3350 50  0001 C CNN
 F 3 "" H 6300 3350 50  0001 C CNN
 	1    6300 3350
@@
 F 0 "L3" V 6250 3650 50  0000 C CNN
 F 1 "2.7nH" V 6375 3650 50  0000 C CNN
-F 2 "" H 6300 3650 50  0001 C CNN
+F 2 "Inductors_SMD:L_0603" H 6300 3650 50  0001 C CNN
 F 3 "" H 6300 3650 50  0001 C CNN
 	1    6300 3650
@@
 F 0 "U7" H 8450 3650 60  0000 C CNN
 F 1 "ANT016008LCS2442MA2" H 8450 3750 60  0000 C CNN
-F 2 "" H 8450 3450 60  0001 C CNN
+F 2 "Custom:ANT016008LCS2442MA2" H 8450 3450 60  0001 C CNN
 F 3 "" H 8450 3450 60  0001 C CNN
 	1    8450 3450

Commit message: Routed rotational module
Parts:
- renumbered C8 to C201, C9 to C202, C10 to C203, C11 to C204, C12 to C205, C13 to C206, C14 to C207, C15 to C208, C16 to C209, L1 to L201, L2 to L202, L3 to L203, R16 to R201, R17 to R202, U6 to U201, U7 to U202, Y2 to Y201
Changed lines of the file:
@@
 $EndDescr
 $Comp
-L nRF24L01+ U6
+L nRF24L01+ U201
 U 1 1 59FAA669
 P 4200 3350
-F 0 "U6" H 4200 3250 50  0000 C CNN
+F 0 "U201" H 4200 3250 50  0000 C CNN
 F 1 "nRF24L01+" H 4200 3450 50  0000 C CNN
 F 2 "Housings_DFN_QFN:QFN-20-1EP_4x4mm_Pitch0.5mm" H 4200 3350 50  0001 C CNN
@@
 $EndComp
 $Comp
-L Crystal_GND24 Y2
+L Crystal_GND24 Y201
 U 1 1 59FAA717
 P 4350 4500
-F 0 "Y2" H 4475 4700 50  0000 L CNN
+F 0 "Y201" H 4475 4700 50  0000 L CNN
 F 1 "16MHz" H 4475 4625 50  0000 L CNN
 F 2 "Crystals:Crystal_SMD_3225-4pin_3.2x2.5mm" H 4350 4500 50  0001 C CNN
@@
 $EndComp
 $Comp
-L C C11
+L C C204
 U 1 1 59FAA746
 P 4000 5150
-F 0 "C11" H 4025 5250 50  0000 L CNN
+F 0 "C204" H 4025 5250 50  0000 L CNN
 F 1 "12pF" H 4025 5050 50  0000 L CNN
 F 2 "Capacitors_SMD:C_0603" H 4038 5000 50  0001 C CNN
@@
 $EndComp
 $Comp
-L C C12
+L C C205
 U 1 1 59FAA76F
 P 4700 5150
-F 0 "C12" H 4725 5250 50  0000 L CNN
+F 0 "C205" H 4725 5250 50  0000 L CNN
 F 1 "12pF" H 4725 5050 50  0000 L CNN
 F 2 "Capacitors_SMD:C_0603" H 4738 5000 50  0001 C CNN
@@
 $EndComp
 $Comp
-L GND #PWR33
+L GND #PWR026
 U 1 1 59FAA7D6
 P 4350 4700
-F 0 "#PWR33" H 4350 4450 50  0001 C CNN
+F 0 "#PWR026" H 4350 4450 50  0001 C CNN
 F 1 "GND" H 4350 4550 50  0000 C CNN
 F 2 "" H 4350 4700 50  0001 C CNN
@@
 $EndComp
 $Comp
-L R R16
+L R R201
 U 1 1 59FAA826
 P 4350 5000
-F 0 "R16" V 4430 5000 50  0000 C CNN
+F 0 "R201" V 4430 5000 50  0000 C CNN
 F 1 "1M" V 4350 5000 50  0000 C CNN
 F 2 "Resistors_SMD:R_0603" V 4280 5000 50  0001 C CNN
@@
 $EndComp
 $Comp
-L GND #PWR30
+L GND #PWR027
 U 1 1 59FAA95E
 P 4100 4300
-F 0 "#PWR30" H 4100 4050 50  0001 C CNN
+F 0 "#PWR027" H 4100 4050 50  0001 C CNN
 F 1 "GND" H 4100 4150 50  0000 C CNN
 F 2 "" H 4100 4300 50  0001 C CNN
@@
 $EndComp
 $Comp
-L C C8
+L C C201
 U 1 1 59FAAA86
 P 2750 2700
-F 0 "C8" H 2775 2800 50  0000 L CNN
+F 0 "C201" H 2775 2800 50  0000 L CNN
 F 1 "10nF" H 2775 2600 50  0000 L CNN
 F 2 "Capacitors_SMD:C_0603" H 2788 2550 50  0001 C CNN
@@
 $EndComp
 $Comp
-L C C9
+L C C202
 U 1 1 59FAAAB3
 P 3100 2700
-F 0 "C9" H 3125 2800 50  0000 L CNN
+F 0 "C202" H 3125 2800 50  0000 L CNN
 F 1 "1nF" H 3125 2600 50  0000 L CNN
 F 2 "Capacitors_SMD:C_0603" H 3138 2550 50  0001 C CNN
@@
 $EndComp
 $Comp
-L GND #PWR27
+L GND #PWR028
 U 1 1 59FC0938
 P 2950 2950
-F 0 "#PWR27" H 2950 2700 50  0001 C CNN
+F 0 "#PWR028" H 2950 2700 50  0001 C CNN
 F 1 "GND" H 2950 2800 50  0000 C CNN
 F 2 "" H 2950 2950 50  0001 C CNN
@@
 $EndComp
 $Comp
-L GND #PWR36
+L GND #PWR029
 U 1 1 59FAAD07
 P 5400 4200
-F 0 "#PWR36" H 5400 3950 50  0001 C CNN
+F 0 "#PWR029" H 5400 3950 50  0001 C CNN
 F 1 "GND" H 5400 4050 50  0000 C CNN
 F 2 "" H 5400 4200 50  0001 C CNN
@@
 $EndComp
 $Comp
-L C C10
+L C C203
 U 1 1 59FAAF03
 P 3750 2250
-F 0 "C10" H 3775 2350 50  0000 L CNN
+F 0 "C203" H 3775 2350 50  0000 L CNN
 F 1 "33nF" H 3775 2150 50  0000 L CNN
 F 2 "Capacitors_SMD:C_0603" H 3788 2100 50  0001 C CNN
@@
 $EndComp
 $Comp
-L GND #PWR28
+L GND #PWR030
 U 1 1 59FAB064
 P 3750 2400
-F 0 "#PWR28" H 3750 2150 50  0001 C CNN
+F 0 "#PWR030" H 3750 2150 50  0001 C CNN
 F 1 "GND" H 3750 2250 50  0000 C CNN
 F 2 "" H 3750 2400 50  0001 C CNN
@@
 $EndComp
 $Comp
-L GND #PWR31
+L GND #PWR031
 U 1 1 59FAB1D4
 P 4200 2150
-F 0 "#PWR31" H 4200 1900 50  0001 C CNN
+F 0 "#PWR031" H 4200 1900 50  0001 C CNN
 F 1 "GND" H 4200 2000 50  0000 C CNN
 F 2 "" H 4200 2150 50  0001 C CNN
@@
 $EndComp
 $Comp
-L R R17
+L R R202
 U 1 1 59FAB24D
 P 4400 2400
-F 0 "R17" V 4480 2400 50  0000 C CNN
+F 0 "R202" V 4480 2400 50  0000 C CNN
 F 1 "22K" V 4400 2400 50  0000 C CNN
 F 2 "Resistors_SMD:R_0603" V 4330 2400 50  0001 C CNN
@@
 Connection ~ 4300 2150
 $Comp
-L C C13
+L C C206
 U 1 1 59FAB50E
 P 6050 4200
-F 0 "C13" H 6075 4300 50  0000 L CNN
+F 0 "C206" H 6075 4300 50  0000 L CNN
 F 1 "2.2nF" H 6075 4100 50  0000 L CNN
 F 2 "Capacitors_SMD:C_0603" H 6088 4050 50  0001 C CNN
@@
 $EndComp
 $Comp
-L C C14
+L C C207
 U 1 1 59FAB5D9
 P 6400 4200
-F 0 "C14" H 6425 4300 50  0000 L CNN
+F 0 "C207" H 6425 4300 50  0000 L CNN
 F 1 "4.7pF" H 6425 4100 50  0000 L CNN
 F 2 "Capacitors_SMD:C_0603" H 6438 4050 50  0001 C CNN
@@
 $EndComp
 $Comp
-L C C15
+L C C208
 U 1 1 59FAB614
 P 6950 3350
-F 0 "C15" H 6975 3450 50  0000 L CNN
+F 0 "C208" H 6975 3450 50  0000 L CNN
 F 1 "1.5pF" H 6975 3250 50  0000 L CNN
 F 2 "Capacitors_SMD:C_0603" H 6988 3200 50  0001 C CNN
@@
 $EndComp
 $Comp
-L C C16
+L C C209
 U 1 1 59FAB67A
 P 7400 3600
-F 0 "C16" H 7425 3700 50  0000 L CNN
+F 0 "C209" H 7425 3700 50  0000 L CNN
 F 1 "1pF" H 7425 3500 50  0000 L CNN
 F 2 "Capacitors_SMD:C_0603" H 7438 3450 50  0001 C CNN
@@
 $EndComp
 $Comp
-L L L1
+L L L201
 U 1 1 59FAB803
 P 5800 3500
-F 0 "L1" V 5750 3500 50  0000 C CNN
+F 0 "L201" V 5750 3500 50  0000 C CNN
 F 1 "8.2nH" V 5875 3500 50  0000 C CNN
 F 2 "Inductors_SMD:L_0603" H 5800 3500 50  0001 C CNN
@@
 $EndComp
 $Comp
-L L L2
+L L L202
 U 1 1 59FAB858
 P 6300 3350
-F 0 "L2" V 6250 3350 50  0000 C CNN
+F 0 "L202" V 6250 3350 50  0000 C CNN
 F 1 "3.9nH" V 6375 3350 50  0000 C CNN
 F 2 "Inductors_SMD:L_0603" H 6300 3350 50  0001 C CNN
@@
 $EndComp
 $Comp
-L L L3
+L L L203
 U 1 1 59FAB893
 P 6300 3650
-F 0 "L3" V 6250 3650 50  0000 C CNN
+F 0 "L203" V 6250 3650 50  0000 C CNN
 F 1 "2.7nH" V 6375 3650 50  0000 C CNN
 F 2 "Inductors_SMD:L_0603" H 6300 3650 50  0001 C CNN
@@
 	7400 3350 7400 3450
 $Comp
-L GND #PWR39
+L GND #PWR032
 U 1 1 59FAC373
 P 7400 3900
-F 0 "#PWR39" H 7400 3650 50  0001 C CNN
+F 0 "#PWR032" H 7400 3650 50  0001 C CNN
 F 1 "GND" H 7400 3750 50  0000 C CNN
 F 2 "" H 7400 3900 50  0001 C CNN
@@
 $EndComp
 $Comp
-L GND #PWR37
+L GND #PWR033
 U 1 1 59FAC3A7
 P 6050 4500
-F 0 "#PWR37" H 6050 4250 50  0001 C CNN
+F 0 "#PWR033" H 6050 4250 50  0001 C CNN
 F 1 "GND" H 6050 4350 50  0000 C CNN
 F 2 "" H 6050 4500 50  0001 C CNN
@@
 $EndComp
 $Comp
-L GND #PWR38
+L GND #PWR034
 U 1 1 59FAC3E9
 P 6400 4500
-F 0 "#PWR38" H 6400 4250 50  0001 C CNN
+F 0 "#PWR034" H 6400 4250 50  0001 C CNN
 F 1 "GND" H 6400 4350 50  0000 C CNN
 F 2 "" H 6400 4500 50  0001 C CNN
@@
 Connection ~ 7400 3350
 $Comp
-L GND #PWR29
+L GND #PWR035
 U 1 1 59FAC80D
 P 4000 5400
-F 0 "#PWR29" H 4000 5150 50  0001 C CNN
+F 0 "#PWR035" H 4000 5150 50  0001 C CNN
 F 1 "GND" H 4000 5250 50  0000 C CNN
 F 2 "" H 4000 5400 50  0001 C CNN
@@
 $EndComp
 $Comp
-L GND #PWR34
+L GND #PWR036
 U 1 1 59FAC948
 P 4700 5400
-F 0 "#PWR34" H 4700 5150 50  0001 C CNN
+F 0 "#PWR036" H 4700 5150 50  0001 C CNN
 F 1 "GND" H 4700 5250 50  0000 C CNN
 F 2 "" H 4700 5400 50  0001 C CNN
@@
 CE
 $Comp
-L ANT016008LCS2442MA2 U7
+L ANT016008LCS2442MA2 U202
 U 1 1 59FC6AEB
 P 8450 3450
-F 0 "U7" H 8450 3650 60  0000 C CNN
+F 0 "U202" H 8450 3650 60  0000 C CNN
 F 1 "ANT016008LCS2442MA2" H 8450 3750 60  0000 C CNN
 F 2 "Custom:ANT016008LCS2442MA2" H 8450 3450 60  0001 C CNN
@@
 	4100 2650 4100 2100
 $Comp
-L +3V3 #PWR26
+L +3V3 #PWR037
 U 1 1 5A050D21
 P 2750 2550
-F 0 "#PWR26" H 2750 2400 50  0001 C CNN
+F 0 "#PWR037" H 2750 2400 50  0001 C CNN
 F 1 "+3V3" H 2750 2690 50  0000 C CNN
 F 2 "" H 2750 2550 50  0001 C CNN
@@
 $EndComp
 $Comp
-L +3V3 #PWR32
+L +3V3 #PWR038
 U 1 1 5A051A80
 P 4200 2650
-F 0 "#PWR32" H 4200 2500 50  0001 C CNN
+F 0 "#PWR038" H 4200 2500 50  0001 C CNN
 F 1 "+3V3" H 4200 2790 50  0000 C CNN
 F 2 "" H 4200 2650 50  0001 C CNN
@@
 $EndComp
 $Comp
-L +3V3 #PWR35
+L +3V3 #PWR039
 U 1 1 5A051B2E
 P 5200 3150
-F 0 "#PWR35" H 5200 3000 50  0001 C CNN
+F 0 "#PWR039" H 5200 3000 50  0001 C CNN
 F 1 "+3V3" H 5200 3290 50  0000 C CNN
 F 2 "" H 5200 3150 50  0001 C CNN

Commit message: Fixed board
Parts:
- R202: value 22K -> 20K
Changed lines of the file:
@@
 P 4400 2400
 F 0 "R202" V 4480 2400 50  0000 C CNN
-F 1 "22K" V 4400 2400 50  0000 C CNN
+F 1 "20K" V 4400 2400 50  0000 C CNN
 F 2 "Resistors_SMD:R_0603" V 4330 2400 50  0001 C CNN
 F 3 "" H 4400 2400 50  0001 C CNN
