File: ultrasonic_localization/powerModule.sch (KiCad schematic (older format))
At the start: 25 parts

Commit message: Changed stuff
Parts:
- added C?: 1uf, symbol C
- added C?: 1uF, symbol C
- added D?: D, symbol D
- added L?: L, symbol L
- added R?: 20K, symbol R
- added R?: 1K, symbol R
- added U?: AP3012, symbol AP3012
Connections:
- net 3V7: now also C?.1, L?.2, U?.4 (SHDN), U?.5 (VIN)
- net GND: now also C?.2, C?.2, R?.2, U?.2 (GND)
- new net: R?.1, R?.2, U?.3 (FB)
- new net: D?.2 (A), L?.1, U?.1 (SW)
- new net 26V: C?.1, D?.1 (K), R?.1
Other:
- note added: "Boost Converter, 26V"
Changed lines of the file:
@@
 Text Notes 8225 3550 0    60   ~ 0
 NOTE: Battery Terminals,\nnot actual batteries here
+$Comp
+L R R?
+U 1 1 59FD3A5A
+P 2675 5550
+F 0 "R?" V 2755 5550 50  0000 C CNN
+F 1 "20K" V 2675 5550 50  0000 C CNN
+F 2 "" V 2605 5550 50  0001 C CNN
+F 3 "" H 2675 5550 50  0001 C CNN
+	1    2675 5550
+	1    0    0    -1
+$EndComp
+$Comp
+L R R?
+U 1 1 59FD3A60
+P 2675 5850
+F 0 "R?" V 2755 5850 50  0000 C CNN
+F 1 "1K" V 2675 5850 50  0000 C CNN
+F 2 "" V 2605 5850 50  0001 C CNN
+F 3 "" H 2675 5850 50  0001 C CNN
+	1    2675 5850
+	1    0    0    -1
+$EndComp
+$Comp
+L AP3012 U?
+U 1 1 59FD3A66
+P 1925 5700
+F 0 "U?" H 1925 6050 60  0000 C CNN
+F 1 "AP3012" H 1925 5700 60  0000 C CNN
+F 2 "" H 1925 5700 60  0001 C CNN
+F 3 "" H 1925 5700 60  0001 C CNN
+	1    1925 5700
+	1    0    0    -1
+$EndComp
+$Comp
+L D D?
+U 1 1 59FD3A6C
+P 2425 5150
+F 0 "D?" H 2425 5250 50  0000 C CNN
+F 1 "D" H 2425 5050 50  0000 C CNN
+F 2 "" H 2425 5150 50  0001 C CNN
+F 3 "" H 2425 5150 50  0001 C CNN
+	1    2425 5150
+	-1   0    0    1
+$EndComp
+$Comp
+L L L?
+U 1 1 59FD3A72
+P 1925 5150
+F 0 "L?" V 1875 5150 50  0000 C CNN
+F 1 "L" V 2000 5150 50  0000 C CNN
+F 2 "" H 1925 5150 50  0001 C CNN
+F 3 "" H 1925 5150 50  0001 C CNN
+	1    1925 5150
+	0    1    1    0
+$EndComp
+$Comp
+L C C?
+U 1 1 59FD3A78
+P 1175 6100
+F 0 "C?" H 1200 6200 50  0000 L CNN
+F 1 "1uf" H 1200 6000 50  0000 L CNN
+F 2 "" H 1213 5950 50  0001 C CNN
+F 3 "" H 1175 6100 50  0001 C CNN
+	1    1175 6100
+	1    0    0    -1
+$EndComp
+$Comp
+L C C?
+U 1 1 59FD3A7E
+P 2975 5700
+F 0 "C?" H 3000 5800 50  0000 L CNN
+F 1 "1uF" H 3000 5600 50  0000 L CNN
+F 2 "" H 3013 5550 50  0001 C CNN
+F 3 "" H 2975 5700 50  0001 C CNN
+	1    2975 5700
+	1    0    0    -1
+$EndComp
+Wire Wire Line
+	2075 5150 2275 5150
+Connection ~ 2125 5150
+Wire Wire Line
+	2575 5150 3125 5150
+Wire Wire Line
+	2675 5400 2675 5150
+Connection ~ 2675 5150
+Wire Wire Line
+	2975 5550 2975 5150
+Connection ~ 2975 5150
+$Comp
+L GND #PWR?
+U 1 1 59FD3A8B
+P 1925 6400
+F 0 "#PWR?" H 1925 6150 50  0001 C CNN
+F 1 "GND" H 1925 6250 50  0000 C CNN
+F 2 "" H 1925 6400 50  0001 C CNN
+F 3 "" H 1925 6400 50  0001 C CNN
+	1    1925 6400
+	1    0    0    -1
+$EndComp
+Wire Wire Line
+	1175 6250 1175 6400
+Wire Wire Line
+	1175 6400 2975 6400
+Wire Wire Line
+	1925 6400 1925 6250
+Wire Wire Line
+	2675 6400 2675 6000
+Connection ~ 1925 6400
+Wire Wire Line
+	2975 6400 2975 5850
+Connection ~ 2675 6400
+Wire Wire Line
+	1175 5150 1175 5950
+Wire Wire Line
+	875  5150 1775 5150
+Connection ~ 1725 5150
+Connection ~ 1175 5700
+Text Label 875  5150 2    60   ~ 0
+3V7
+Connection ~ 1175 5150
+Text Notes 1550 6800 0    60   ~ 0
+Boost Converter, 26V
+Wire Notes Line
+	3700 4825 600  4825
+Wire Notes Line
+	600  4825 600  7050
+Wire Notes Line
+	600  7050 3700 7050
+Wire Notes Line
+	3700 7050 3700 4825
+Text HLabel 3125 5150 2    60   Output ~ 0
+26V
 $EndSCHEMATC

Commit message: Added IMU
Parts:
- added C? (x2): 1uF, symbol C
- added U?: LP5907SNX-3.3/NOPB, DQN4, symbol LP5907SNX-3.3/NOPB
Connections:
- net 3V7: now also C?.1, U?.3 (EN), U?.4 (IN)
- net GND: now also C?.2, C?.2, U?.2 (GND)
- new net 1V8: C?.1, U?.1 (OUT)
- no-connect marks 0 -> 1
Changed lines of the file:
@@
 Text HLabel 3125 5150 2    60   Output ~ 0
 26V
+$Comp
+L LP5907SNX-3.3/NOPB U?
+U 1 1 5A06BF49
+P 5350 5800
+F 0 "U?" H 5350 5500 60  0000 C CNN
+F 1 "LP5907SNX-3.3/NOPB" H 5350 6150 60  0000 C CNN
+F 2 "DQN4" H 5350 5400 60  0001 C CNN
+F 3 "" H 4550 5800 60  0000 C CNN
+	1    5350 5800
+	-1   0    0    1
+$EndComp
+$Comp
+L C C?
+U 1 1 5A06E83F
+P 4350 5750
+F 0 "C?" H 4375 5850 50  0000 L CNN
+F 1 "1uF" H 4375 5650 50  0000 L CNN
+F 2 "" H 4388 5600 50  0001 C CNN
+F 3 "" H 4350 5750 50  0001 C CNN
+	1    4350 5750
+	1    0    0    -1
+$EndComp
+Wire Wire Line
+	4800 5600 4350 5600
+Wire Wire Line
+	4800 5800 4800 5600
+$Comp
+L GND #PWR?
+U 1 1 5A06EF81
+P 4350 6000
+F 0 "#PWR?" H 4350 5750 50  0001 C CNN
+F 1 "GND" H 4350 5850 50  0000 C CNN
+F 2 "" H 4350 6000 50  0001 C CNN
+F 3 "" H 4350 6000 50  0001 C CNN
+	1    4350 6000
+	1    0    0    -1
+$EndComp
+Wire Wire Line
+	4350 5900 4350 6000
+Text Label 4350 5600 2    60   ~ 0
+3V7
+$Comp
+L GND #PWR?
+U 1 1 5A075608
+P 5950 6450
+F 0 "#PWR?" H 5950 6200 50  0001 C CNN
+F 1 "GND" H 5950 6300 50  0000 C CNN
+F 2 "" H 5950 6450 50  0001 C CNN
+F 3 "" H 5950 6450 50  0001 C CNN
+	1    5950 6450
+	1    0    0    -1
+$EndComp
+Text HLabel 6225 5900 2    60   Output ~ 0
+1V8
+$Comp
+L C C?
+U 1 1 5A076E77
+P 6150 6200
+F 0 "C?" H 6175 6300 50  0000 L CNN
+F 1 "1uF" H 6175 6100 50  0000 L CNN
+F 2 "" H 6188 6050 50  0001 C CNN
+F 3 "" H 6150 6200 50  0001 C CNN
+	1    6150 6200
+	1    0    0    -1
+$EndComp
+Wire Wire Line
+	6150 6350 6150 6450
+Wire Wire Line
+	6150 6450 5950 6450
+Wire Wire Line
+	5900 5900 6225 5900
+Wire Wire Line
+	6150 6050 6150 5900
+Connection ~ 6150 5900
+Wire Wire Line
+	5900 5700 5950 5700
+Wire Wire Line
+	5950 5700 5950 6450
+NoConn ~ 4800 6000
+Wire Notes Line
+	4100 4825 4100 7050
+Wire Notes Line
+	4100 7050 6750 7050
+Wire Notes Line
+	6750 7050 6750 4825
+Wire Notes Line
+	6750 4825 4100 4825
 $EndSCHEMATC

Commit message: sim + analysis for 40kHz filter
Parts:
- gave numbers to parts that had none: 35
