File: ultrasonic_localization/powerModule.sch (KiCad schematic (older format))
At the start: 35 parts, among them U10 AP3012, U11 AP3012, U12 TPS6223x, U13 LP5907SNX-3.3/NOPB, U14 BQ2423

Commit message: IMU pulldown
Other:
- note added: "1V8 Regulator"
Changed lines of the file:
@@
 Wire Notes Line
 	6750 4825 4100 4825
+Text Notes 5050 6825 0    60   ~ 0
+1V8 Regulator
 $EndSCHEMATC

Commit message: Assigned many footprints to things
Parts:
- removed BT1: Battery_Cell, symbol Battery_Cell
- added J?: Screw_Terminal_1x02, Custom:1x2_Screw_Terminal_5mm_pitch, symbol Screw_Terminal_1x02
- U10: footprint (none) -> TO_SOT_Packages_SMD:SOT-23-5
- U12: footprint (none) -> Custom:UFDFN-6-1.5x1.05mm_Pitch0.5mm
- U13: footprint DQN4 -> TO_SOT_Packages_SMD:SOT-23-5
- U14: footprint MODULE -> Housings_DFN_QFN:QFN-16-1EP_3x3mm_Pitch0.5mm_ThermalVias
Connections:
- wire segments 64 -> 66
Other:
- note removed: "NOTE: Battery Terminals,\nnot actual batteries here"
- moved on the sheet: C33
Changed lines of the file:
@@
 F 0 "U12" H 1950 1050 60  0000 C CNN
 F 1 "TPS6223x" H 1950 1350 60  0000 C CNN
-F 2 "" H 1950 1050 60  0001 C CNN
+F 2 "Custom:UFDFN-6-1.5x1.05mm_Pitch0.5mm" H 1950 1050 60  0001 C CNN
 F 3 "" H 1950 1050 60  0001 C CNN
 	1    1950 1050
@@
 $EndComp
 $Comp
-L Battery_Cell BT1
-U 1 1 59FB3930
-P 8650 2925
-F 0 "BT1" H 8750 3025 50  0000 L CNN
-F 1 "Battery_Cell" H 8750 2925 50  0000 L CNN
-F 2 "" V 8650 2985 50  0001 C CNN
-F 3 "" V 8650 2985 50  0001 C CNN
-	1    8650 2925
-	1    0    0    -1
-$EndComp
-$Comp
 L C C33
 U 1 1 59FB3937
-P 8350 2875
-F 0 "C33" H 8375 2975 50  0000 L CNN
-F 1 "10uF" H 8375 2775 50  0000 L CNN
-F 2 "" H 8388 2725 50  0001 C CNN
-F 3 "" H 8350 2875 50  0001 C CNN
-	1    8350 2875
+P 8650 2875
+F 0 "C33" H 8675 2975 50  0000 L CNN
+F 1 "10uF" H 8675 2775 50  0000 L CNN
+F 2 "" H 8688 2725 50  0001 C CNN
+F 3 "" H 8650 2875 50  0001 C CNN
+	1    8650 2875
 	1    0    0    -1
 $EndComp
@@
 F 0 "U14" H 9850 2125 50  0000 C CNN
 F 1 "BQ2423" H 9850 2325 50  0000 C CNN
-F 2 "MODULE" H 9850 2225 50  0001 C CNN
+F 2 "Housings_DFN_QFN:QFN-16-1EP_3x3mm_Pitch0.5mm_ThermalVias" H 9850 2225 50  0001 C CNN
 F 3 "DOCUMENTATION" H 9850 2225 50  0001 C CNN
 	1    9850 2225
@@
 F 0 "U10" H 1925 3475 60  0000 C CNN
 F 1 "AP3012" H 1925 3125 60  0000 C CNN
-F 2 "" H 1925 3125 60  0001 C CNN
+F 2 "TO_SOT_Packages_SMD:SOT-23-5" H 1925 3125 60  0001 C CNN
 F 3 "" H 1925 3125 60  0001 C CNN
 	1    1925 3125
@@
 Text HLabel 3500 900  2    60   Output ~ 0
 3V3
-Text Notes 8225 3550 0    60   ~ 0
-NOTE: Battery Terminals,\nnot actual batteries here
 $Comp
 L R R38
@@
 F 0 "U13" H 5350 5500 60  0000 C CNN
 F 1 "LP5907SNX-3.3/NOPB" H 5350 6150 60  0000 C CNN
-F 2 "DQN4" H 5350 5400 60  0001 C CNN
+F 2 "TO_SOT_Packages_SMD:SOT-23-5" H 5350 5400 60  0001 C CNN
 F 3 "" H 4550 5800 60  0000 C CNN
 	1    5350 5800
@@
 Text Notes 5050 6825 0    60   ~ 0
 1V8 Regulator
+$Comp
+L Screw_Terminal_1x02 J?
+U 1 1 5A059A6F
+P 8150 2875
+F 0 "J?" H 8150 3125 50  0000 C TNN
+F 1 "Screw_Terminal_1x02" V 8000 2875 50  0000 C TNN
+F 2 "Custom:1x2_Screw_Terminal_5mm_pitch" H 8150 2650 50  0001 C CNN
+F 3 "" H 8125 2875 50  0001 C CNN
+	1    8150 2875
+	1    0    0    -1
+$EndComp
+Wire Wire Line
+	8350 2725 8350 2775
+Wire Wire Line
+	8350 3025 8350 2975
 $EndSCHEMATC

Commit message: almost resolved DRC
Parts:
- removed J?: Screw_Terminal_1x02, Custom:1x2_Screw_Terminal_5mm_pitch, symbol Screw_Terminal_1x02
- added J3: Screw_Terminal_1x02_Bat, Custom:1x2_Screw_Terminal_5mm_pitch, symbol Screw_Terminal_1x02_Bat
Connections:
- wire segments 66 -> 67
Changed lines of the file:
@@
 	1300 900  1300 1050
 $Comp
-L GND #PWR059
+L GND #PWR057
 U 1 1 59FB2340
 P 925 1325
-F 0 "#PWR059" H 925 1075 50  0001 C CNN
+F 0 "#PWR057" H 925 1075 50  0001 C CNN
 F 1 "GND" H 925 1175 50  0000 C CNN
 F 2 "" H 925 1325 50  0001 C CNN
@@
 	925  1200 925  1325
 $Comp
-L GND #PWR060
+L GND #PWR058
 U 1 1 59FB2347
 P 2600 1300
-F 0 "#PWR060" H 2600 1050 50  0001 C CNN
+F 0 "#PWR058" H 2600 1050 50  0001 C CNN
 F 1 "GND" H 2600 1150 50  0000 C CNN
 F 2 "" H 2600 1300 50  0001 C CNN
@@
 	2600 1300 2600 1200
 $Comp
-L GND #PWR061
+L GND #PWR059
 U 1 1 59FB234E
 P 3275 1300
-F 0 "#PWR061" H 3275 1050 50  0001 C CNN
+F 0 "#PWR059" H 3275 1050 50  0001 C CNN
 F 1 "GND" H 3275 1150 50  0000 C CNN
 F 2 "" H 3275 1300 50  0001 C CNN
@@
 $EndComp
 $Comp
-L GND #PWR062
+L GND #PWR060
 U 1 1 59FB392A
 P 8700 2425
-F 0 "#PWR062" H 8700 2175 50  0001 C CNN
+F 0 "#PWR060" H 8700 2175 50  0001 C CNN
 F 1 "GND" H 8700 2275 50  0000 C CNN
 F 2 "" H 8700 2425 50  0001 C CNN
@@
 $EndComp
 $Comp
-L GND #PWR063
+L GND #PWR061
 U 1 1 59FB394B
 P 8650 3175
-F 0 "#PWR063" H 8650 2925 50  0001 C CNN
+F 0 "#PWR061" H 8650 2925 50  0001 C CNN
 F 1 "GND" H 8650 3025 50  0000 C CNN
 F 2 "" H 8650 3175 50  0001 C CNN
@@
 $EndComp
 $Comp
-L GND #PWR064
+L GND #PWR062
 U 1 1 59FB396D
 P 9650 3375
-F 0 "#PWR064" H 9650 3125 50  0001 C CNN
+F 0 "#PWR062" H 9650 3125 50  0001 C CNN
 F 1 "GND" H 9650 3225 50  0000 C CNN
 F 2 "" H 9650 3375 50  0001 C CNN
@@
 $EndComp
 $Comp
-L GND #PWR065
+L GND #PWR063
 U 1 1 59FB397A
 P 10750 2475
-F 0 "#PWR065" H 10750 2225 50  0001 C CNN
+F 0 "#PWR063" H 10750 2225 50  0001 C CNN
 F 1 "GND" H 10750 2325 50  0000 C CNN
 F 2 "" H 10750 2475 50  0001 C CNN
@@
 $EndComp
 $Comp
-L GND #PWR066
+L GND #PWR064
 U 1 1 59FB3987
 P 10550 1475
-F 0 "#PWR066" H 10550 1225 50  0001 C CNN
+F 0 "#PWR064" H 10550 1225 50  0001 C CNN
 F 1 "GND" H 10550 1325 50  0000 C CNN
 F 2 "" H 10550 1475 50  0001 C CNN
@@
 	8650 3025 8650 3175
 Wire Wire Line
-	9100 2725 9100 2625
-Wire Wire Line
 	8350 2725 9100 2725
 Connection ~ 8650 2725
-Wire Wire Line
-	8350 3025 8650 3025
 Wire Wire Line
 	9650 3375 10600 3375
@@
 Connection ~ 2975 2575
 $Comp
-L GND #PWR067
+L GND #PWR065
 U 1 1 59FB4920
 P 1925 3825
-F 0 "#PWR067" H 1925 3575 50  0001 C CNN
+F 0 "#PWR065" H 1925 3575 50  0001 C CNN
 F 1 "GND" H 1925 3675 50  0000 C CNN
 F 2 "" H 1925 3825 50  0001 C CNN
@@
 Connection ~ 2975 5150
 $Comp
-L GND #PWR068
+L GND #PWR066
 U 1 1 59FD3A8B
 P 1925 6400
-F 0 "#PWR068" H 1925 6150 50  0001 C CNN
+F 0 "#PWR066" H 1925 6150 50  0001 C CNN
 F 1 "GND" H 1925 6250 50  0000 C CNN
 F 2 "" H 1925 6400 50  0001 C CNN
@@
 	4800 5800 4800 5600
 $Comp
-L GND #PWR069
+L GND #PWR067
 U 1 1 5A06EF81
 P 4350 6000
-F 0 "#PWR069" H 4350 5750 50  0001 C CNN
+F 0 "#PWR067" H 4350 5750 50  0001 C CNN
 F 1 "GND" H 4350 5850 50  0000 C CNN
 F 2 "" H 4350 6000 50  0001 C CNN
@@
 3V7
 $Comp
-L GND #PWR070
+L GND #PWR068
 U 1 1 5A075608
 P 5950 6450
-F 0 "#PWR070" H 5950 6200 50  0001 C CNN
+F 0 "#PWR068" H 5950 6200 50  0001 C CNN
 F 1 "GND" H 5950 6300 50  0000 C CNN
 F 2 "" H 5950 6450 50  0001 C CNN
@@
 Text Notes 5050 6825 0    60   ~ 0
 1V8 Regulator
-$Comp
-L Screw_Terminal_1x02 J?
-U 1 1 5A059A6F
+Wire Wire Line
+	8350 2725 8350 2775
+Connection ~ 10600 1775
+$Comp
+L Screw_Terminal_1x02_Bat J3
+U 1 1 5A054FA5
 P 8150 2875
-F 0 "J?" H 8150 3125 50  0000 C TNN
-F 1 "Screw_Terminal_1x02" V 8000 2875 50  0000 C TNN
+F 0 "J3" H 8150 3125 50  0000 C TNN
+F 1 "Screw_Terminal_1x02_Bat" V 8000 2875 50  0000 C TNN
 F 2 "Custom:1x2_Screw_Terminal_5mm_pitch" H 8150 2650 50  0001 C CNN
 F 3 "" H 8125 2875 50  0001 C CNN
@@
 $EndComp
 Wire Wire Line
-	8350 2725 8350 2775
-Wire Wire Line
-	8350 3025 8350 2975
+	8350 2975 8350 3025
+Wire Wire Line
+	8350 3025 8650 3025
+Connection ~ 8650 3025
+Wire Wire Line
+	8900 2725 8900 2625
+Wire Wire Line
+	8900 2625 9100 2625
+Connection ~ 8900 2725
 $EndSCHEMATC

Commit message: Assigned footprints to menial components
Parts:
- C25, C33, C35: footprint (none) -> Capacitors_SMD:C_0805
- C26, C27, C28, C29, C30, C31, C32, C34: footprint (none) -> Capacitors_SMD:C_0603
- D4, D5: footprint (none) -> Diodes_SMD:D_SOD-123
- D6, D7: footprint (none) -> LEDs:LED_0805
- L4, L5, L6: footprint (none) -> Inductors_SMD:L_0603
- R36, R37, R38, R39, R40, R41, R42, R43, R44, R45, R46: footprint (none) -> Resistors_SMD:R_0603
- U11: footprint (none) -> TO_SOT_Packages_SMD:SOT-23-5
Changed lines of the file:
@@
 F 0 "L6" V 2825 900 50  0000 C CNN
 F 1 "2.2uH" V 2950 900 50  0000 C CNN
-F 2 "" H 2875 900 50  0001 C CNN
+F 2 "Inductors_SMD:L_0603" H 2875 900 50  0001 C CNN
 F 3 "" H 2875 900 50  0001 C CNN
 	1    2875 900
@@
 F 0 "C30" H 3300 1150 50  0000 L CNN
 F 1 "4.7uF" H 3300 950 50  0000 L CNN
-F 2 "" H 3313 900 50  0001 C CNN
+F 2 "Capacitors_SMD:C_0603" H 3313 900 50  0001 C CNN
 F 3 "" H 3275 1050 50  0001 C CNN
 	1    3275 1050
@@
 F 0 "C25" H 950 1150 50  0000 L CNN
 F 1 "10uF" H 950 950 50  0000 L CNN
-F 2 "" H 963 900 50  0001 C CNN
+F 2 "Capacitors_SMD:C_0805" H 963 900 50  0001 C CNN
 F 3 "" H 925 1050 50  0001 C CNN
 	1    925  1050
@@
 F 0 "R40" V 9030 2425 50  0000 C CNN
 F 1 "10K" V 8950 2425 50  0000 C CNN
-F 2 "" V 8880 2425 50  0001 C CNN
+F 2 "Resistors_SMD:R_0603" V 8880 2425 50  0001 C CNN
 F 3 "" H 8950 2425 50  0001 C CNN
 	1    8950 2425
@@
 F 0 "C33" H 8675 2975 50  0000 L CNN
 F 1 "10uF" H 8675 2775 50  0000 L CNN
-F 2 "" H 8688 2725 50  0001 C CNN
+F 2 "Capacitors_SMD:C_0805" H 8688 2725 50  0001 C CNN
 F 3 "" H 8650 2875 50  0001 C CNN
 	1    8650 2875
@@
 F 0 "C34" H 8925 2125 50  0000 L CNN
 F 1 "1uF" H 8925 1925 50  0000 L CNN
-F 2 "" H 8938 1875 50  0001 C CNN
+F 2 "Capacitors_SMD:C_0603" H 8938 1875 50  0001 C CNN
 F 3 "" H 8900 2025 50  0001 C CNN
 	1    8900 2025
@@
 F 0 "R41" V 9730 3225 50  0000 C CNN
 F 1 "3.57K" V 9650 3225 50  0000 C CNN
-F 2 "" V 9580 3225 50  0001 C CNN
+F 2 "Resistors_SMD:R_0603" V 9580 3225 50  0001 C CNN
 F 3 "" H 9650 3225 50  0001 C CNN
 	1    9650 3225
@@
 F 0 "R43" V 9930 3225 50  0000 C CNN
 F 1 "2.94K" V 9850 3225 50  0000 C CNN
-F 2 "" V 9780 3225 50  0001 C CNN
+F 2 "Resistors_SMD:R_0603" V 9780 3225 50  0001 C CNN
 F 3 "" H 9850 3225 50  0001 C CNN
 	1    9850 3225
@@
 F 0 "R45" V 10130 3225 50  0000 C CNN
 F 1 "4.32K" V 10050 3225 50  0000 C CNN
-F 2 "" V 9980 3225 50  0001 C CNN
+F 2 "Resistors_SMD:R_0603" V 9980 3225 50  0001 C CNN
 F 3 "" H 10050 3225 50  0001 C CNN
 	1    10050 3225
@@
 F 0 "R46" V 10680 2825 50  0000 C CNN
 F 1 "56.2K" V 10600 2825 50  0000 C CNN
-F 2 "" V 10530 2825 50  0001 C CNN
+F 2 "Resistors_SMD:R_0603" V 10530 2825 50  0001 C CNN
 F 3 "" H 10600 2825 50  0001 C CNN
 	1    10600 2825
@@
 F 0 "C35" H 10775 1725 50  0000 L CNN
 F 1 "10uF" H 10775 1525 50  0000 L CNN
-F 2 "" H 10788 1475 50  0001 C CNN
+F 2 "Capacitors_SMD:C_0805" H 10788 1475 50  0001 C CNN
 F 3 "" H 10750 1625 50  0001 C CNN
 	1    10750 1625
@@
 F 0 "D6" H 9700 1225 50  0000 C CNN
 F 1 "LED" H 9700 1025 50  0000 C CNN
-F 2 "" H 9700 1125 50  0001 C CNN
+F 2 "LEDs:LED_0805" H 9700 1125 50  0001 C CNN
 F 3 "" H 9700 1125 50  0001 C CNN
 	1    9700 1125
@@
 F 0 "D7" H 10000 1225 50  0000 C CNN
 F 1 "LED" H 10000 1025 50  0000 C CNN
-F 2 "" H 10000 1125 50  0001 C CNN
+F 2 "LEDs:LED_0805" H 10000 1125 50  0001 C CNN
 F 3 "" H 10000 1125 50  0001 C CNN
 	1    10000 1125
@@
 F 0 "R42" V 9780 775 50  0000 C CNN
 F 1 "1.5K" V 9700 775 50  0000 C CNN
-F 2 "" V 9630 775 50  0001 C CNN
+F 2 "Resistors_SMD:R_0603" V 9630 775 50  0001 C CNN
 F 3 "" H 9700 775 50  0001 C CNN
 	1    9700 775
@@
 F 0 "R44" V 10080 775 50  0000 C CNN
 F 1 "1.5K" V 10000 775 50  0000 C CNN
-F 2 "" V 9930 775 50  0001 C CNN
+F 2 "Resistors_SMD:R_0603" V 9930 775 50  0001 C CNN
 F 3 "" H 10000 775 50  0001 C CNN
 	1    10000 775
@@
 F 0 "R36" V 2755 2975 50  0000 C CNN
 F 1 "3.01K" V 2675 2975 50  0000 C CNN
-F 2 "" V 2605 2975 50  0001 C CNN
+F 2 "Resistors_SMD:R_0603" V 2605 2975 50  0001 C CNN
 F 3 "" H 2675 2975 50  0001 C CNN
 	1    2675 2975
@@
 F 0 "R37" V 2755 3275 50  0000 C CNN
 F 1 "1K" V 2675 3275 50  0000 C CNN
-F 2 "" V 2605 3275 50  0001 C CNN
+F 2 "Resistors_SMD:R_0603" V 2605 3275 50  0001 C CNN
 F 3 "" H 2675 3275 50  0001 C CNN
 	1    2675 3275
@@
 F 0 "D4" H 2425 2675 50  0000 C CNN
 F 1 "D" H 2425 2475 50  0000 C CNN
-F 2 "" H 2425 2575 50  0001 C CNN
+F 2 "Diodes_SMD:D_SOD-123" H 2425 2575 50  0001 C CNN
 F 3 "" H 2425 2575 50  0001 C CNN
 	1    2425 2575
@@
 F 0 "L4" V 1875 2575 50  0000 C CNN
 F 1 "L" V 2000 2575 50  0000 C CNN
-F 2 "" H 1925 2575 50  0001 C CNN
+F 2 "Inductors_SMD:L_0603" H 1925 2575 50  0001 C CNN
 F 3 "" H 1925 2575 50  0001 C CNN
 	1    1925 2575
@@
 F 0 "C26" H 1200 3625 50  0000 L CNN
 F 1 "1uf" H 1200 3425 50  0000 L CNN
-F 2 "" H 1213 3375 50  0001 C CNN
+F 2 "Capacitors_SMD:C_0603" H 1213 3375 50  0001 C CNN
 F 3 "" H 1175 3525 50  0001 C CNN
 	1    1175 3525
@@
 F 0 "C28" H 3000 3225 50  0000 L CNN
 F 1 "1uF" H 3000 3025 50  0000 L CNN
-F 2 "" H 3013 2975 50  0001 C CNN
+F 2 "Capacitors_SMD:C_0603" H 3013 2975 50  0001 C CNN
 F 3 "" H 2975 3125 50  0001 C CNN
 	1    2975 3125
@@
 F 0 "R38" V 2755 5550 50  0000 C CNN
 F 1 "20K" V 2675 5550 50  0000 C CNN
-F 2 "" V 2605 5550 50  0001 C CNN
+F 2 "Resistors_SMD:R_0603" V 2605 5550 50  0001 C CNN
 F 3 "" H 2675 5550 50  0001 C CNN
 	1    2675 5550
@@
 F 0 "R39" V 2755 5850 50  0000 C CNN
 F 1 "1K" V 2675 5850 50  0000 C CNN
-F 2 "" V 2605 5850 50  0001 C CNN
+F 2 "Resistors_SMD:R_0603" V 2605 5850 50  0001 C CNN
 F 3 "" H 2675 5850 50  0001 C CNN
 	1    2675 5850
@@
 F 0 "U11" H 1925 6050 60  0000 C CNN
 F 1 "AP3012" H 1925 5700 60  0000 C CNN
-F 2 "" H 1925 5700 60  0001 C CNN
+F 2 "TO_SOT_Packages_SMD:SOT-23-5" H 1925 5700 60  0001 C CNN
 F 3 "" H 1925 5700 60  0001 C CNN
 	1    1925 5700
@@
 F 0 "D5" H 2425 5250 50  0000 C CNN
 F 1 "D" H 2425 5050 50  0000 C CNN
-F 2 "" H 2425 5150 50  0001 C CNN
+F 2 "Diodes_SMD:D_SOD-123" H 2425 5150 50  0001 C CNN
 F 3 "" H 2425 5150 50  0001 C CNN
 	1    2425 5150
@@
 F 0 "L5" V 1875 5150 50  0000 C CNN
 F 1 "L" V 2000 5150 50  0000 C CNN
-F 2 "" H 1925 5150 50  0001 C CNN
+F 2 "Inductors_SMD:L_0603" H 1925 5150 50  0001 C CNN
 F 3 "" H 1925 5150 50  0001 C CNN
 	1    1925 5150
@@
 F 0 "C27" H 1200 6200 50  0000 L CNN
 F 1 "1uf" H 1200 6000 50  0000 L CNN
-F 2 "" H 1213 5950 50  0001 C CNN
+F 2 "Capacitors_SMD:C_0603" H 1213 5950 50  0001 C CNN
 F 3 "" H 1175 6100 50  0001 C CNN
 	1    1175 6100
@@
 F 0 "C29" H 3000 5800 50  0000 L CNN
 F 1 "1uF" H 3000 5600 50  0000 L CNN
-F 2 "" H 3013 5550 50  0001 C CNN
+F 2 "Capacitors_SMD:C_0603" H 3013 5550 50  0001 C CNN
 F 3 "" H 2975 5700 50  0001 C CNN
 	1    2975 5700
@@
 F 0 "C31" H 4375 5850 50  0000 L CNN
 F 1 "1uF" H 4375 5650 50  0000 L CNN
-F 2 "" H 4388 5600 50  0001 C CNN
+F 2 "Capacitors_SMD:C_0603" H 4388 5600 50  0001 C CNN
 F 3 "" H 4350 5750 50  0001 C CNN
 	1    4350 5750
@@
 F 0 "C32" H 6175 6300 50  0000 L CNN
 F 1 "1uF" H 6175 6100 50  0000 L CNN
-F 2 "" H 6188 6050 50  0001 C CNN
+F 2 "Capacitors_SMD:C_0603" H 6188 6050 50  0001 C CNN
 F 3 "" H 6150 6200 50  0001 C CNN
 	1    6150 6200

Commit message: all associated
Parts:
- removed D4, D5: D, Diodes_SMD:D_SOD-123, symbol D
- added D4, D5: 1N5819, Diodes_SMD:D_SOD-123, symbol D_Schottky
- L4, L5: value L -> 10uH
Connections:
- net 26V: now also D5.1 (K)
- net 5V: now also D4.1 (K)
- net at L4.1, U10.1 (SW): now also D4.2 (A)
- net at L5.1, U11.1 (SW): now also D5.2 (A)
Changed lines of the file:
@@
 	1300 900  1300 1050
 $Comp
-L GND #PWR057
+L GND #PWR57
 U 1 1 59FB2340
 P 925 1325
-F 0 "#PWR057" H 925 1075 50  0001 C CNN
+F 0 "#PWR57" H 925 1075 50  0001 C CNN
 F 1 "GND" H 925 1175 50  0000 C CNN
 F 2 "" H 925 1325 50  0001 C CNN
@@
 	925  1200 925  1325
 $Comp
-L GND #PWR058
+L GND #PWR60
 U 1 1 59FB2347
 P 2600 1300
-F 0 "#PWR058" H 2600 1050 50  0001 C CNN
+F 0 "#PWR60" H 2600 1050 50  0001 C CNN
 F 1 "GND" H 2600 1150 50  0000 C CNN
 F 2 "" H 2600 1300 50  0001 C CNN
@@
 	2600 1300 2600 1200
 $Comp
-L GND #PWR059
+L GND #PWR61
 U 1 1 59FB234E
 P 3275 1300
-F 0 "#PWR059" H 3275 1050 50  0001 C CNN
+F 0 "#PWR61" H 3275 1050 50  0001 C CNN
 F 1 "GND" H 3275 1150 50  0000 C CNN
 F 2 "" H 3275 1300 50  0001 C CNN
@@
 $EndComp
 $Comp
-L GND #PWR060
+L GND #PWR65
 U 1 1 59FB392A
 P 8700 2425
-F 0 "#PWR060" H 8700 2175 50  0001 C CNN
+F 0 "#PWR65" H 8700 2175 50  0001 C CNN
 F 1 "GND" H 8700 2275 50  0000 C CNN
 F 2 "" H 8700 2425 50  0001 C CNN
@@
 $EndComp
 $Comp
-L GND #PWR061
+L GND #PWR64
 U 1 1 59FB394B
 P 8650 3175
-F 0 "#PWR061" H 8650 2925 50  0001 C CNN
+F 0 "#PWR64" H 8650 2925 50  0001 C CNN
 F 1 "GND" H 8650 3025 50  0000 C CNN
 F 2 "" H 8650 3175 50  0001 C CNN
@@
 $EndComp
 $Comp
-L GND #PWR062
+L GND #PWR66
 U 1 1 59FB396D
 P 9650 3375
-F 0 "#PWR062" H 9650 3125 50  0001 C CNN
+F 0 "#PWR66" H 9650 3125 50  0001 C CNN
 F 1 "GND" H 9650 3225 50  0000 C CNN
 F 2 "" H 9650 3375 50  0001 C CNN
@@
 $EndComp
 $Comp
-L GND #PWR063
+L GND #PWR68
 U 1 1 59FB397A
 P 10750 2475
-F 0 "#PWR063" H 10750 2225 50  0001 C CNN
+F 0 "#PWR68" H 10750 2225 50  0001 C CNN
 F 1 "GND" H 10750 2325 50  0000 C CNN
 F 2 "" H 10750 2475 50  0001 C CNN
@@
 $EndComp
 $Comp
-L GND #PWR064
+L GND #PWR67
 U 1 1 59FB3987
 P 10550 1475
-F 0 "#PWR064" H 10550 1225 50  0001 C CNN
+F 0 "#PWR67" H 10550 1225 50  0001 C CNN
 F 1 "GND" H 10550 1325 50  0000 C CNN
 F 2 "" H 10550 1475 50  0001 C CNN
@@
 $EndComp
 $Comp
-L D D4
-U 1 1 59FB48FA
-P 2425 2575
-F 0 "D4" H 2425 2675 50  0000 C CNN
-F 1 "D" H 2425 2475 50  0000 C CNN
-F 2 "Diodes_SMD:D_SOD-123" H 2425 2575 50  0001 C CNN
-F 3 "" H 2425 2575 50  0001 C CNN
-	1    2425 2575
-	-1   0    0    1
-$EndComp
-$Comp
 L L L4
 U 1 1 59FB4901
 P 1925 2575
 F 0 "L4" V 1875 2575 50  0000 C CNN
-F 1 "L" V 2000 2575 50  0000 C CNN
+F 1 "10uH" V 2000 2575 50  0000 C CNN
 F 2 "Inductors_SMD:L_0603" H 1925 2575 50  0001 C CNN
 F 3 "" H 1925 2575 50  0001 C CNN
@@
 Connection ~ 2975 2575
 $Comp
-L GND #PWR065
+L GND #PWR58
 U 1 1 59FB4920
 P 1925 3825
-F 0 "#PWR065" H 1925 3575 50  0001 C CNN
+F 0 "#PWR58" H 1925 3575 50  0001 C CNN
 F 1 "GND" H 1925 3675 50  0000 C CNN
 F 2 "" H 1925 3825 50  0001 C CNN
@@
 $EndComp
 $Comp
-L D D5
-U 1 1 59FD3A6C
-P 2425 5150
-F 0 "D5" H 2425 5250 50  0000 C CNN
-F 1 "D" H 2425 5050 50  0000 C CNN
-F 2 "Diodes_SMD:D_SOD-123" H 2425 5150 50  0001 C CNN
-F 3 "" H 2425 5150 50  0001 C CNN
-	1    2425 5150
-	-1   0    0    1
-$EndComp
-$Comp
 L L L5
 U 1 1 59FD3A72
 P 1925 5150
 F 0 "L5" V 1875 5150 50  0000 C CNN
-F 1 "L" V 2000 5150 50  0000 C CNN
+F 1 "10uH" V 2000 5150 50  0000 C CNN
 F 2 "Inductors_SMD:L_0603" H 1925 5150 50  0001 C CNN
 F 3 "" H 1925 5150 50  0001 C CNN
@@
 Connection ~ 2975 5150
 $Comp
-L GND #PWR066
+L GND #PWR59
 U 1 1 59FD3A8B
 P 1925 6400
-F 0 "#PWR066" H 1925 6150 50  0001 C CNN
+F 0 "#PWR59" H 1925 6150 50  0001 C CNN
 F 1 "GND" H 1925 6250 50  0000 C CNN
 F 2 "" H 1925 6400 50  0001 C CNN
@@
 	4800 5800 4800 5600
 $Comp
-L GND #PWR067
+L GND #PWR62
 U 1 1 5A06EF81
 P 4350 6000
-F 0 "#PWR067" H 4350 5750 50  0001 C CNN
+F 0 "#PWR62" H 4350 5750 50  0001 C CNN
 F 1 "GND" H 4350 5850 50  0000 C CNN
 F 2 "" H 4350 6000 50  0001 C CNN
@@
 3V7
 $Comp
-L GND #PWR068
+L GND #PWR63
 U 1 1 5A075608
 P 5950 6450
-F 0 "#PWR068" H 5950 6200 50  0001 C CNN
+F 0 "#PWR63" H 5950 6200 50  0001 C CNN
 F 1 "GND" H 5950 6300 50  0000 C CNN
 F 2 "" H 5950 6450 50  0001 C CNN
@@
 	8900 2625 9100 2625
 Connection ~ 8900 2725
+$Comp
+L D_Schottky D4
+U 1 1 5A07B3FC
+P 2425 2575
+F 0 "D4" H 2425 2675 50  0000 C CNN
+F 1 "1N5819" H 2425 2475 50  0000 C CNN
+F 2 "Diodes_SMD:D_SOD-123" H 2425 2575 50  0001 C CNN
+F 3 "" H 2425 2575 50  0001 C CNN
+	1    2425 2575
+	-1   0    0    1
+$EndComp
+$Comp
+L D_Schottky D5
+U 1 1 5A07B848
+P 2425 5150
+F 0 "D5" H 2425 5250 50  0000 C CNN
+F 1 "1N5819" H 2425 5050 50  0000 C CNN
+F 2 "Diodes_SMD:D_SOD-123" H 2425 5150 50  0001 C CNN
+F 3 "" H 2425 5150 50  0001 C CNN
+	1    2425 5150
+	-1   0    0    1
+$EndComp
 $EndSCHEMATC
