File: ultrasonic_localization/soundModule.sch (KiCad schematic (older format))
At the start: 36 parts

Commit message: ultrasonic figured out
Connections:
- net TX?OUT1 is gone; now on net SW?b: U?.14 (T1OUT)
- net TX?OUT2 is gone; now on net GND: U?.7 (T2OUT)
- net GND: now also U?.2
- net SW1 renamed SW?b
- net SW2 renamed SW?a
- net TX?IN1 renamed TX?a
- net TX?IN2 renamed TX?b
Changed lines of the file:
@@
 $Descr A4 11693 8268
 encoding utf-8
-Sheet 1 2
+Sheet 2 3
 Title ""
 Date ""
@@
 	1    0    0    -1
 $EndComp
-Text HLabel 9800 5100 2    60   Output ~ 0
-TX?OUT1
-Text HLabel 9800 5300 2    60   Output ~ 0
-TX?OUT2
 $Comp
 L GND #PWR?
 U 1 1 59FB1823
-P 2000 1575
-F 0 "#PWR?" H 2000 1325 50  0001 C CNN
-F 1 "GND" H 2000 1425 50  0000 C CNN
-F 2 "" H 2000 1575 50  0001 C CNN
-F 3 "" H 2000 1575 50  0001 C CNN
-	1    2000 1575
-	1    0    0    -1
-$EndComp
-Text HLabel 8200 5100 0    60   Input ~ 0
-TX?IN1
-Text HLabel 8200 5300 0    60   Input ~ 0
-TX?IN2
+P 1025 2725
+F 0 "#PWR?" H 1025 2475 50  0001 C CNN
+F 1 "GND" H 1025 2575 50  0000 C CNN
+F 2 "" H 1025 2725 50  0001 C CNN
+F 3 "" H 1025 2725 50  0001 C CNN
+	1    1025 2725
+	1    0    0    -1
+$EndComp
 $Comp
 L MAX232 U?
@@
 	4300 1075 4125 1075
 Wire Wire Line
-	4300 625  4300 1525
+	4300 625  4300 800
+Wire Wire Line
+	4300 800  4300 1075
+Wire Wire Line
+	4300 1075 4300 1525
 Wire Wire Line
 	4125 800  4300 800
@@
 	3650 1425 3700 1425
 Wire Wire Line
-	3650 800  3650 1425
+	3650 800  3650 1075
+Wire Wire Line
+	3650 1075 3650 1425
 Wire Wire Line
 	3650 1075 3825 1075
@@
 Connection ~ 3050 1425
 Wire Wire Line
-	3350 625  3350 1575
+	3350 625  3350 1425
+Wire Wire Line
+	3350 1425 3350 1575
 Wire Wire Line
 	4300 625  3650 625
@@
 Connection ~ 1300 1025
 Wire Wire Line
-	750  1025 1425 1025
-Wire Wire Line
-	3050 925  3050 1525
+	750  1025 1025 1025
+Wire Wire Line
+	1025 1025 1300 1025
+Wire Wire Line
+	1300 1025 1425 1025
+Wire Wire Line
+	3050 925  3050 1425
+Wire Wire Line
+	3050 1425 3050 1525
 Wire Wire Line
 	3050 925  2900 925
@@
 	5275 925  5325 925
 Wire Wire Line
-	5875 925  5875 1525
+	5875 925  5875 1425
+Wire Wire Line
+	5875 1425 5875 1525
 Wire Wire Line
 	5875 925  5625 925
@@
 	3350 1875 3350 2025
 Wire Wire Line
-	750  1325 1300 1325
+	750  1325 1025 1325
+Wire Wire Line
+	1025 1325 1300 1325
 Connection ~ 1025 1325
 Connection ~ 1025 1025
 Wire Wire Line
-	6200 950  7875 950
+	6200 950  7575 950
+Wire Wire Line
+	7575 950  7875 950
 Wire Wire Line
 	7875 950  7875 1450
@@
 	7875 1450 8025 1450
 Wire Wire Line
-	5275 1925 5275 2175
-Wire Wire Line
-	4900 2325 5100 2325
+	5275 1925 5275 2025
+Wire Wire Line
+	5275 2025 5275 2175
+Wire Wire Line
+	4900 2325 5000 2325
+Wire Wire Line
+	5000 2325 5100 2325
 Connection ~ 5000 2325
 Wire Wire Line
-	4900 2025 6250 2025
+	4900 2025 5100 2025
+Wire Wire Line
+	5100 2025 5275 2025
+Wire Wire Line
+	5275 2025 6250 2025
 Connection ~ 5275 2025
 Connection ~ 5100 2025
@@
 Connection ~ 7575 950
 Wire Wire Line
-	1850 1575 2000 1575
-Wire Wire Line
-	9000 3800 10250 3800
+	9000 3800 9600 3800
+Wire Wire Line
+	9600 3800 10250 3800
 Wire Wire Line
 	10250 3800 10250 4300
@@
 Connection ~ 6200 950
 Wire Wire Line
-	6175 1425 6250 1425
+	6175 1425 6200 1425
+Wire Wire Line
+	6200 1425 6250 1425
 Connection ~ 5875 1425
 Wire Wire Line
@@
 	6850 1525 7275 1525
 Text HLabel 1025 1975 0    60   Input ~ 0
-SW1
+SW?b
 Text HLabel 1850 1425 0    60   Input ~ 0
-SW2
+SW?a
 $Comp
 L TCT40-16R/T U?
@@
 	0    1    1    0
 $EndComp
+Text HLabel 8200 5300 0    60   Input ~ 0
+TX?b
+Text HLabel 8200 5100 0    60   Input ~ 0
+TX?a
+Text Label 9800 5100 0    60   ~ 0
+TX1
+Text Label 9800 5300 0    60   ~ 0
+TX2
+Text Label 1025 1975 0    60   ~ 0
+TX1
+Text Label 1025 2725 0    60   ~ 0
+TX2
 $EndSCHEMATC

Commit message: organization
Parts:
- gave numbers to parts that had none: 33
Connections:
- net SIG? renamed SIG
- net SW?a renamed SWa
- net SW?b renamed SWb
- net THRESH? renamed THRESH
- net TX?a renamed TXa
- net TX?b renamed TXb
Other:
- note added: "TX : Prone To Change"
- note removed: "TX"
- moved on the sheet: C13, C14, C15, C16, C17, C18, C19, C20, C21, C22, C23, C24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

Commit message: refactored power
Parts:
- renumbered C15 to C?, C18 to C?, C17 to C?, C16 to C?, C19 to C?, C14 to C?, C13 to C?, C20 to C?, C21 to C?, C22 to C?, C23 to C?, C24 to C?, Q1 to Q?, R16 to R?, R15 to R?, R17 to R?, R18 to R?, R19 to R?, R13 to R?, R14 to R?, R20 to R?, R24 to R?, R25 to R?, R22 to R?, R28 to R?, R29 to R?, R27 to R?, R26 to R?, R23 to R?, R21 to R?, U10 to U?, U9 to U?, U11 to U?
Connections:
- net VGND: now also U?.3 (+), U?.3 (+); no longer U?.10 (+), U?.5 (+)
- net at C?.1, C?.2, R?.1: now also U?.2 (-); no longer U?.6 (-)
- net at C?.2, C?.2, R?.1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: now also U?.1; no longer U?.7
- net at R?.2, R?.2: now also U?.1; no longer U?.8
- net at C?.2, R?.1: now also U?.2 (-); no longer U?.9 (-)
- net at R?.1, R?.2: now also U?.3 (+); no longer U?.12 (+)
- net at C?.1, R?.1, R?.1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: now also U?.2 (-); no longer U?.13 (-)
- net at R?.1: now also U?.1; no longer U?.14

Commit message: schematic review version
Parts:
- added D? (x2): D, symbol D
- added R?: R, symbol R
Connections:
- net GND: now also D?.1 (K), D?.2 (A), R?.1; no longer U?.2, U?.7 (T2OUT)
- net SWa: now also D?.1 (K)
- new net TX2: R?.2, U?.2, U?.7 (T2OUT)
Other:
- note added: "Amplify to 30V"
Changed lines of the file:
@@
 L GND #PWR?
 U 1 1 59FB1823
-P 2350 1525
-F 0 "#PWR?" H 2350 1275 50  0001 C CNN
-F 1 "GND" H 2350 1375 50  0000 C CNN
-F 2 "" H 2350 1525 50  0001 C CNN
-F 3 "" H 2350 1525 50  0001 C CNN
-	1    2350 1525
+P 2350 1825
+F 0 "#PWR?" H 2350 1575 50  0001 C CNN
+F 1 "GND" H 2350 1675 50  0000 C CNN
+F 2 "" H 2350 1825 50  0001 C CNN
+F 3 "" H 2350 1825 50  0001 C CNN
+	1    2350 1825
 	1    0    0    -1
 $EndComp
@@
 Text HLabel 2350 775  0    60   Input ~ 0
 SWb
-Text HLabel 1075 3150 0    60   Input ~ 0
+Text HLabel 650  2900 1    60   Input ~ 0
 SWa
 $Comp
@@
 Text Label 2350 1525 0    60   ~ 0
 TX2
+$Comp
+L D D?
+U 1 1 59FBB6AA
+P 875 3300
+F 0 "D?" H 875 3400 50  0000 C CNN
+F 1 "D" H 875 3200 50  0000 C CNN
+F 2 "" H 875 3300 50  0001 C CNN
+F 3 "" H 875 3300 50  0001 C CNN
+	1    875  3300
+	0    -1   -1   0
+$EndComp
+Wire Wire Line
+	650  2900 650  3150
+Wire Wire Line
+	650  3150 1075 3150
+$Comp
+L D D?
+U 1 1 59FBB896
+P 1075 3300
+F 0 "D?" H 1075 3400 50  0000 C CNN
+F 1 "D" H 1075 3200 50  0000 C CNN
+F 2 "" H 1075 3300 50  0001 C CNN
+F 3 "" H 1075 3300 50  0001 C CNN
+	1    1075 3300
+	0    1    1    0
+$EndComp
+Connection ~ 650  3150
+$Comp
+L GND #PWR?
+U 1 1 59FBBAD1
+P 1075 3450
+F 0 "#PWR?" H 1075 3200 50  0001 C CNN
+F 1 "GND" H 1075 3300 50  0000 C CNN
+F 2 "" H 1075 3450 50  0001 C CNN
+F 3 "" H 1075 3450 50  0001 C CNN
+	1    1075 3450
+	1    0    0    -1
+$EndComp
+Text Notes 9925 2525 0    60   ~ 0
+Amplify to 30V
+Connection ~ 875  3450
+$Comp
+L R R?
+U 1 1 59FBFEDB
+P 2350 1675
+F 0 "R?" V 2430 1675 50  0000 C CNN
+F 1 "R" V 2350 1675 50  0000 C CNN
+F 2 "" V 2280 1675 50  0001 C CNN
+F 3 "" H 2350 1675 50  0001 C CNN
+	1    2350 1675
+	-1   0    0    1
+$EndComp
+Wire Wire Line
+	875  3450 1075 3450
 $EndSCHEMATC

Commit message: finished ultrasound and some other stuff
Parts:
- removed C? (x4): 150nF, symbol C
- removed U?: MAX232, symbol MAX232
Connections:
- net TX2 is gone; now on net TXb: R?.2, U?.2
- no-connect marks 4 -> 0
Other:
- note removed: "Amplify to 30V"
- note removed: "TX : Prone To Change"
- moved on the sheet: C?, D?, Q?, R?, U?A

Commit message: added osc src
Parts:
- R?: value R -> 10K
Other:
- note added: "TODO - Fill Values\nCheck VGND"
- note added: "VGND?"
- moved on the sheet: R?, U?
Changed lines of the file:
@@
 L GND #PWR?
 U 1 1 59FB1823
-P 2350 1825
+P 4450 2000
 AR Path="/59FBBECF/59FB1823" Ref="#PWR?"  Part="1"
 AR Path="/59FBFC85/59FB1823" Ref="#PWR?"  Part="1"
 AR Path="/59FBAACD/59FB1823" Ref="#PWR?"  Part="1"
-F 0 "#PWR?" H 2350 1575 50  0001 C CNN
-F 1 "GND" H 2350 1675 50  0000 C CNN
-F 2 "" H 2350 1825 50  0001 C CNN
-F 3 "" H 2350 1825 50  0001 C CNN
-	1    2350 1825
+F 0 "#PWR?" H 4450 1750 50  0001 C CNN
+F 1 "GND" H 4450 1850 50  0000 C CNN
+F 2 "" H 4450 2000 50  0001 C CNN
+F 3 "" H 4450 2000 50  0001 C CNN
+	1    4450 2000
 	1    0    0    -1
 $EndComp
@@
 Wire Wire Line
 	8050 4225 8475 4225
-Text HLabel 2350 775  0    60   Input ~ 0
+Text HLabel 4450 950  0    60   Input ~ 0
 SWb
 Text HLabel 2625 3875 1    60   Input ~ 0
@@
 L TCT40-16R/T U?
 U 1 1 59FAA88E
-P 2350 1150
+P 4450 1325
 AR Path="/59FBBECF/59FAA88E" Ref="U?"  Part="1"
 AR Path="/59FBFC85/59FAA88E" Ref="U?"  Part="1"
 AR Path="/59FBAACD/59FAA88E" Ref="U?"  Part="1"
-F 0 "U?" H 2350 1150 60  0000 C CNN
-F 1 "TCT40-16R/T" H 2350 1425 60  0000 C CNN
-F 2 "" H 2350 1150 60  0001 C CNN
-F 3 "" H 2350 1150 60  0001 C CNN
-	1    2350 1150
+F 0 "U?" H 4450 1325 60  0000 C CNN
+F 1 "TCT40-16R/T" H 4450 1600 60  0000 C CNN
+F 2 "" H 4450 1325 60  0001 C CNN
+F 3 "" H 4450 1325 60  0001 C CNN
+	1    4450 1325
 	0    1    1    0
 $EndComp
-Text HLabel 2350 1525 0    60   Input ~ 0
+Text HLabel 4450 1700 0    60   Input ~ 0
 TXb
-Text HLabel 2350 675  0    60   Input ~ 0
+Text HLabel 4450 850  0    60   Input ~ 0
 TXa
-Text Label 2350 775  0    60   ~ 0
+Text Label 4450 950  0    60   ~ 0
 TX1
-Text Label 2350 1525 0    60   ~ 0
+Text Label 4450 1700 0    60   ~ 0
 TX2
 $Comp
@@
 L R R?
 U 1 1 59FBFEDB
-P 2350 1675
+P 4450 1850
 AR Path="/59FBBECF/59FBFEDB" Ref="R?"  Part="1"
 AR Path="/59FBFC85/59FBFEDB" Ref="R?"  Part="1"
 AR Path="/59FBAACD/59FBFEDB" Ref="R?"  Part="1"
-F 0 "R?" V 2430 1675 50  0000 C CNN
-F 1 "R" V 2350 1675 50  0000 C CNN
-F 2 "" V 2280 1675 50  0001 C CNN
-F 3 "" H 2350 1675 50  0001 C CNN
-	1    2350 1675
+F 0 "R?" V 4530 1850 50  0000 C CNN
+F 1 "10K" V 4450 1850 50  0000 C CNN
+F 2 "" V 4380 1850 50  0001 C CNN
+F 3 "" H 4450 1850 50  0001 C CNN
+	1    4450 1850
 	-1   0    0    1
 $EndComp
@@
 	2850 4425 3050 4425
 Wire Wire Line
-	2350 775  2350 675
+	4450 950  4450 850
+Text Notes 2925 4700 0    60   ~ 0
+VGND?
+Text Notes 3100 3200 0    60   ~ 0
+TODO - Fill Values\nCheck VGND
 $EndSCHEMATC

Commit message: sim + analysis for 40kHz filter
Parts:
- removed D? (x2): D, symbol D
- C46, C50, C51: renamed from C?; value C -> 10nF
- C47, C48: renamed from C?; value C -> 1nF
- C49: renamed from C?; value C -> 12pF
- R67, R73: renamed from R?; value R -> 10K
- R68: renamed from R?; value R -> 62K
- R69: renamed from R?; value R -> 660
- R71: renamed from R?; value R -> 1K
- R72: renamed from R?; value R -> 40K
- R74: renamed from R?; value R -> 3.3M
- R75: renamed from R?; value R -> 120K
- R76, R77: renamed from R?; value R -> 75K
- gave numbers to parts that had none: 13
Connections:
- net SWa: now also U18.1; no longer R67.2
- net SWb: now also R67.2; no longer U18.1
- net VGND: now also U17.10 (+), U17.5 (+); no longer U17.3 (+), U17.3 (+)
- net at C47.2, C49.2, R72.2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: now also U17.7; no longer U17.1
- net at C48.2, C49.1, R72.1: now also U17.6 (-); no longer U17.2 (-)
- net at R77.2, R78.2: now also U17.8; no longer U17.1
- net at C50.2, R77.1: now also U17.9 (-); no longer U17.2 (-)
- net at R81.1: now also U17.14; no longer U17.1
- net at C51.1, R74.1, R75.2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: now also U17.13 (-); no longer U17.2 (-)
- net at R78.1, R80.2: now also U17.12 (+); no longer U17.3 (+)
Other:
- note added: "TODO : diode?\n"
- note added: "TODO : investigate thresh utility"
- note removed: "TODO - Fill Values\nCheck VGND"
- note removed: "VGND?"
- moved on the sheet: C38, C39, C40, C41, C42, C43, Q3, R49, R50, R51, R53, R54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
