File: ultrasonic_localization/soundModule.sch (KiCad schematic (older format))
At the start: 29 parts, among them Q4 BC847, U17 LM324, U18 TCT40-16R/T

Commit message: IMU pulldown
Parts:
- added D? (x2): D, symbol D
Connections:
- net GND: now also D?.1 (K), D?.2 (A)
Other:
- note added: "TODO : In LTSpice sim, adjusting THRESH doesn't seem to do anything,\nwhereas it should have set reception sensitivity.\nSee https://uglyduck.ath.cx/ep/archive/2014/01/Making_a_better_HC_SR04_Echo_Locator.html For Reference"
- note added: "TODO : Need a diode??"
- note removed: "TODO : diode?\n"
- note removed: "TODO : investigate thresh utility"

Commit message: Assigned many footprints to things
Parts:
- R67: footprint (none) -> Resistors_SMD:R_0603
- U17: footprint (none) -> Housings_SOIC:SOIC-16_3.9x9.9mm_Pitch1.27mm
- U18: footprint (none) -> TCT40-16R_T:TCT40-16R_T
Connections:
- net +5V: now also U17.11 (V-); no longer U17.4 (V+)
- net GND: now also U17.4 (V+); no longer U17.11 (V-)
Changed lines of the file:
@@
 F 0 "U15" H 3100 4175 50  0000 L CNN
 F 1 "LM324" H 3100 3775 50  0000 L CNN
-F 2 "" H 3050 4075 50  0001 C CNN
+F 2 "Housings_SOIC:SOIC-16_3.9x9.9mm_Pitch1.27mm" H 3050 4075 50  0001 C CNN
 F 3 "" H 3150 4175 50  0001 C CNN
 	1    3100 3975
@@
 F 0 "U15" H 4350 4175 50  0000 L CNN
 F 1 "LM324" H 4350 3775 50  0000 L CNN
-F 2 "" H 4300 4075 50  0001 C CNN
+F 2 "Housings_SOIC:SOIC-16_3.9x9.9mm_Pitch1.27mm" H 4300 4075 50  0001 C CNN
 F 3 "" H 4400 4175 50  0001 C CNN
 	2    4350 3975
@@
 F 0 "U15" H 5925 4175 50  0000 L CNN
 F 1 "LM324" H 5925 3775 50  0000 L CNN
-F 2 "" H 5875 4075 50  0001 C CNN
+F 2 "Housings_SOIC:SOIC-16_3.9x9.9mm_Pitch1.27mm" H 5875 4075 50  0001 C CNN
 F 3 "" H 5975 4175 50  0001 C CNN
 	3    5925 3975
@@
 F 0 "R49" V 2430 3875 50  0000 C CNN
 F 1 "10K" V 2350 3875 50  0000 C CNN
-F 2 "" V 2280 3875 50  0001 C CNN
+F 2 "Resistors_SMD:R_0603" V 2280 3875 50  0001 C CNN
 F 3 "" H 2350 3875 50  0001 C CNN
 	1    2350 3875
@@
 $EndComp
 $Comp
-L GND #PWR092
-U 1 1 59FAA379
-P 6800 4275
-AR Path="/59FBBECF/59FAA379" Ref="#PWR092"  Part="1"
-AR Path="/59FBFC85/59FAA379" Ref="#PWR050"  Part="1"
-AR Path="/59FBAACD/59FAA379" Ref="#PWR077"  Part="1"
-AR Path="/59FBC20F/59FAA379" Ref="#PWR0107"  Part="1"
-F 0 "#PWR077" H 6800 4025 50  0001 C CNN
-F 1 "GND" H 6800 4125 50  0000 C CNN
-F 2 "" H 6800 4275 50  0001 C CNN
-F 3 "" H 6800 4275 50  0001 C CNN
-	1    6800 4275
-	1    0    0    -1
-$EndComp
-$Comp
 L +5V #PWR093
 U 1 1 59FAA3C0
@@
 L +5V #PWR095
 U 1 1 59FAA430
-P 6800 3675
+P 6650 4275
 AR Path="/59FBBECF/59FAA430" Ref="#PWR095"  Part="1"
 AR Path="/59FBFC85/59FAA430" Ref="#PWR053"  Part="1"
 AR Path="/59FBAACD/59FAA430" Ref="#PWR080"  Part="1"
 AR Path="/59FBC20F/59FAA430" Ref="#PWR0110"  Part="1"
-F 0 "#PWR080" H 6800 3525 50  0001 C CNN
-F 1 "+5V" H 6675 3675 50  0000 C CNN
-F 2 "" H 6800 3675 50  0001 C CNN
-F 3 "" H 6800 3675 50  0001 C CNN
-	1    6800 3675
+F 0 "#PWR080" H 6650 4125 50  0001 C CNN
+F 1 "+5V" H 6525 4275 50  0000 C CNN
+F 2 "" H 6650 4275 50  0001 C CNN
+F 3 "" H 6650 4275 50  0001 C CNN
+	1    6650 4275
 	1    0    0    -1
 $EndComp
@@
 F 0 "U15" H 6900 4175 50  0000 L CNN
 F 1 "LM324" H 6900 3775 50  0000 L CNN
-F 2 "" H 6850 4075 50  0001 C CNN
+F 2 "Housings_SOIC:SOIC-16_3.9x9.9mm_Pitch1.27mm" H 6850 4075 50  0001 C CNN
 F 3 "" H 6950 4175 50  0001 C CNN
 	4    6900 3975
@@
 F 0 "U16" H 4450 1325 60  0000 C CNN
 F 1 "TCT40-16R/T" H 4450 1600 60  0000 C CNN
-F 2 "" H 4450 1325 60  0001 C CNN
+F 2 "TCT40-16R_T:TCT40-16R_T" H 4450 1325 60  0001 C CNN
 F 3 "" H 4450 1325 60  0001 C CNN
 	1    4450 1325
@@
 	1    0    0    -1
 $EndComp
+Wire Wire Line
+	6650 4275 6800 4275
+$Comp
+L GND #PWR?
+U 1 1 5A068EAF
+P 7250 3675
+F 0 "#PWR?" H 7250 3425 50  0001 C CNN
+F 1 "GND" H 7250 3525 50  0000 C CNN
+F 2 "" H 7250 3675 50  0001 C CNN
+F 3 "" H 7250 3675 50  0001 C CNN
+	1    7250 3675
+	1    0    0    -1
+$EndComp
+Wire Wire Line
+	6800 3675 7250 3675
 $EndSCHEMATC

Commit message: almost resolved DRC
Parts:
- gave numbers to parts that had none: 2
Connections:
- net +5V: now also U17.4 (V+), U17.4 (V+), U17.4 (V+), U17.4 (V+); no longer U17.11 (V-), U17.11 (V-), U17.11 (V-), U17.11 (V-)
- net GND: now also U17.11 (V-), U17.11 (V-), U17.11 (V-), U17.11 (V-); no longer U17.4 (V+), U17.4 (V+), U17.4 (V+), U17.4 (V+)
- net SWb: now also D2.1 (K), D3.2 (A)
Other:
- note added: "Consider Gain-Bandwidth Tradeoff"

Commit message: Assigned footprints to menial components
Parts:
- C44, C45, C46, C47, C48, C49, C50, C51: footprint (none) -> Capacitors_SMD:C_0603
- D2, D3: footprint (none) -> Diodes_SMD:D_SOD-123
- R65, R66, R68, R69, R70, R71, R72, R73, R74, R75, R76, R77, R78, R79, R80, R81, R82: footprint (none) -> Resistors_SMD:R_0603

Commit message: all associated
Parts:
- D2, D3: value D -> BAS16GWJ
- U18: footprint TCT40-16R_T:TCT40-16R_T -> Custom:TCT40-16R_T
Other:
- moved on the sheet: D12, D13

Commit message: Routed rotational module
Parts:
- removed R70: 10K, Resistors_SMD:R_0603, symbol R
- renumbered C44 to C501, C45 to C502, C46 to C503, C47 to C504, C48 to C505, C49 to C506, C50 to C507, C51 to C508, D2 to D501, D3 to D502, Q4 to Q501, R65 to R501, R66 to R502, R67 to R503, R68 to R504, R69 to R505, R71 to R506, R72 to R507, R73 to R508, R74 to R509, R75 to R510, R76 to R511, R77 to R512, R78 to R513, R79 to R514, R80 to R515, R81 to R516, R82 to R517, U17 to U501, U18 to U502
