File: ultrasonic_localization/soundModule.sch (KiCad schematic (older format))
At the start: 30 parts, among them Q501 BC847, U501 LM324, U502 TCT40-16R/T

Commit message: added mux
Connections:
- net TXb is gone; now on net GND: U502.2
- net SWa renamed UX
- net SWb renamed RX

Commit message: Fixed board
Parts:
- C502: value 1.2uF -> 1uF
- R505: value 660 -> 665
- R507: value 40K -> 40.2K
- U501: footprint Housings_SOIC:SOIC-16_3.9x9.9mm_Pitch1.27mm -> Housings_SOIC:SOIC-14_3.9x8.7mm_Pitch1.27mm

Commit message: stuff
Other:
- note removed: "Consider Gain-Bandwidth Tradeoff"
- note removed: "NOTE : Flipped Op Amp"
- note removed: "TODO : In LTSpice sim, adjusting THRESH doesn't seem to do anything,\nwhereas it should have set reception sensitivity.\nSee https://uglyduck.ath.cx/ep/archive/2014/01/Making_a_better_HC_SR04_Echo_Locator.html For Reference"
- note removed: "TODO : Need a diode??"
