File: ultrasonic_localization/IMUModule.sch (KiCad schematic (older format))
At the start: 10 parts

Commit message: pushing stuff
Other:
- note added: "PULLUP INT?"
Changed lines of the file:
@@
 	2875 4025 2875 4225
 Wire Wire Line
-	2575 4225 3375 4225
+	2575 4225 2875 4225
+Wire Wire Line
+	2875 4225 3000 4225
+Wire Wire Line
+	3000 4225 3375 4225
 Connection ~ 2875 4225
 Wire Wire Line
-	3825 4575 3825 4875
+	3825 4575 3825 4700
+Wire Wire Line
+	3825 4700 3825 4875
 Wire Wire Line
 	3825 4875 4225 4875
@@
 	7625 4750 7625 4850
 Wire Wire Line
-	7625 4850 8575 4850
+	7625 4850 7875 4850
+Wire Wire Line
+	7875 4850 8125 4850
+Wire Wire Line
+	8125 4850 8325 4850
+Wire Wire Line
+	8325 4850 8575 4850
 Wire Wire Line
 	7875 4750 7875 4850
@@
 INT2
 Wire Wire Line
-	6475 3650 5775 3650
-Wire Wire Line
-	6475 3850 5775 3850
+	6475 3650 6125 3650
+Wire Wire Line
+	6125 3650 5775 3650
+Wire Wire Line
+	6475 3850 5900 3850
+Wire Wire Line
+	5900 3850 5775 3850
 Wire Wire Line
 	6125 3650 6125 4000
@@
 $EndComp
 Wire Wire Line
-	5575 4300 6125 4300
+	5575 4300 5900 4300
+Wire Wire Line
+	5900 4300 6125 4300
 Connection ~ 5900 4300
 Text HLabel 8325 3650 2    60   Input ~ 0
@@
 Text HLabel 7875 4050 2    60   Input ~ 0
 INT2
+Text Notes 7625 5000 0    60   ~ 0
+PULLUP INT?
 $EndSCHEMATC

Commit message: IMU pulldown
Connections:
- net +5V: no longer R?.2, R?.2
- net GND: now also R?.2, R?.2
Other:
- note removed: "PULLUP INT?"
Changed lines of the file:
@@
 	2875 4025 2875 4225
 Wire Wire Line
-	2575 4225 2875 4225
-Wire Wire Line
-	2875 4225 3000 4225
-Wire Wire Line
-	3000 4225 3375 4225
+	2575 4225 3375 4225
 Connection ~ 2875 4225
 Wire Wire Line
-	3825 4575 3825 4700
-Wire Wire Line
-	3825 4700 3825 4875
+	3825 4575 3825 4875
 Wire Wire Line
 	3825 4875 4225 4875
@@
 	7625 4750 7625 4850
 Wire Wire Line
-	7625 4850 7875 4850
-Wire Wire Line
-	7875 4850 8125 4850
-Wire Wire Line
-	8125 4850 8325 4850
-Wire Wire Line
-	8325 4850 8575 4850
-Wire Wire Line
-	7875 4750 7875 4850
-Connection ~ 7875 4850
+	7875 4850 7875 4750
 Wire Wire Line
 	8125 4750 8125 4850
@@
 INT2
 Wire Wire Line
-	6475 3650 6125 3650
-Wire Wire Line
-	6125 3650 5775 3650
-Wire Wire Line
-	6475 3850 5900 3850
-Wire Wire Line
-	5900 3850 5775 3850
+	5775 3650 6475 3650
+Wire Wire Line
+	5775 3850 6475 3850
 Wire Wire Line
 	6125 3650 6125 4000
@@
 $EndComp
 Wire Wire Line
-	5575 4300 5900 4300
-Wire Wire Line
-	5900 4300 6125 4300
+	5575 4300 6125 4300
 Connection ~ 5900 4300
 Text HLabel 8325 3650 2    60   Input ~ 0
@@
 Text HLabel 7875 4050 2    60   Input ~ 0
 INT2
-Text Notes 7625 5000 0    60   ~ 0
-PULLUP INT?
+$Comp
+L GND #PWR?
+U 1 1 5A04C7D6
+P 7725 4850
+F 0 "#PWR?" H 7725 4600 50  0001 C CNN
+F 1 "GND" H 7725 4700 50  0000 C CNN
+F 2 "" H 7725 4850 50  0001 C CNN
+F 3 "" H 7725 4850 50  0001 C CNN
+	1    7725 4850
+	1    0    0    -1
+$EndComp
+Wire Wire Line
+	7625 4850 7875 4850
+Connection ~ 7725 4850
+Wire Wire Line
+	8125 4850 8575 4850
 $EndSCHEMATC

Commit message: Assigned many footprints to things
Parts:
- U?: footprint (none) -> Housings_LGA:Bosch_LGA-14_3x2.5mm_Pitch0.5mm
- U?: footprint (none) -> Housings_SSOP:TSSOP-14_4.4x5mm_Pitch0.65mm
Changed lines of the file:
@@
 F 0 "U?" H 4025 3825 60  0000 C CNN
 F 1 "IMU" H 4025 3925 60  0000 C CNN
-F 2 "" H 4025 3925 60  0001 C CNN
+F 2 "Housings_LGA:Bosch_LGA-14_3x2.5mm_Pitch0.5mm" H 4025 3925 60  0001 C CNN
 F 3 "" H 4025 3925 60  0001 C CNN
 	1    4025 3925
@@
 F 0 "U?" H 6975 3750 60  0000 C CNN
 F 1 "Level_Shifter_4Channel" H 6975 4450 60  0000 C CNN
-F 2 "" H 6975 3750 60  0001 C CNN
+F 2 "Housings_SSOP:TSSOP-14_4.4x5mm_Pitch0.65mm" H 6975 3750 60  0001 C CNN
 F 3 "" H 6975 3750 60  0001 C CNN
 	1    6975 3750

Commit message: almost resolved DRC
Parts:
- gave numbers to parts that had none: 10
Connections:
- net L_HI is gone; now on an unnamed net: U2.1 (SDO/SA0)
Changed lines of the file:
@@
 $EndDescr
 $Comp
-L IMU U?
+L IMU U2
 U 1 1 5A13EED2
 P 4025 3925
-F 0 "U?" H 4025 3825 60  0000 C CNN
+F 0 "U2" H 4025 3825 60  0000 C CNN
 F 1 "IMU" H 4025 3925 60  0000 C CNN
 F 2 "Housings_LGA:Bosch_LGA-14_3x2.5mm_Pitch0.5mm" H 4025 3925 60  0001 C CNN
@@
 $EndComp
 $Comp
-L R R?
+L R R4
 U 1 1 5A13EED9
 P 2875 3875
-F 0 "R?" V 2955 3875 50  0000 C CNN
+F 0 "R4" V 2955 3875 50  0000 C CNN
 F 1 "10K" V 2875 3875 50  0000 C CNN
 F 2 "" V 2805 3875 50  0001 C CNN
@@
 $EndComp
 $Comp
-L C C?
+L C C6
 U 1 1 5A13EEE0
 P 4225 4725
-F 0 "C?" H 4250 4825 50  0000 L CNN
+F 0 "C6" H 4250 4825 50  0000 L CNN
 F 1 "100nF" H 4250 4625 50  0000 L CNN
 F 2 "" H 4263 4575 50  0001 C CNN
@@
 $EndComp
 $Comp
-L GND #PWR?
+L GND #PWR0120
 U 1 1 5A13EEE7
 P 3825 4875
-F 0 "#PWR?" H 3825 4625 50  0001 C CNN
+F 0 "#PWR0120" H 3825 4625 50  0001 C CNN
 F 1 "GND" H 3825 4725 50  0000 C CNN
 F 2 "" H 3825 4875 50  0001 C CNN
@@
 $EndComp
 $Comp
-L GND #PWR?
+L GND #PWR0121
 U 1 1 5A13EEED
 P 5125 4025
-F 0 "#PWR?" H 5125 3775 50  0001 C CNN
+F 0 "#PWR0121" H 5125 3775 50  0001 C CNN
 F 1 "GND" H 5125 3875 50  0000 C CNN
 F 2 "" H 5125 4025 50  0001 C CNN
@@
 $EndComp
 $Comp
-L +1V8 #PWR?
+L +1V8 #PWR0122
 U 1 1 5A13EEF3
 P 2575 4225
-F 0 "#PWR?" H 2575 4075 50  0001 C CNN
+F 0 "#PWR0122" H 2575 4075 50  0001 C CNN
 F 1 "+1V8" H 2575 4365 50  0000 C CNN
 F 2 "" H 2575 4225 50  0001 C CNN
@@
 	3825 3275 3825 3125
 Wire Wire Line
-	3825 3125 2875 3125
+	2875 3125 4675 3125
 Wire Wire Line
 	2875 3125 2875 3725
@@
 Text Label 4225 3275 1    60   ~ 0
 SDA_1V8
-Text Label 4675 3825 0    60   ~ 0
-L_HI
 Text Label 4675 4225 0    60   ~ 0
 INT1
@@
 NoConn ~ 3375 3825
 $Comp
-L Level_Shifter_4Channel U?
+L Level_Shifter_4Channel U4
 U 1 1 5A13EF11
 P 6975 3750
-F 0 "U?" H 6975 3750 60  0000 C CNN
+F 0 "U4" H 6975 3750 60  0000 C CNN
 F 1 "Level_Shifter_4Channel" H 6975 4450 60  0000 C CNN
 F 2 "Housings_SSOP:TSSOP-14_4.4x5mm_Pitch0.65mm" H 6975 3750 60  0001 C CNN
@@
 $EndComp
 $Comp
-L +5V #PWR?
+L +5V #PWR0123
 U 1 1 5A13EF18
 P 7800 3250
-F 0 "#PWR?" H 7800 3100 50  0001 C CNN
+F 0 "#PWR0123" H 7800 3100 50  0001 C CNN
 F 1 "+5V" H 7800 3390 50  0000 C CNN
 F 2 "" H 7800 3250 50  0001 C CNN
@@
 $EndComp
 $Comp
-L R R?
+L R R12
 U 1 1 5A13EF1E
 P 7875 4600
-F 0 "R?" V 7955 4600 50  0000 C CNN
+F 0 "R12" V 7955 4600 50  0000 C CNN
 F 1 "10K" V 7875 4600 50  0000 C CNN
 F 2 "" V 7805 4600 50  0001 C CNN
@@
 $EndComp
 $Comp
-L R R?
+L R R11
 U 1 1 5A13EF25
 P 7625 4600
-F 0 "R?" V 7705 4600 50  0000 C CNN
+F 0 "R11" V 7705 4600 50  0000 C CNN
 F 1 "10K" V 7625 4600 50  0000 C CNN
 F 2 "" V 7555 4600 50  0001 C CNN
@@
 $EndComp
 $Comp
-L R R?
+L R R13
 U 1 1 5A13EF2C
 P 8125 4600
-F 0 "R?" V 8205 4600 50  0000 C CNN
+F 0 "R13" V 8205 4600 50  0000 C CNN
 F 1 "10K" V 8125 4600 50  0000 C CNN
 F 2 "" V 8055 4600 50  0001 C CNN
@@
 $EndComp
 $Comp
-L R R?
+L R R14
 U 1 1 5A13EF33
 P 8325 4600
-F 0 "R?" V 8405 4600 50  0000 C CNN
+F 0 "R14" V 8405 4600 50  0000 C CNN
 F 1 "10K" V 8325 4600 50  0000 C CNN
 F 2 "" V 8255 4600 50  0001 C CNN
@@
 	7625 4250 7625 4450
 $Comp
-L +5V #PWR?
+L +5V #PWR0124
 U 1 1 5A13EF46
 P 8575 4850
-F 0 "#PWR?" H 8575 4700 50  0001 C CNN
+F 0 "#PWR0124" H 8575 4700 50  0001 C CNN
 F 1 "+5V" H 8575 4990 50  0000 C CNN
 F 2 "" H 8575 4850 50  0001 C CNN
@@
 	7800 3450 7800 3250
 $Comp
-L GND #PWR?
+L GND #PWR0125
 U 1 1 5A13EF57
 P 6175 3250
-F 0 "#PWR?" H 6175 3000 50  0001 C CNN
+F 0 "#PWR0125" H 6175 3000 50  0001 C CNN
 F 1 "GND" H 6175 3100 50  0000 C CNN
 F 2 "" H 6175 3250 50  0001 C CNN
@@
 	6475 3250 6175 3250
 $Comp
-L +1V8 #PWR?
+L +1V8 #PWR0126
 U 1 1 5A13EF5E
 P 6375 3450
-F 0 "#PWR?" H 6375 3300 50  0001 C CNN
+F 0 "#PWR0126" H 6375 3300 50  0001 C CNN
 F 1 "+1V8" H 6375 3590 50  0000 C CNN
 F 2 "" H 6375 3450 50  0001 C CNN
@@
 SCL_1V8
 $Comp
-L R R?
+L R R7
 U 1 1 5A13EF67
 P 6125 4150
-F 0 "R?" V 6205 4150 50  0000 C CNN
+F 0 "R7" V 6205 4150 50  0000 C CNN
 F 1 "10K" V 6125 4150 50  0000 C CNN
 F 2 "" V 6055 4150 50  0001 C CNN
@@
 $EndComp
 $Comp
-L R R?
+L R R6
 U 1 1 5A13EF6E
 P 5900 4150
-F 0 "R?" V 5980 4150 50  0000 C CNN
+F 0 "R6" V 5980 4150 50  0000 C CNN
 F 1 "10K" V 5900 4150 50  0000 C CNN
 F 2 "" V 5830 4150 50  0001 C CNN
@@
 Connection ~ 5900 3850
 $Comp
-L +1V8 #PWR?
+L +1V8 #PWR0127
 U 1 1 5A13EF7D
 P 5575 4300
-F 0 "#PWR?" H 5575 4150 50  0001 C CNN
+F 0 "#PWR0127" H 5575 4150 50  0001 C CNN
 F 1 "+1V8" H 5575 4440 50  0000 C CNN
 F 2 "" H 5575 4300 50  0001 C CNN
@@
 INT2
 $Comp
-L GND #PWR?
+L GND #PWR0128
 U 1 1 5A04C7D6
 P 7725 4850
-F 0 "#PWR?" H 7725 4600 50  0001 C CNN
+F 0 "#PWR0128" H 7725 4600 50  0001 C CNN
 F 1 "GND" H 7725 4700 50  0000 C CNN
 F 2 "" H 7725 4850 50  0001 C CNN
@@
 Wire Wire Line
 	8125 4850 8575 4850
+Wire Wire Line
+	4675 3125 4675 3825
+Connection ~ 3825 3125
 $EndSCHEMATC

Commit message: Assigned footprints to menial components
Parts:
- C6: footprint (none) -> Capacitors_SMD:C_0603
- R11, R12, R13, R14, R4, R6, R7: footprint (none) -> Resistors_SMD:R_0603
Changed lines of the file:
@@
 F 0 "R4" V 2955 3875 50  0000 C CNN
 F 1 "10K" V 2875 3875 50  0000 C CNN
-F 2 "" V 2805 3875 50  0001 C CNN
+F 2 "Resistors_SMD:R_0603" V 2805 3875 50  0001 C CNN
 F 3 "" H 2875 3875 50  0001 C CNN
 	1    2875 3875
@@
 F 0 "C6" H 4250 4825 50  0000 L CNN
 F 1 "100nF" H 4250 4625 50  0000 L CNN
-F 2 "" H 4263 4575 50  0001 C CNN
+F 2 "Capacitors_SMD:C_0603" H 4263 4575 50  0001 C CNN
 F 3 "" H 4225 4725 50  0001 C CNN
 	1    4225 4725
@@
 F 0 "R12" V 7955 4600 50  0000 C CNN
 F 1 "10K" V 7875 4600 50  0000 C CNN
-F 2 "" V 7805 4600 50  0001 C CNN
+F 2 "Resistors_SMD:R_0603" V 7805 4600 50  0001 C CNN
 F 3 "" H 7875 4600 50  0001 C CNN
 	1    7875 4600
@@
 F 0 "R11" V 7705 4600 50  0000 C CNN
 F 1 "10K" V 7625 4600 50  0000 C CNN
-F 2 "" V 7555 4600 50  0001 C CNN
+F 2 "Resistors_SMD:R_0603" V 7555 4600 50  0001 C CNN
 F 3 "" H 7625 4600 50  0001 C CNN
 	1    7625 4600
@@
 F 0 "R13" V 8205 4600 50  0000 C CNN
 F 1 "10K" V 8125 4600 50  0000 C CNN
-F 2 "" V 8055 4600 50  0001 C CNN
+F 2 "Resistors_SMD:R_0603" V 8055 4600 50  0001 C CNN
 F 3 "" H 8125 4600 50  0001 C CNN
 	1    8125 4600
@@
 F 0 "R14" V 8405 4600 50  0000 C CNN
 F 1 "10K" V 8325 4600 50  0000 C CNN
-F 2 "" V 8255 4600 50  0001 C CNN
+F 2 "Resistors_SMD:R_0603" V 8255 4600 50  0001 C CNN
 F 3 "" H 8325 4600 50  0001 C CNN
 	1    8325 4600
@@
 F 0 "R7" V 6205 4150 50  0000 C CNN
 F 1 "10K" V 6125 4150 50  0000 C CNN
-F 2 "" V 6055 4150 50  0001 C CNN
+F 2 "Resistors_SMD:R_0603" V 6055 4150 50  0001 C CNN
 F 3 "" H 6125 4150 50  0001 C CNN
 	1    6125 4150
@@
 F 0 "R6" V 5980 4150 50  0000 C CNN
 F 1 "10K" V 5900 4150 50  0000 C CNN
-F 2 "" V 5830 4150 50  0001 C CNN
+F 2 "Resistors_SMD:R_0603" V 5830 4150 50  0001 C CNN
 F 3 "" H 5900 4150 50  0001 C CNN
 	1    5900 4150

Commit message: Routed rotational module
Parts:
- renumbered C6 to C801, R4 to R801, R6 to R802, R7 to R803, R11 to R804, R12 to R805, R13 to R806, R14 to R807, U2 to U801, U4 to U802
Changed lines of the file:
@@
 $EndDescr
 $Comp
-L IMU U2
+L IMU U801
 U 1 1 5A13EED2
 P 4025 3925
-F 0 "U2" H 4025 3825 60  0000 C CNN
+F 0 "U801" H 4025 3825 60  0000 C CNN
 F 1 "IMU" H 4025 3925 60  0000 C CNN
 F 2 "Housings_LGA:Bosch_LGA-14_3x2.5mm_Pitch0.5mm" H 4025 3925 60  0001 C CNN
@@
 $EndComp
 $Comp
-L R R4
+L R R801
 U 1 1 5A13EED9
 P 2875 3875
-F 0 "R4" V 2955 3875 50  0000 C CNN
+F 0 "R801" V 2955 3875 50  0000 C CNN
 F 1 "10K" V 2875 3875 50  0000 C CNN
 F 2 "Resistors_SMD:R_0603" V 2805 3875 50  0001 C CNN
@@
 $EndComp
 $Comp
-L C C6
+L C C801
 U 1 1 5A13EEE0
 P 4225 4725
-F 0 "C6" H 4250 4825 50  0000 L CNN
+F 0 "C801" H 4250 4825 50  0000 L CNN
 F 1 "100nF" H 4250 4625 50  0000 L CNN
 F 2 "Capacitors_SMD:C_0603" H 4263 4575 50  0001 C CNN
@@
 $EndComp
 $Comp
-L GND #PWR121
+L GND #PWR0116
 U 1 1 5A13EEE7
 P 3825 4875
-F 0 "#PWR121" H 3825 4625 50  0001 C CNN
+F 0 "#PWR0116" H 3825 4625 50  0001 C CNN
 F 1 "GND" H 3825 4725 50  0000 C CNN
 F 2 "" H 3825 4875 50  0001 C CNN
@@
 $EndComp
 $Comp
-L GND #PWR122
+L GND #PWR0117
 U 1 1 5A13EEED
 P 5125 4025
-F 0 "#PWR122" H 5125 3775 50  0001 C CNN
+F 0 "#PWR0117" H 5125 3775 50  0001 C CNN
 F 1 "GND" H 5125 3875 50  0000 C CNN
 F 2 "" H 5125 4025 50  0001 C CNN
@@
 $EndComp
 $Comp
-L +1V8 #PWR120
+L +1V8 #PWR0118
 U 1 1 5A13EEF3
 P 2575 4225
-F 0 "#PWR120" H 2575 4075 50  0001 C CNN
+F 0 "#PWR0118" H 2575 4075 50  0001 C CNN
 F 1 "+1V8" H 2575 4365 50  0000 C CNN
 F 2 "" H 2575 4225 50  0001 C CNN
@@
 NoConn ~ 3375 3825
 $Comp
-L Level_Shifter_4Channel U4
+L Level_Shifter_4Channel U802
 U 1 1 5A13EF11
 P 6975 3750
-F 0 "U4" H 6975 3750 60  0000 C CNN
+F 0 "U802" H 6975 3750 60  0000 C CNN
 F 1 "Level_Shifter_4Channel" H 6975 4450 60  0000 C CNN
 F 2 "Housings_SSOP:TSSOP-14_4.4x5mm_Pitch0.65mm" H 6975 3750 60  0001 C CNN
@@
 $EndComp
 $Comp
-L +5V #PWR127
+L +5V #PWR0119
 U 1 1 5A13EF18
 P 7800 3250
-F 0 "#PWR127" H 7800 3100 50  0001 C CNN
+F 0 "#PWR0119" H 7800 3100 50  0001 C CNN
 F 1 "+5V" H 7800 3390 50  0000 C CNN
 F 2 "" H 7800 3250 50  0001 C CNN
@@
 $EndComp
 $Comp
-L R R12
+L R R805
 U 1 1 5A13EF1E
 P 7875 4600
-F 0 "R12" V 7955 4600 50  0000 C CNN
+F 0 "R805" V 7955 4600 50  0000 C CNN
 F 1 "10K" V 7875 4600 50  0000 C CNN
 F 2 "Resistors_SMD:R_0603" V 7805 4600 50  0001 C CNN
@@
 $EndComp
 $Comp
-L R R11
+L R R804
 U 1 1 5A13EF25
 P 7625 4600
-F 0 "R11" V 7705 4600 50  0000 C CNN
+F 0 "R804" V 7705 4600 50  0000 C CNN
 F 1 "10K" V 7625 4600 50  0000 C CNN
 F 2 "Resistors_SMD:R_0603" V 7555 4600 50  0001 C CNN
@@
 $EndComp
 $Comp
-L R R13
+L R R806
 U 1 1 5A13EF2C
 P 8125 4600
-F 0 "R13" V 8205 4600 50  0000 C CNN
+F 0 "R806" V 8205 4600 50  0000 C CNN
 F 1 "10K" V 8125 4600 50  0000 C CNN
 F 2 "Resistors_SMD:R_0603" V 8055 4600 50  0001 C CNN
@@
 $EndComp
 $Comp
-L R R14
+L R R807
 U 1 1 5A13EF33
 P 8325 4600
-F 0 "R14" V 8405 4600 50  0000 C CNN
+F 0 "R807" V 8405 4600 50  0000 C CNN
 F 1 "10K" V 8325 4600 50  0000 C CNN
 F 2 "Resistors_SMD:R_0603" V 8255 4600 50  0001 C CNN
@@
 	7625 4250 7625 4450
 $Comp
-L +5V #PWR128
+L +5V #PWR0120
 U 1 1 5A13EF46
 P 8575 4850
-F 0 "#PWR128" H 8575 4700 50  0001 C CNN
+F 0 "#PWR0120" H 8575 4700 50  0001 C CNN
 F 1 "+5V" H 8575 4990 50  0000 C CNN
 F 2 "" H 8575 4850 50  0001 C CNN
@@
 	7800 3450 7800 3250
 $Comp
-L GND #PWR124
+L GND #PWR0121
 U 1 1 5A13EF57
 P 6175 3250
-F 0 "#PWR124" H 6175 3000 50  0001 C CNN
+F 0 "#PWR0121" H 6175 3000 50  0001 C CNN
 F 1 "GND" H 6175 3100 50  0000 C CNN
 F 2 "" H 6175 3250 50  0001 C CNN
@@
 	6475 3250 6175 3250
 $Comp
-L +1V8 #PWR125
+L +1V8 #PWR0122
 U 1 1 5A13EF5E
 P 6375 3450
-F 0 "#PWR125" H 6375 3300 50  0001 C CNN
+F 0 "#PWR0122" H 6375 3300 50  0001 C CNN
 F 1 "+1V8" H 6375 3590 50  0000 C CNN
 F 2 "" H 6375 3450 50  0001 C CNN
@@
 SCL_1V8
 $Comp
-L R R7
+L R R803
 U 1 1 5A13EF67
 P 6125 4150
-F 0 "R7" V 6205 4150 50  0000 C CNN
+F 0 "R803" V 6205 4150 50  0000 C CNN
 F 1 "10K" V 6125 4150 50  0000 C CNN
 F 2 "Resistors_SMD:R_0603" V 6055 4150 50  0001 C CNN
@@
 $EndComp
 $Comp
-L R R6
+L R R802
 U 1 1 5A13EF6E
 P 5900 4150
-F 0 "R6" V 5980 4150 50  0000 C CNN
+F 0 "R802" V 5980 4150 50  0000 C CNN
 F 1 "10K" V 5900 4150 50  0000 C CNN
 F 2 "Resistors_SMD:R_0603" V 5830 4150 50  0001 C CNN
@@
 Connection ~ 5900 3850
 $Comp
-L +1V8 #PWR123
+L +1V8 #PWR0123
 U 1 1 5A13EF7D
 P 5575 4300
-F 0 "#PWR123" H 5575 4150 50  0001 C CNN
+F 0 "#PWR0123" H 5575 4150 50  0001 C CNN
 F 1 "+1V8" H 5575 4440 50  0000 C CNN
 F 2 "" H 5575 4300 50  0001 C CNN
@@
 INT2
 $Comp
-L GND #PWR126
+L GND #PWR0124
 U 1 1 5A04C7D6
 P 7725 4850
-F 0 "#PWR126" H 7725 4600 50  0001 C CNN
+F 0 "#PWR0124" H 7725 4600 50  0001 C CNN
 F 1 "GND" H 7725 4700 50  0000 C CNN
 F 2 "" H 7725 4850 50  0001 C CNN

Commit message: fixed symbols, some connections, and laid out submodules
Connections:
- net INT1: no longer U801.4 (INT1), U802.5 (A4)
- net INT2: no longer U801.9 (INT2), U802.4 (A3)
- new net INT1_1V8: U801.4 (INT1), U802.5 (A4)
- new net INT2_1V8: U801.9 (INT2), U802.4 (A3)
Changed lines of the file:
@@
 SDA_1V8
 Text Label 4675 4225 0    60   ~ 0
-INT1
+INT1_1V8
 Text Label 3375 4025 2    60   ~ 0
-INT2
+INT2_1V8
 NoConn ~ 3375 3625
 NoConn ~ 3375 3825
@@
 $EndComp
 Text Label 6475 4250 2    60   ~ 0
-INT1
+INT1_1V8
 Text Label 6475 4050 2    60   ~ 0
-INT2
+INT2_1V8
 Wire Wire Line
 	5775 3650 6475 3650
