File: ultrasonic_localization/IMUModule.sch (KiCad schematic (older format))
At the start: 10 parts, among them U801 IMU, U802 Level_Shifter_4Channel

Commit message: Routed most of the board
Parts:
- U802: symbol Level_Shifter_4Channel -> Level_Shifter_4Channel-RESCUE-ultrasonic_localization
Changed lines of the file:
@@
 EESchema Schematic File Version 2
+LIBS:ultrasonic_localization-rescue
 LIBS:power
 LIBS:device
@@
 NoConn ~ 3375 3825
 $Comp
-L Level_Shifter_4Channel U802
+L Level_Shifter_4Channel-RESCUE-ultrasonic_localization U802
 U 1 1 5A13EF11
 P 6975 3750
