File: ultrasonic_localization/ultrasonic_localization.kicad_pcb (KiCad board)
At the start: 2 copper layers, 212 parts, among them J101 USB_OTG_fix, J102 Conn_02x03_Odd_Even, J401 Screw_Terminal_1x02_Bat, Q101 BUK9Y29-40E, Q301 BC847, Q501 BC847, Q601 BC847, Q701 BC847, SW101 SW_Push, SW102 SW_DPDT, SW103 SW_DPDT, U101 ATMEGA32U4RC-AU, U102 MD0105, U103 4047, U201 nRF24L01+, U202 ANT016008LCS2442MA2, U301 LM324, U302 TCT40-16R/T, U401 AP3012, U402 AP3012, U403 TPS6223x, U404 LP5907SNX-3.3/NOPB, U405 BQ2423, U501 LM324, U502 TCT40-16R/T, U601 LM324, U602 TCT40-16R/T, U701 LM324, U702 TCT40-16R/T, U801 IMU, U802 Level_Shifter_4Channel, Y101 16MHz, Y201 16MHz

Commit message: fixed symbols, some connections, and laid out submodules
Parts:
- removed C301, C601, C701: 150nF, Capacitors_SMD:C_0603
- removed C302, C602, C702: 1.2uF, Capacitors_SMD:C_0603
- removed C303, C307, C308, C603, C607, C608, C703, C707, C708: 10nF, Capacitors_SMD:C_0603
- removed C304, C305, C604, C605, C704, C705: 1nF, Capacitors_SMD:C_0603
- removed C306, C606, C706: 12pF, Capacitors_SMD:C_0603
- removed D301, D302, D601, D602, D701, D702: BAS16GWJ, Diodes_SMD:D_SOD-123
- removed Q301, Q601, Q701: BC847, TO_SOT_Packages_SMD:SOT-23
- removed R301, R302, R306, R601, R602, R606, R701, R702, R706: 1K, Resistors_SMD:R_0603
- removed R303, R308, R314, R316, R603, R608, R614, R616, R703, R708, R714, R716: 10K, Resistors_SMD:R_0603
- removed R304, R604, R704: 62K, Resistors_SMD:R_0603
- removed R305, R605, R705: 660, Resistors_SMD:R_0603
- removed R307, R607, R707: 40K, Resistors_SMD:R_0603
- removed R309, R609, R709: 3.3M, Resistors_SMD:R_0603
- removed R310, R315, R610, R615, R710, R715: 120K, Resistors_SMD:R_0603
- removed R311, R312, R611, R612, R711, R712: 75K, Resistors_SMD:R_0603
- removed R313, R613, R713: 4.53K, Resistors_SMD:R_0603
- removed R317, R617, R717: 3.9K, Resistors_SMD:R_0603
- removed U301, U601, U701: LM324, Housings_SOIC:SOIC-16_3.9x9.9mm_Pitch1.27mm
- removed U302, U602, U702: TCT40-16R/T, Custom:TCT40-16R_T
- added C501: 150nF, Capacitors_SMD:C_0603, F.Cu at (94.1, 93.9)
- added C501: 150nF, Capacitors_SMD:C_0603, F.Cu at (98.2, 122.4)
- added C501: 150nF, Capacitors_SMD:C_0603, F.Cu at (85.3, 88.3)
- added C502: 1.2uF, Capacitors_SMD:C_0603, F.Cu at (95.5, 93.8)
- added C502: 1.2uF, Capacitors_SMD:C_0603, F.Cu at (97.6, 123.6)
- added C502: 1.2uF, Capacitors_SMD:C_0603, F.Cu at (84.6, 87.1)
- added C503: 10nF, Capacitors_SMD:C_0603, F.Cu at (95.5, 106.6)
- added C503: 10nF, Capacitors_SMD:C_0603, F.Cu at (86.5, 117.3)
- added C503: 10nF, Capacitors_SMD:C_0603, F.Cu at (95.6, 80.7)
- added C504: 1nF, Capacitors_SMD:C_0603, F.Cu at (103.5, 106.6)
- added C504: 1nF, Capacitors_SMD:C_0603, F.Cu at (82.5, 124.2)
- added C504: 1nF, Capacitors_SMD:C_0603, F.Cu at (91.6, 73.8)
- added C505: 1nF, Capacitors_SMD:C_0603, F.Cu at (104.9, 106.6)
- added C505: 1nF, Capacitors_SMD:C_0603, F.Cu at (81.8, 125.4)
- added C505: 1nF, Capacitors_SMD:C_0603, F.Cu at (90.9, 72.6)
- added C506: 12pF, Capacitors_SMD:C_0603, F.Cu at (108.0, 106.5)
- added C506: 12pF, Capacitors_SMD:C_0603, F.Cu at (80.3, 128.0)
- added C506: 12pF, Capacitors_SMD:C_0603, F.Cu at (89.3, 70.0)
- added C507: 10nF, Capacitors_SMD:C_0603, F.Cu at (107.6, 101.0)
- added C507: 10nF, Capacitors_SMD:C_0603, F.Cu at (85.3, 130.5)
- added C507: 10nF, Capacitors_SMD:C_0603, F.Cu at (84.7, 73.1)
- added C508: 10nF, Capacitors_SMD:C_0603, F.Cu at (105.4, 108.8)
- added C508: 10nF, Capacitors_SMD:C_0603, F.Cu at (79.6, 124.7)
- added C508: 10nF, Capacitors_SMD:C_0603, F.Cu at (92.6, 71.0)
- added D501: BAS16GWJ, Diodes_SMD:D_SOD-123, F.Cu at (93.6, 106.4)
- added D501: BAS16GWJ, Diodes_SMD:D_SOD-123, F.Cu at (87.6, 115.7)
- added D501: BAS16GWJ, Diodes_SMD:D_SOD-123, F.Cu at (96.4, 82.5)
- added D502: BAS16GWJ, Diodes_SMD:D_SOD-123, F.Cu at (93.6, 101.5)
- added D502: BAS16GWJ, Diodes_SMD:D_SOD-123, F.Cu at (91.9, 118.1)
- added D502: BAS16GWJ, Diodes_SMD:D_SOD-123, F.Cu at (92.1, 84.9)
- added Q501: BC847, TO_SOT_Packages_SMD:SOT-23, F.Cu at (94.1, 97.2)
- added Q501: BC847, TO_SOT_Packages_SMD:SOT-23, F.Cu at (95.4, 120.7)
- added Q501: BC847, TO_SOT_Packages_SMD:SOT-23, F.Cu at (88.1, 86.6)
- added R501: 1K, Resistors_SMD:R_0603, F.Cu at (97.0, 93.6)
- added R501: 1K, Resistors_SMD:R_0603, F.Cu at (97.0, 125.1)
- added R501: 1K, Resistors_SMD:R_0603, F.Cu at (83.6, 85.9)
- added R502: 1K, Resistors_SMD:R_0603, F.Cu at (98.6, 93.6)
- added R502: 1K, Resistors_SMD:R_0603, F.Cu at (96.2, 126.4)
- added R502: 1K, Resistors_SMD:R_0603, F.Cu at (82.8, 84.6)
- added R503: 10K, Resistors_SMD:R_0603, F.Cu at (95.5, 103.9)
- added R503: 10K, Resistors_SMD:R_0603, F.Cu at (88.9, 118.6)
- added R503: 10K, Resistors_SMD:R_0603, F.Cu at (93.2, 82.1)
- added R504: 62K, Resistors_SMD:R_0603, F.Cu at (97.0, 106.6)
- added R504: 62K, Resistors_SMD:R_0603, F.Cu at (85.8, 118.6)
- added R504: 62K, Resistors_SMD:R_0603, F.Cu at (94.8, 79.4)
- added R505: 660, Resistors_SMD:R_0603, F.Cu at (99.2, 106.6)
- added R505: 660, Resistors_SMD:R_0603, F.Cu at (84.7, 120.4)
- added R505: 660, Resistors_SMD:R_0603, F.Cu at (93.7, 77.5)
- added R506: 1K, Resistors_SMD:R_0603, F.Cu at (100.0, 108.8)
- added R506: 1K, Resistors_SMD:R_0603, F.Cu at (82.3, 120.0)
- added R506: 1K, Resistors_SMD:R_0603, F.Cu at (95.3, 75.7)
- added R507: 40K, Resistors_SMD:R_0603, F.Cu at (106.4, 106.4)
- added R507: 40K, Resistors_SMD:R_0603, F.Cu at (81.2, 126.8)
- added R507: 40K, Resistors_SMD:R_0603, F.Cu at (90.0, 71.3)
- added R508: 10K, Resistors_SMD:R_0603, F.Cu at (107.6, 103.7)
- added R508: 10K, Resistors_SMD:R_0603, F.Cu at (82.9, 129.1)
- added R508: 10K, Resistors_SMD:R_0603, F.Cu at (87.1, 71.7)
- added R509: 3.3M, Resistors_SMD:R_0603, F.Cu at (105.4, 110.4)
- added R509: 3.3M, Resistors_SMD:R_0603, F.Cu at (78.3, 123.9)
- added R509: 3.3M, Resistors_SMD:R_0603, F.Cu at (93.9, 70.3)
- added R510: 120K, Resistors_SMD:R_0603, F.Cu at (102.6, 108.8)
- added R510: 120K, Resistors_SMD:R_0603, F.Cu at (81.0, 122.3)
- added R510: 120K, Resistors_SMD:R_0603, F.Cu at (94.0, 73.4)
- added R511: 75K, Resistors_SMD:R_0603, F.Cu at (102.6, 110.4)
- added R511: 75K, Resistors_SMD:R_0603, F.Cu at (79.7, 121.5)
- added R511: 75K, Resistors_SMD:R_0603, F.Cu at (95.3, 72.7)
- added R512: 75K, Resistors_SMD:R_0603, F.Cu at (108.0, 98.3)
- added R512: 75K, Resistors_SMD:R_0603, F.Cu at (87.5, 132.2)
- added R512: 75K, Resistors_SMD:R_0603, F.Cu at (82.2, 74.1)
- added R513: 4.53K, Resistors_SMD:R_0603, F.Cu at (107.9, 96.8)
- added R513: 4.53K, Resistors_SMD:R_0603, F.Cu at (88.8, 132.9)
- added R513: 4.53K, Resistors_SMD:R_0603, F.Cu at (80.9, 74.9)
- added R514: 10K, Resistors_SMD:R_0603, F.Cu at (104.3, 96.0)
- added R514: 10K, Resistors_SMD:R_0603, F.Cu at (91.3, 130.1)
- added R514: 10K, Resistors_SMD:R_0603, F.Cu at (82.1, 78.4)
- added R515: 120K, Resistors_SMD:R_0603, F.Cu at (105.8, 96.0)
- added R515: 120K, Resistors_SMD:R_0603, F.Cu at (90.5, 131.4)
- added R515: 120K, Resistors_SMD:R_0603, F.Cu at (81.3, 77.1)
- added R516: 10K, Resistors_SMD:R_0603, F.Cu at (99.6, 96.1)
- added R516: 10K, Resistors_SMD:R_0603, F.Cu at (93.5, 126.0)
- added R516: 10K, Resistors_SMD:R_0603, F.Cu at (84.5, 82.4)
- added R517: 3.9K, Resistors_SMD:R_0603, F.Cu at (98.0, 96.1)
- added R517: 3.9K, Resistors_SMD:R_0603, F.Cu at (94.3, 124.7)
- added R517: 3.9K, Resistors_SMD:R_0603, F.Cu at (85.3, 83.7)
- added U501: LM324, Housings_SOIC:SOIC-16_3.9x9.9mm_Pitch1.27mm, F.Cu at (101.5, 101.2)
- added U501: LM324, Housings_SOIC:SOIC-16_3.9x9.9mm_Pitch1.27mm, F.Cu at (88.2, 125.1)
- added U501: LM324, Housings_SOIC:SOIC-16_3.9x9.9mm_Pitch1.27mm, F.Cu at (87.9, 78.3)
- added U502: TCT40-16R/T, Custom:TCT40-16R_T, F.Cu at (101.5, 101.2)
- added U502: TCT40-16R/T, Custom:TCT40-16R_T, F.Cu at (88.1, 125.1)
- added U502: TCT40-16R/T, Custom:TCT40-16R_T, F.Cu at (88.0, 78.2)
- Y101: value 16MHz -> Crystal_GND24
- moved U404 458.3 mm to (574.5, -9.13)
- moved C408 440.2 mm to (577.3, -9.14), turned to 270 degrees
- moved C406 431.9 mm to (558.3, -10.7), turned to 270 degrees
- moved D402 427.5 mm to (539.2, -8.89)
- moved U403 426.9 mm to (556.5, -10.7)
- moved U401 421.7 mm to (526.3, -9.40)
- moved C407 421.3 mm to (571.8, -8.39), turned to 90 degrees
- moved C405 420.2 mm to (538.7, -7.11)
- moved C401 417.0 mm to (554.5, -10.4), turned to 90 degrees
- moved L403 415.7 mm to (556.5, -13.2), turned to 180 degrees
- moved R408 415.0 mm to (543.6, 8.64)
- moved C409 414.3 mm to (535.9, 10.4), turned to 270 degrees
- moved C411 413.7 mm to (538.2, 13.0), turned to 180 degrees
- moved U402 410.9 mm to (542.3, -5.59)
- moved L402 409.9 mm to (543.1, -8.89)
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Connections:
- U801 pad 4: /D2 -> /IMU Module/INT1_1V8
- U801 pad 9: /D3 -> /IMU Module/INT2_1V8
- U802 pad 10: /SCL -> /D2
- U802 pad 11: +5V -> /D3
- U802 pad 12: +5V -> /SDA
- U802 pad 13: (no net) -> /SCL
- U802 pad 14: (no net) -> +5V
- U802 pad 4: /D3 -> /IMU Module/INT2_1V8
- U802 pad 5: /D2 -> /IMU Module/INT1_1V8
- U802 pad 6: GND -> (no net)
- U802 pad 7: /D2 -> GND
- U802 pad 8: /D3 -> +5V
- U802 pad 9: /SDA -> (no net)
- Y101 pad 3: GND -> Net-(C103-Pad1)
- Y101 pad 4: Net-(C103-Pad1) -> GND
Routing:
- net /Sound Module/VGND: track 24.6 -> 98.5 mm
- net /SIG1: track 21.5 -> 85.9 mm
- net Net-(C508-Pad1): track 19.6 -> 78.4 mm, vias 2 -> 8
- net GND: track 19.0 -> 76.0 mm
- net Net-(C504-Pad2): track 13.0 -> 51.9 mm
- net +5V: track 9.64 -> 38.6 mm, vias 2 -> 8
- net Net-(R512-Pad2): track 9.48 -> 37.9 mm
- net Net-(C503-Pad2): track 8.83 -> 35.3 mm
- net Net-(C504-Pad1): track 7.66 -> 30.7 mm
- net Net-(Q501-Pad1): track 7.09 -> 28.4 mm
- net Net-(C505-Pad2): track 6.49 -> 26.0 mm
- net Net-(R513-Pad1): track 6.16 -> 24.6 mm
- net Net-(R504-Pad1): track 4.09 -> 16.4 mm
- net Net-(C507-Pad2): track 3.45 -> 13.8 mm
- net Net-(R516-Pad1): track 1.60 -> 6.39 mm
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
Commit message: Routed most of the board
Parts:
- moved C408 492.0 mm to (101.1, 114.3), turned to 90 degrees
- moved U404 486.5 mm to (103.9, 114.3), turned to 180 degrees
- moved C407 480.8 mm to (106.7, 113.5), turned to 270 degrees
- moved C406 471.5 mm to (105.2, 119.5)
- moved L403 471.5 mm to (103.4, 117.0)
- moved U403 471.5 mm to (103.4, 119.5)
- moved C401 471.5 mm to (101.3, 119.8)
- moved D402 461.6 mm to (93.5, 111.0)
- moved U402 461.6 mm to (96.5, 114.3)
- moved C405 461.6 mm to (93.0, 112.8)
- moved L402 461.6 mm to (97.3, 111.0)
- moved C403 461.6 mm to (99.6, 114.3)
- moved R403 461.6 mm to (91.9, 115.1)
- moved R404 461.6 mm to (93.7, 115.1)
- moved R804 454.1 mm to (114.6, 108.3), turned to 270 degrees
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- renumbered C501 to C301, C502 to C302, C503 to C303, C504 to C304, C505 to C305, C506 to C306, C507 to C307, C508 to C308, C501 to C601, C502 to C602, C503 to C603, C504 to C604, C505 to C605, C506 to C606, C507 to C607, C508 to C608, C501 to C701, C502 to C702, C503 to C703, C504 to C704, C505 to C705, C506 to C706, C507 to C707, C508 to C708, D501 to D301, D502 to D302, D501 to D601, D502 to D602, D501 to D701, D502 to D702, Q501 to Q301, Q501 to Q601, Q501 to Q701, R501 to R301, R502 to R302, R503 to R303, R504 to R304, R505 to R305, R506 to R306, R507 to R307, R508 to R308, R509 to R309, R510 to R310, R511 to R311, R512 to R312, R513 to R313, R514 to R314, R515 to R315, R516 to R316, R517 to R317, R501 to R601, R502 to R602, R503 to R603, R504 to R604, R505 to R605, R506 to R606, R507 to R607, R508 to R608, R509 to R609, R510 to R610, R511 to R611, R512 to R612, R513 to R613, R514 to R614, R515 to R615, R516 to R616, R517 to R617, R501 to R701, R502 to R702, R503 to R703, R504 to R704, R505 to R705, R506 to R706, R507 to R707, R508 to R708, R509 to R709, R510 to R710, R511 to R711, R512 to R712, R513 to R713, R514 to R714, R515 to R715, R516 to R716, R517 to R717, U501 to U301, U502 to U302, U501 to U601, U502 to U602, U501 to U701, U502 to U702
Connections:
- C301 pad 2: /Sound Module/VGND -> /Sound Module 2/VGND
- C302 pad 2: /Sound Module/VGND -> /Sound Module 2/VGND
- C303 pad 1: Net-(C503-Pad1) -> Net-(C303-Pad1)
- C303 pad 2: Net-(C503-Pad2) -> Net-(C303-Pad2)
- C304 pad 1: Net-(C504-Pad1) -> Net-(C304-Pad1)
- C304 pad 2: Net-(C504-Pad2) -> Net-(C304-Pad2)
- C305 pad 1: Net-(C504-Pad1) -> Net-(C304-Pad1)
- C305 pad 2: Net-(C505-Pad2) -> Net-(C305-Pad2)
- C306 pad 1: Net-(C505-Pad2) -> Net-(C305-Pad2)
- C306 pad 2: Net-(C504-Pad2) -> Net-(C304-Pad2)
- C307 pad 1: Net-(C507-Pad1) -> Net-(C307-Pad1)
- C307 pad 2: Net-(C507-Pad2) -> Net-(C307-Pad2)
- C308 pad 1: Net-(C508-Pad1) -> Net-(C308-Pad1)
- C601 pad 2: /Sound Module/VGND -> /Sound Module 3/VGND
- C602 pad 2: /Sound Module/VGND -> /Sound Module 3/VGND
- C603 pad 1: Net-(C503-Pad1) -> Net-(C603-Pad1)
- C603 pad 2: Net-(C503-Pad2) -> Net-(C603-Pad2)
- C604 pad 1: Net-(C504-Pad1) -> Net-(C604-Pad1)
- C604 pad 2: Net-(C504-Pad2) -> Net-(C604-Pad2)
- C605 pad 1: Net-(C504-Pad1) -> Net-(C604-Pad1)
- C605 pad 2: Net-(C505-Pad2) -> Net-(C605-Pad2)
- C606 pad 1: Net-(C505-Pad2) -> Net-(C605-Pad2)
- C606 pad 2: Net-(C504-Pad2) -> Net-(C604-Pad2)
- C607 pad 1: Net-(C507-Pad1) -> Net-(C607-Pad1)
- C607 pad 2: Net-(C507-Pad2) -> Net-(C607-Pad2)
- C608 pad 1: Net-(C508-Pad1) -> Net-(C608-Pad1)
- C701 pad 2: /Sound Module/VGND -> /Sound Module 4/VGND
- C702 pad 2: /Sound Module/VGND -> /Sound Module 4/VGND
- C703 pad 1: Net-(C503-Pad1) -> Net-(C703-Pad1)
- C703 pad 2: Net-(C503-Pad2) -> Net-(C703-Pad2)
- C704 pad 1: Net-(C504-Pad1) -> Net-(C704-Pad1)
- C704 pad 2: Net-(C504-Pad2) -> Net-(C704-Pad2)
- C705 pad 1: Net-(C504-Pad1) -> Net-(C704-Pad1)
- C705 pad 2: Net-(C505-Pad2) -> Net-(C705-Pad2)
- C706 pad 1: Net-(C505-Pad2) -> Net-(C705-Pad2)
- C706 pad 2: Net-(C504-Pad2) -> Net-(C704-Pad2)
- C707 pad 1: Net-(C507-Pad1) -> Net-(C707-Pad1)
- C707 pad 2: Net-(C507-Pad2) -> Net-(C707-Pad2)
- C708 pad 1: Net-(C508-Pad1) -> Net-(C708-Pad1)
- D301 pad 1: /SW1b -> /SW2b
- D302 pad 2: /SW1b -> /SW2b
- D601 pad 1: /SW1b -> /SW3b
- D602 pad 2: /SW1b -> /SW3b
- D701 pad 1: /SW1b -> /SW4b
- D702 pad 2: /SW1b -> /SW4b
- Q301 pad 1: Net-(Q501-Pad1) -> Net-(Q301-Pad1)
- Q301 pad 3: /SIG1 -> /SIG2
- Q601 pad 1: Net-(Q501-Pad1) -> Net-(Q601-Pad1)
- Q601 pad 3: /SIG1 -> /SIG3
- Q701 pad 1: Net-(Q501-Pad1) -> Net-(Q701-Pad1)
- Q701 pad 3: /SIG1 -> /SIG4
- R301 pad 1: /Sound Module/VGND -> /Sound Module 2/VGND
- R302 pad 2: /Sound Module/VGND -> /Sound Module 2/VGND
- R303 pad 1: Net-(C503-Pad1) -> Net-(C303-Pad1)
- R303 pad 2: /SW1b -> /SW2b
- R304 pad 1: Net-(R504-Pad1) -> Net-(R304-Pad1)
- R304 pad 2: Net-(C503-Pad2) -> Net-(C303-Pad2)
- R305 pad 1: Net-(C504-Pad1) -> Net-(C304-Pad1)
- R305 pad 2: Net-(R504-Pad1) -> Net-(R304-Pad1)
- R306 pad 1: Net-(C504-Pad1) -> Net-(C304-Pad1)
- R306 pad 2: /Sound Module/VGND -> /Sound Module 2/VGND
- R307 pad 1: Net-(C505-Pad2) -> Net-(C305-Pad2)
- R307 pad 2: Net-(C504-Pad2) -> Net-(C304-Pad2)
- R308 pad 1: Net-(C504-Pad2) -> Net-(C304-Pad2)
- R308 pad 2: Net-(C507-Pad1) -> Net-(C307-Pad1)
- R309 pad 1: Net-(C508-Pad1) -> Net-(C308-Pad1)
- R310 pad 1: /Sound Module/VGND -> /Sound Module 2/VGND
- R310 pad 2: Net-(C508-Pad1) -> Net-(C308-Pad1)
- R311 pad 1: Net-(C508-Pad1) -> Net-(C308-Pad1)
- R312 pad 1: Net-(C507-Pad2) -> Net-(C307-Pad2)
- R312 pad 2: Net-(R512-Pad2) -> Net-(R312-Pad2)
- R313 pad 1: Net-(R513-Pad1) -> Net-(R313-Pad1)
- R313 pad 2: Net-(R512-Pad2) -> Net-(R312-Pad2)
- R314 pad 2: /SIG1 -> /SIG2
- R315 pad 1: /SIG1 -> /SIG2
- R315 pad 2: Net-(R513-Pad1) -> Net-(R313-Pad1)
- R316 pad 1: Net-(R516-Pad1) -> Net-(R316-Pad1)
- R316 pad 2: Net-(Q501-Pad1) -> Net-(Q301-Pad1)
- R317 pad 1: Net-(Q501-Pad1) -> Net-(Q301-Pad1)
- R601 pad 1: /Sound Module/VGND -> /Sound Module 3/VGND
- R602 pad 2: /Sound Module/VGND -> /Sound Module 3/VGND
- R603 pad 1: Net-(C503-Pad1) -> Net-(C603-Pad1)
- R603 pad 2: /SW1b -> /SW3b
- R604 pad 1: Net-(R504-Pad1) -> Net-(R604-Pad1)
- R604 pad 2: Net-(C503-Pad2) -> Net-(C603-Pad2)
- R605 pad 1: Net-(C504-Pad1) -> Net-(C604-Pad1)
- R605 pad 2: Net-(R504-Pad1) -> Net-(R604-Pad1)
- R606 pad 1: Net-(C504-Pad1) -> Net-(C604-Pad1)
- R606 pad 2: /Sound Module/VGND -> /Sound Module 3/VGND
- R607 pad 1: Net-(C505-Pad2) -> Net-(C605-Pad2)
- R607 pad 2: Net-(C504-Pad2) -> Net-(C604-Pad2)
- R608 pad 1: Net-(C504-Pad2) -> Net-(C604-Pad2)
- R608 pad 2: Net-(C507-Pad1) -> Net-(C607-Pad1)
- R609 pad 1: Net-(C508-Pad1) -> Net-(C608-Pad1)
- R610 pad 1: /Sound Module/VGND -> /Sound Module 3/VGND
- R610 pad 2: Net-(C508-Pad1) -> Net-(C608-Pad1)
- R611 pad 1: Net-(C508-Pad1) -> Net-(C608-Pad1)
- R612 pad 1: Net-(C507-Pad2) -> Net-(C607-Pad2)
- R612 pad 2: Net-(R512-Pad2) -> Net-(R612-Pad2)
- R613 pad 1: Net-(R513-Pad1) -> Net-(R613-Pad1)
- R613 pad 2: Net-(R512-Pad2) -> Net-(R612-Pad2)
- R614 pad 2: /SIG1 -> /SIG3
- R615 pad 1: /SIG1 -> /SIG3
- R615 pad 2: Net-(R513-Pad1) -> Net-(R613-Pad1)
- R616 pad 1: Net-(R516-Pad1) -> Net-(R616-Pad1)
- R616 pad 2: Net-(Q501-Pad1) -> Net-(Q601-Pad1)
- R617 pad 1: Net-(Q501-Pad1) -> Net-(Q601-Pad1)
- R701 pad 1: /Sound Module/VGND -> /Sound Module 4/VGND
- R702 pad 2: /Sound Module/VGND -> /Sound Module 4/VGND
- R703 pad 1: Net-(C503-Pad1) -> Net-(C703-Pad1)
- R703 pad 2: /SW1b -> /SW4b
- R704 pad 1: Net-(R504-Pad1) -> Net-(R704-Pad1)
- R704 pad 2: Net-(C503-Pad2) -> Net-(C703-Pad2)
- R705 pad 1: Net-(C504-Pad1) -> Net-(C704-Pad1)
- R705 pad 2: Net-(R504-Pad1) -> Net-(R704-Pad1)
- R706 pad 1: Net-(C504-Pad1) -> Net-(C704-Pad1)
- R706 pad 2: /Sound Module/VGND -> /Sound Module 4/VGND
- R707 pad 1: Net-(C505-Pad2) -> Net-(C705-Pad2)
- R707 pad 2: Net-(C504-Pad2) -> Net-(C704-Pad2)
- R708 pad 1: Net-(C504-Pad2) -> Net-(C704-Pad2)
- R708 pad 2: Net-(C507-Pad1) -> Net-(C707-Pad1)
- R709 pad 1: Net-(C508-Pad1) -> Net-(C708-Pad1)
- R710 pad 1: /Sound Module/VGND -> /Sound Module 4/VGND
- R710 pad 2: Net-(C508-Pad1) -> Net-(C708-Pad1)
- R711 pad 1: Net-(C508-Pad1) -> Net-(C708-Pad1)
- R712 pad 1: Net-(C507-Pad2) -> Net-(C707-Pad2)
- R712 pad 2: Net-(R512-Pad2) -> Net-(R712-Pad2)
- R713 pad 1: Net-(R513-Pad1) -> Net-(R713-Pad1)
- R713 pad 2: Net-(R512-Pad2) -> Net-(R712-Pad2)
- R714 pad 2: /SIG1 -> /SIG4
- R715 pad 1: /SIG1 -> /SIG4
- R715 pad 2: Net-(R513-Pad1) -> Net-(R713-Pad1)
- R716 pad 1: Net-(R516-Pad1) -> Net-(R716-Pad1)
- R716 pad 2: Net-(Q501-Pad1) -> Net-(Q701-Pad1)
- R717 pad 1: Net-(Q501-Pad1) -> Net-(Q701-Pad1)
- U301 pad 1: Net-(R504-Pad1) -> Net-(R304-Pad1)
- U301 pad 10: /Sound Module/VGND -> /Sound Module 2/VGND
- U301 pad 12: Net-(R513-Pad1) -> Net-(R313-Pad1)
- U301 pad 13: Net-(C508-Pad1) -> Net-(C308-Pad1)
- U301 pad 14: Net-(R516-Pad1) -> Net-(R316-Pad1)
- U301 pad 2: Net-(C503-Pad2) -> Net-(C303-Pad2)
- U301 pad 3: /Sound Module/VGND -> /Sound Module 2/VGND
- U301 pad 5: /Sound Module/VGND -> /Sound Module 2/VGND
- U301 pad 6: Net-(C505-Pad2) -> Net-(C305-Pad2)
- U301 pad 7: Net-(C504-Pad2) -> Net-(C304-Pad2)
- U301 pad 8: Net-(R512-Pad2) -> Net-(R312-Pad2)
- U301 pad 9: Net-(C507-Pad2) -> Net-(C307-Pad2)
- U601 pad 1: Net-(R504-Pad1) -> Net-(R604-Pad1)
- U601 pad 10: /Sound Module/VGND -> /Sound Module 3/VGND
- U601 pad 12: Net-(R513-Pad1) -> Net-(R613-Pad1)
- U601 pad 13: Net-(C508-Pad1) -> Net-(C608-Pad1)
- U601 pad 14: Net-(R516-Pad1) -> Net-(R616-Pad1)
- U601 pad 2: Net-(C503-Pad2) -> Net-(C603-Pad2)
- U601 pad 3: /Sound Module/VGND -> /Sound Module 3/VGND
- U601 pad 5: /Sound Module/VGND -> /Sound Module 3/VGND
- U601 pad 6: Net-(C505-Pad2) -> Net-(C605-Pad2)
- U601 pad 7: Net-(C504-Pad2) -> Net-(C604-Pad2)
- U601 pad 8: Net-(R512-Pad2) -> Net-(R612-Pad2)
- U601 pad 9: Net-(C507-Pad2) -> Net-(C607-Pad2)
- U701 pad 1: Net-(R504-Pad1) -> Net-(R704-Pad1)
- U701 pad 10: /Sound Module/VGND -> /Sound Module 4/VGND
- U701 pad 12: Net-(R513-Pad1) -> Net-(R713-Pad1)
- U701 pad 13: Net-(C508-Pad1) -> Net-(C708-Pad1)
- U701 pad 14: Net-(R516-Pad1) -> Net-(R716-Pad1)
- U701 pad 2: Net-(C503-Pad2) -> Net-(C703-Pad2)
- U701 pad 3: /Sound Module/VGND -> /Sound Module 4/VGND
- U701 pad 5: /Sound Module/VGND -> /Sound Module 4/VGND
- U701 pad 6: Net-(C505-Pad2) -> Net-(C705-Pad2)
- U701 pad 7: Net-(C504-Pad2) -> Net-(C704-Pad2)
- U701 pad 8: Net-(R512-Pad2) -> Net-(R712-Pad2)
- U701 pad 9: Net-(C507-Pad2) -> Net-(C707-Pad2)
- U802 pad 10: /D2 -> /SCL
- U802 pad 11: /D3 -> +5V
- U802 pad 12: /SDA -> +5V
- U802 pad 13: /SCL -> (no net)
- U802 pad 14: +5V -> (no net)
- U802 pad 6: (no net) -> GND
- U802 pad 7: GND -> /D2
- U802 pad 8: +5V -> /D3
- U802 pad 9: (no net) -> /SDA
Routing:
- net GND: track 76.0 -> 295.5 mm, vias 0 -> 28
- net /SW1a: track 0.00 -> 125.6 mm, vias 0 -> 17
- net /SW1b: track 0.00 -> 80.8 mm, vias 0 -> 2
- net +5V: track 38.6 -> 117.0 mm, vias 8 -> 14
- net /Sound Module/VGND: track 98.5 -> 24.6 mm
- net /Power/3V7: track 0.00 -> 73.4 mm, vias 0 -> 15
- net /RESET: track 0.00 -> 68.2 mm, vias 0 -> 1
- net /ID: track 0.00 -> 68.1 mm, vias 0 -> 2
- net /SW3b: track 0.00 -> 67.3 mm, vias 0 -> 2
- net /MISO: track 0.00 -> 65.3 mm, vias 0 -> 2
- net /THRESH: track 0.00 -> 60.5 mm, vias 0 -> 8
- net Net-(C508-Pad1): track 78.4 -> 19.6 mm, vias 8 -> 2
- net /SIG3: track 0.00 -> 50.7 mm, vias 0 -> 2
- net /OSC_MCU: track 0.00 -> 48.7 mm, vias 0 -> 4
- net /MOSI: track 0.00 -> 46.4 mm, vias 0 -> 4
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- added copper zone on B.Cu, net GND
Other:
- board outline added: 69.6 x 80.4 mm

Commit message: Finished routing
Routing:
- net +5V: track 117.0 -> 297.4 mm, vias 14 -> 34
- net GND: track 295.5 -> 438.4 mm, vias 28 -> 52
- net Net-(Q101-Pad4): track 0.00 -> 101.9 mm, vias 0 -> 2
- net /THRESH: track 60.5 -> 138.0 mm, vias 8 -> 17
- net /OSC_IC: track 1.88 -> 59.5 mm, vias 0 -> 2
- net /SCL: track 5.50 -> 62.1 mm, vias 0 -> 7
- net +1V8: track 18.8 -> 70.4 mm, vias 2 -> 7
- net /D2: track 9.67 -> 59.8 mm, vias 2 -> 4
- net /USB5V: track 19.2 -> 65.1 mm, vias 2 -> 10
- net /SDA: track 6.51 -> 52.3 mm, vias 0 -> 7
- net /D3: track 6.56 -> 44.2 mm, vias 0 -> 5
- net /Power/3V7: track 73.4 -> 104.3 mm, vias 15 -> 20
- net /SIG2: track 21.8 -> 43.2 mm, vias 0 -> 5
- net Net-(R101-Pad2): track 0.00 -> 20.0 mm, vias 0 -> 2
- net Net-(R102-Pad1): track 0.00 -> 19.9 mm, vias 0 -> 2
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
Commit message: Made all of the text nice
Routing:
- net GND: track 438.4 -> 445.5 mm, vias 52 -> 54
- net /USB5V: track 65.1 -> 65.6 mm
